Commit message: Ros2 Control integration and debugging Fixes #42

File: src/robot_description/arm_description/urdf/arm_real.xacro (robot description, xacro)
@@ -2,5 +2,5 @@
 <robot xmlns:xacro="http://ros.org/wiki/xacro">
     <xacro:include filename="$(find arm_description)/urdf/arm_base.xacro" />
-    <!-- <xacro:include filename="$(find arm_description)/urdf/macros/ros2_control.xacro" /> -->
-    <!-- <xacro:arm_ros2_control/> -->
+    <xacro:include filename="$(find arm_description)/urdf/macros/ros2_control.xacro" />
+    <xacro:arm_ros2_control/>
 </robot>

File: src/robot_description/arm_description/urdf/macros/ros2_control.xacro (robot description, xacro)
@@ -1,7 +1,9 @@
 <?xml version="1.0"?>
-<xacro:macro xmlns:xacro="http://ros.org/wiki/xacro">
+<robot xmlns:xacro="http://ros.org/wiki/xacro">
+<xacro:macro name="arm_ros2_control">
     <ros2_control name="ArmSystem" type="system">
         <hardware>
-            <plugin>arm_hardware/ArmHardwareInterface</plugin>
+            <!-- <plugin>arm_hardware/ArmHardwareInterface</plugin> -->
+                <plugin>gazebo_ros2_control/GazeboSystem</plugin>
         </hardware>
         <joint name="base_rotation_joint">
@@ -30,8 +32,5 @@
             <state_interface name="velocity" />
         </joint>
-        <joint name="end_effector_joint">
-            <command_interface name="position" />
-            <state_interface name="position" />
-        </joint>
     </ros2_control>
 </xacro:macro>
+</robot>
