Commit message: update base_fixture_link to base_link

File: src/robot_description/arm_description/urdf/arm_base.xacro (robot description, xacro)
@@ -4,5 +4,5 @@
     <xacro:include filename="$(find arm_description)/urdf/macros/materials.xacro" />
     <!-- Base link -->
-    <!-- <xacro:include filename="$(find arm_description)/urdf/links/base_fixture_link.xacro" /> -->
+    <!-- <xacro:include filename="$(find arm_description)/urdf/links/base_link.xacro" /> -->
     <!-- Arm Links -->
     <xacro:include filename="$(find arm_description)/urdf/links/arm_links.xacro" />

File: src/robot_description/arm_description/urdf/macros/camera.xacro (robot description, xacro)
@@ -27,5 +27,5 @@
     </link>
     <joint name="base_camera_joint" type="fixed">
-        <parent link="base_fixture_link" />
+        <parent link="base_link" />
         <child link="head_depth_camera_optical_frame" />
         <origin xyz="0 0 1.2" rpy="0 0 0" />

File: src/robot_description/arm_description/urdf/macros/depth_camera.xacro (robot description, xacro)
@@ -10,5 +10,5 @@
     Usage:
       <xacro:depth_camera
-        parent_link="base_fixture_link"
+        parent_link="base_link"
         xyz="0 0 0.15"
         rpy="0 0 0"
