Commit message: Add URDF and RViz configuration for 5-DOF humanoid arm system

File: src/robot_description/arm_description/urdf/humanoid_arm_5dof.urdf (robot description, URDF)
Before this commit: robot humanoid_arm_5dof, 14 links, 13 joints
Links:
- link base_link: geometry collision mesh filename=package://arm_description/meshes/visual/suport.STL; visual mesh filename=package://arm_description/meshes/visual/suport.STL
- link elbow_flange_link: geometry collision mesh filename=package://arm_description/meshes/visual/flansa .STL; visual mesh filename=package://arm_description/meshes/visual/flansa .STL
- link elbow_motor_link: geometry collision mesh filename=package://arm_description/meshes/visual/pmotor3.STL; visual mesh filename=package://arm_description/meshes/visual/pmotor3.STL
- link end_effector_link: geometry collision mesh filename=package://arm_description/meshes/visual/incheietura.STL; visual mesh filename=package://arm_description/meshes/visual/incheietura.STL
- link end_motor_link: geometry collision mesh filename=package://arm_description/meshes/visual/pmotor6.STL; visual mesh filename=package://arm_description/meshes/visual/pmotor6.STL
- link forearm_link: geometry collision mesh filename=package://arm_description/meshes/visual/umar2.STL; visual mesh filename=package://arm_description/meshes/visual/umar2.STL
- link shoulder_motor_link: geometry collision mesh filename=package://arm_description/meshes/visual/pmotor1.STL; visual mesh filename=package://arm_description/meshes/visual/pmotor1.STL
- link shoulder_pitch_motor_link: geometry collision mesh filename=package://arm_description/meshes/visual/pmotor2.STL; visual mesh filename=package://arm_description/meshes/visual/pmotor2.STL
- link upper_arm_link: geometry collision mesh filename=package://arm_description/meshes/visual/umar1.STL; visual mesh filename=package://arm_description/meshes/visual/umar1.STL
- link wrist_assembly_link: geometry collision mesh filename=package://arm_description/meshes/visual/cot3.STL; visual mesh filename=package://arm_description/meshes/visual/cot3.STL
- link wrist_base_link: geometry collision mesh filename=package://arm_description/meshes/visual/cot1.STL; visual mesh filename=package://arm_description/meshes/visual/cot1.STL
- link wrist_motor_link: geometry collision mesh filename=package://arm_description/meshes/visual/pmotor4.STL; visual mesh filename=package://arm_description/meshes/visual/pmotor4.STL
- link wrist_pitch_link: geometry collision mesh filename=package://arm_description/meshes/visual/cot2.STL; visual mesh filename=package://arm_description/meshes/visual/cot2.STL
- link wrist_roll_motor_link: geometry collision mesh filename=package://arm_description/meshes/visual/pmotor5.STL; visual mesh filename=package://arm_description/meshes/visual/pmotor5.STL

Commit message: Add new rpy axes for left hand

File: src/robot_description/arm_description/urdf/humanoid_arm_5dof.urdf (robot description, URDF)
Before this commit: robot humanoid_arm_5dof, 23 links, 22 joints
Links:
- removed link base_link
- removed link left_palm
- removed link left_palm_left_finger
- removed link left_palm_right_finger
- added link 1220_m4x16_left_shoulder_yaw_screws, mass 0.00141036418698184; collision mesh filename=package://humanoid_arm_5dof/meshes/1220_m4x16_left_shoulder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; visual mesh filename=package://humanoid_arm_5dof/meshes/1220_m4x16_left_shoulder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
- added link base_fixture_link, mass 400; collision mesh filename=package://humanoid_arm_5dof/meshes/base_fixture_link.STL; visual mesh filename=package://humanoid_arm_5dof/meshes/base_fixture_link.STL
- added link left_elbow_shaft, mass 16.3859228521728; collision mesh filename=package://humanoid_arm_5dof/meshes/left_elbow_shaft.STL; visual mesh filename=package://humanoid_arm_5dof/meshes/left_elbow_shaft.STL
- added link left_shoulder_yaw_shaft, mass 0.00090364967437399; collision mesh filename=package://humanoid_arm_5dof/meshes/left_shoulder_yaw_shaft.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; visual mesh filename=package://humanoid_arm_5dof/meshes/left_shoulder_yaw_shaft.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
- added link left_wrist_shaft, mass 0.000903649674373956; collision mesh filename=package://humanoid_arm_5dof/meshes/left_wrist_shaft.STL; visual mesh filename=package://humanoid_arm_5dof/meshes/left_wrist_shaft.STL
- added link m3x16_left_hand_screws, mass 0.00139374174732656; collision mesh filename=package://humanoid_arm_5dof/meshes/m3x16_left_hand_screws.S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; visual mesh filename=package://humanoid_arm_5dof/meshes/m3x16_left_hand_screws.S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
- added link m3x20_left_wrist_screws, mass 0.00162137028637932; collision mesh filename=package://humanoid_arm_5dof/meshes/m3x20_left_wrist_screws.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; visual mesh filename=package://humanoid_arm_5dof/meshes/m3x20_left_wrist_screws.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
- added link m4x16_eft_elbow_screws, mass 0.00270184358647762; collision mesh filename=package://humanoid_arm_5dof/meshes/m4x16_eft_elbow_screws.S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; visual mesh filename=package://humanoid_arm_5dof/meshes/m4x16_eft_elbow_screws.S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
- added link m4x16_left_shoulder_yaw_screws, mass 0.00270184474693414; collision mesh filename=package://humanoid_arm_5dof/meshes/m4x16_left_shoulder_yaw_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; visual mesh filename=package://humanoid_arm_5dof/meshes/m4x16_left_shoulder_yaw_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
- added link m4x20_left_wrist_screws, mass 0.00232797016313296; collision mesh filename=package://humanoid_arm_5dof/meshes/m4x20_left_wrist_screws.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; visual mesh filename=package://humanoid_arm_5dof/meshes/m4x20_left_wrist_screws.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
- added link m4x25_left_elbow_screws, mass 0.00270858033444499; collision mesh filename=package://humanoid_arm_5dof/meshes/m4x25_left_elbow_screws.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; visual mesh filename=package://humanoid_arm_5dof/meshes/m4x25_left_elbow_screws.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
- added link m4x25_left_shoulder_screws_roll, mass 0.00451430348886334; collision mesh filename=package://humanoid_arm_5dof/meshes/m4x25_left_shoulder_scre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; visual mesh filename=package://humanoid_arm_5dof/meshes/m4x25_left_shoulder_scre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
- added link m4x25_left_shoulder_yaw_screws, mass 0.00270858202481966; collision mesh filename=package://humanoid_arm_5dof/meshes/m4x25_left_shoulder_yaw_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; visual mesh filename=package://humanoid_arm_5dof/meshes/m4x25_left_shoulder_yaw_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
- added link m5x22_screws_left_shoulder_pitch, mass 0.00474644340626584; collision mesh filename=package://humanoid_arm_5dof/meshes/m5x22_screws_left_should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; visual mesh filename=package://humanoid_arm_5dof/meshes/m5x22_screws_left_should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
- added link m5x22_screws_left_shoulder_roll, mass 0.00610257053905775; collision mesh filename=package://humanoid_arm_5dof/meshes/m5x22_screws_left_should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; visual mesh filename=package://humanoid_arm_5dof/meshes/m5x22_screws_left_should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
- link left_elbow: mass 0.1949 -> 0.779765456040378; geometry collision mesh filename=package://humanoid_arm_5dof/meshes/left_elbow.STL; visual mesh filename=package://humanoid_arm_5dof/meshes/left_elbow.STL
- link left_elbow_rs03_actuator: mass 0.83 -> 0.35655089089686; geometry collision mesh filename=package://humanoid_arm_5dof/meshes/left_elbow_rs03_actuator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; visual mesh filename=package://humanoid_arm_5dof/meshes/left_elbow_rs03_actuator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
- link left_elbow_rs03_flange: mass 0.005 -> 0.00407555097398919; geometry collision mesh filename=package://humanoid_arm_5dof/meshes/left_elbow_rs03_flange.S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; visual mesh filename=package://humanoid_arm_5dof/meshes/left_elbow_rs03_flange.S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
- link left_hand: mass 0.07138 -> 0.285530357232192; geometry collision mesh filename=package://humanoid_arm_5dof/meshes/left_hand.STL; visual mesh filename=package://humanoid_arm_5dof/meshes/left_hand.STL
- link left_hand_rs02: mass 0.38 -> 0.180583065420556; geometry collision mesh filename=package://humanoid_arm_5dof/meshes/left_hand_rs02.STL; visual mesh filename=package://humanoid_arm_5dof/meshes/left_hand_rs02.STL
- link left_hand_rs02_flange: mass 0.0025 -> 0.00245793392108123; geometry collision mesh filename=package://humanoid_arm_5dof/meshes/left_hand_rs02_flange.STL; visual mesh filename=package://humanoid_arm_5dof/meshes/left_hand_rs02_flange.STL
- link left_shoulder_pitch: mass 0.29944 -> 1.19772099939528; geometry collision mesh filename=package://humanoid_arm_5dof/meshes/left_shoulder_pitch.STL; visual mesh filename=package://humanoid_arm_5dof/meshes/left_shoulder_pitch.STL
- link left_shoulder_pitch_rs04_actuator: mass 1.345 -> 0.517423577893353; geometry collision mesh filename=package://humanoid_arm_5dof/meshes/left_shoulder_pitch_rs04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; visual mesh filename=package://humanoid_arm_5dof/meshes/left_shoulder_pitch_rs04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
- link left_shoulder_pitch_rs04_flange: mass 0.0075 -> 0.00758352122244511; geometry collision mesh filename=package://humanoid_arm_5dof/meshes/left_shoulder_pitch_rs04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; visual mesh filename=package://humanoid_arm_5dof/meshes/left_shoulder_pitch_rs04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
- link left_shoulder_roll: mass 0.2494 -> 0.997620681307434; geometry collision mesh filename=package://humanoid_arm_5dof/meshes/left_shoulder_roll.STL; visual mesh filename=package://humanoid_arm_5dof/meshes/left_shoulder_roll.STL
- link left_shoulder_roll_rs04_actuator: mass 1.345 -> 0.517423577893355; geometry collision mesh filename=package://humanoid_arm_5dof/meshes/left_shoulder_roll_rs04_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; visual mesh filename=package://humanoid_arm_5dof/meshes/left_shoulder_roll_rs04_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
- link left_shoulder_roll_rs04_flange: mass 0.0075 -> 0.00758352122244512; geometry collision mesh filename=package://humanoid_arm_5dof/meshes/left_shoulder_roll_rs04_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; visual mesh filename=package://humanoid_arm_5dof/meshes/left_shoulder_roll_rs04_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
- link left_shoulder_yaw: mass 0.122018 -> 0.488068654987172; geometry collision mesh filename=package://humanoid_arm_5dof/meshes/left_shoulder_yaw.STL; visual mesh filename=package://humanoid_arm_5dof/meshes/left_shoulder_yaw.STL
- link left_shoulder_yaw_flange: mass 0.008838 -> 0.035353146109953; geometry collision mesh filename=package://humanoid_arm_5dof/meshes/left_shoulder_yaw_flange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; visual mesh filename=package://humanoid_arm_5dof/meshes/left_shoulder_yaw_flange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
- link left_shoulder_yaw_rs03_actuator: mass 0.83 -> 0.356550969588106; geometry collision mesh filename=package://humanoid_arm_5dof/meshes/left_shoulder_yaw_rs03_a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; visual mesh filename=package://humanoid_arm_5dof/meshes/left_shoulder_yaw_rs03_a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
- link left_shoulder_yaw_rs03_flange: mass 0.005 -> 0.00407555097398896; geometry collision mesh filename=package://humanoid_arm_5dof/meshes/left_shoulder_yaw_rs03_f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; visual mesh filename=package://humanoid_arm_5dof/meshes/left_shoulder_yaw_rs03_f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
- link left_wrist: mass 0.09723 -> 0.388950905166551; geometry collision mesh filename=package://humanoid_arm_5dof/meshes/left_wrist.STL; visual mesh filename=package://humanoid_arm_5dof/meshes/left_wrist.STL
- link left_wrist_actuator: mass 0.38 -> 0.180583065420556; geometry collision mesh filename=package://humanoid_arm_5dof/meshes/left_wrist_actuator.STL; visual mesh filename=package://humanoid_arm_5dof/meshes/left_wrist_actuator.STL
- link left_wrist_rs02_flange: mass 0.0025 -> 0.00245793392108141; geometry collision mesh filename=package://humanoid_arm_5dof/meshes/left_wrist_rs02_flange.S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; visual mesh filename=package://humanoid_arm_5dof/meshes/left_wrist_rs02_flange.S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
Joints:
- removed joint left_elbow_fixture
- removed joint left_elbow_rs03
- removed joint left_hand_fixture
- removed joint left_hand_rs02
- removed joint left_palm_fixture
- removed joint left_palm_left_finger
- removed joint left_palm_right_finger
- removed joint left_shoulde_roll_fixture
- removed joint left_shoulder_pitch_fixture
- removed joint left_shoulder_pitch_rs04
- removed joint left_shoulder_roll_rs04
- removed joint left_shoulder_roll_rs04_flange
- removed joint left_shoulder_yaw_fixture
- removed joint left_shoulder_yaw_flange_fixture
- removed joint left_shoulder_yaw_rs03
- removed joint left_wrist_fixture
- removed joint left_wrist_rs02
- removed joint left_wrist_rs02_actuator_fixture_link
- added joint 1220_m4x16_left_shoulder_yaw_screws_fixture_joint: type fixed, parent left_shoulder_yaw_flange, child 1220_m4x16_left_shoulder_yaw_screws, origin xyz=0 0 0 rpy=0 0 0, axis 0 0 0
- added joint left_elbow_fixture_joint: type fixed, parent m4x25_left_elbow_screws, child left_elbow, origin xyz=0 0 0 rpy=0 0 0, axis 0 0 0
- added joint left_elbow_rs03_joint: type revolute, parent left_elbow_rs03_actuator, child left_elbow_rs03_flange, origin xyz=0 0 0 rpy=0 0 0, axis 0.442871169532447 0.896585259301625 0, limit lower=-1.3 upper=1.9 effort=60 velocity=1.6
- added joint left_elbow_shaft_fixture_joint: type fixed, parent left_elbow_rs03_flange, child left_elbow_shaft, origin xyz=0 0 0 rpy=0 0 0, axis 0 0 0
- added joint left_hand_fixture_joint: type fixed, parent left_hand_rs02_flange, child left_hand, origin xyz=0 0 0 rpy=0 0 0, axis 0 0 0
- added joint left_hand_rs02_joint: type revolute, parent left_hand_rs02, child left_hand_rs02_flange, origin xyz=0 0 0 rpy=0 0 0, axis 0.999999999999999 0 0, limit lower=-1.5 upper=1.7 effort=17 velocity=0.8
- added joint left_shoulde_roll_fixture_joint: type fixed, parent m4x25_left_shoulder_screws_roll, child left_shoulder_roll, origin xyz=0 0 0 rpy=0 0 0, axis 0 0 0
- added joint left_shoulder_pitch_fixture_joint: type fixed, parent m5x22_screws_left_shoulder_pitch, child left_shoulder_pitch, origin xyz=0 0 0 rpy=0 0 0, axis 0 0 0
- added joint left_shoulder_pitch_rs04_joint: type revolute, parent left_shoulder_pitch_rs04_actuator, child left_shoulder_pitch_rs04_flange, origin xyz=0 0 0 rpy=0 0 0, axis 1 0 0, limit lower=-3.14 upper=3.14 effort=120 velocity=3
- added joint left_shoulder_roll_rs04_flange_joint: type fixed, parent m5x22_screws_left_shoulder_roll, child left_shoulder_roll_rs04_flange, origin xyz=0.116775431275821 0.0487000000004332 -2.70558071411298E-05 rpy=0 0 0, axis 0 0 0
- added joint left_shoulder_roll_rs04_joint: type revolute, parent left_shoulder_roll_rs04_flange, child left_shoulder_roll_rs04_actuator, origin xyz=0 0 0 rpy=0 0 0, axis 0 -1 0, limit lower=-3.5 upper=0.6 effort=120 velocity=3
- added joint left_shoulder_yaw_fixture_joint: type fixed, parent m4x25_left_shoulder_yaw_screws, child left_shoulder_yaw, origin xyz=0 0 0 rpy=0 0 0, axis 0 0 0
- added joint left_shoulder_yaw_flange_fixture_joint: type fixed, parent left_shoulder_yaw_shaft, child left_shoulder_yaw_flange, origin xyz=0 0 0 rpy=0 0 0, axis 0 0 0
- added joint left_shoulder_yaw_rs03_joint: type revolute, parent left_shoulder_yaw_rs03_actuator, child left_shoulder_yaw_rs03_flange, origin xyz=0 0 0 rpy=0 0 0, axis 0 0 1, limit lower=-3.14 upper=3.14 effort=60 velocity=1.6
- added joint left_shoulder_yaw_shaft_fixture_joint: type fixed, parent left_shoulder_yaw_rs03_flange, child left_shoulder_yaw_shaft, origin xyz=0 0 0 rpy=0 0 0, axis 0 0 0, limit lower=0 upper=0 effort=0 velocity=0
- added joint left_wrist_actuator_fixture_link: type fixed, parent m3x20_left_wrist_screws, child left_wrist_actuator, origin xyz=0 0 0 rpy=0 0 0, axis 0 0 0
- added joint left_wrist_fixture_joint: type fixed, parent left_wrist_shaft, child left_wrist, origin xyz=0 0 0 rpy=0 0 0, axis 0 0 0
- added joint left_wrist_rs02_joint: type revolute, parent left_wrist_actuator, child left_wrist_rs02_flange, origin xyz=0 0 0 rpy=0 0 0, axis 0 1 0, limit lower=-3.14 upper=3.14 effort=17 velocity=0.8
- added joint left_wrist_shaft_fixture_joint: type fixed, parent m4x20_left_wrist_screws, child left_wrist_shaft, origin xyz=0 0 0 rpy=0 0 0, axis 0 0 0
- added joint m3x16_left_hand_screws_fixture_joint: type fixed, parent left_wrist, child m3x16_left_hand_screws, origin xyz=0 0.0944999999998815 0 rpy=0 0 0, axis 0 0 0
- added joint m3x20_left_wrist_screws_fixture_joint: type fixed, parent left_elbow, child m3x20_left_wrist_screws, origin xyz=0.0370688771049235 -0.0244446769789257 -0.15848929336033 rpy=0 0 0, axis 0 0 0
- added joint m4x16_eft_elbow_screws_fixture_joint: type fixed, parent left_shoulder_yaw, child m4x16_eft_elbow_screws, origin xyz=0 0 -0.0987000004167595 rpy=0 0 0, axis 0 0 0
- added joint m4x16_left_shoulder_yaw_screws_fixture_joint: type fixed, parent left_shoulder_roll, child m4x16_left_shoulder_yaw_screws, origin xyz=-0.0219716026665047 0.037700000000231 -0.173578614834026 rpy=0.0571232457871902 0.112571265320765 0.47087557604578, axis 0 0 0
- added joint m4x20_left_wrist_screws_fixture_joint: type fixed, parent left_wrist_rs02_flange, child m4x20_left_wrist_screws, origin xyz=0 0 0 rpy=0 0 0, axis 0 0 0
- added joint m4x25_left_elbow_screws_fixture_joint: type fixed, parent left_elbow_shaft, child m4x25_left_elbow_screws, origin xyz=0 0 0 rpy=0 0 0, axis 0 0 0
- added joint m4x25_left_shoulder_screws_roll_fixture_joint: type fixed, parent left_shoulder_roll_rs04_actuator, child m4x25_left_shoulder_screws_roll, origin xyz=0 0 0 rpy=0 0 0, axis 0 0 0
- added joint m4x25_left_shoulder_yaw_screws_fixture_joint: type fixed, parent 1220_m4x16_left_shoulder_yaw_screws, child m4x25_left_shoulder_yaw_screws, origin xyz=0 0 0 rpy=0 0 0, axis 0 0 0
- added joint m5x22_screws_left_shoulder_pitch_fixture_joint: type fixed, parent left_shoulder_pitch_rs04_flange, child m5x22_screws_left_shoulder_pitch, origin xyz=0 0 0 rpy=0 0 0, axis 0 0 0
- added joint m5x22_screws_left_shoulder_roll_fixture_joint: type fixed, parent left_shoulder_pitch, child m5x22_screws_left_shoulder_roll, origin xyz=0 0 0 rpy=0 0 0, axis 0 0 0
- joint left_elbow_rs03_actuator_ficture_link: origin xyz=0 0 -0.0987 rpy=0 0 0 -> xyz=0 0 0 rpy=0 0 0; parent left_shoulder_yaw -> m4x16_eft_elbow_screws
- joint left_hand_rs02_fixture_link: origin xyz=0 0.0945 0 rpy=0.64485 0.44406 0 -> xyz=0 0 0 rpy=0 0 0; parent left_wrist -> m3x16_left_hand_screws
- joint left_shoulder_pitch_rs04_actuator_fixture_link: origin xyz=-0.1079 0 1.425 rpy=-0.67594 0 3.1416 -> xyz=0 0.382699999999936 1.45000000000145 rpy=0 0 0; parent base_link -> base_fixture_link
- joint left_shoulder_yaw_rs03_actuator_fixture_link: origin xyz=-0.021972 0.0377 -0.17358 rpy=0.057123 0.11257 0.47088 -> xyz=0 0 0 rpy=0 0 0; parent left_shoulder_roll -> m4x16_left_shoulder_yaw_screws
