Commit message: arm_description xacro/macros Fixes #35

File: src/robot_description/arm_description/urdf/arm.urdf.xacro (robot description, xacro)
@@ -2,12 +2,16 @@
 <robot xmlns:xacro="http://ros.org/wiki/xacro" name="arm_description">
     <!-- Include common macros -->
-    <!-- <xacro:include filename="$(find arm_description)/urdf/macros/materials.xacro" />
-  <xacro:include filename="$(find arm_description)/urdf/macros/utils.xacro" /> -->
-    <!-- Select robot variant (base, gazebo, or real) -->
-    <xacro:arg name="use_sim" default="false" />
+    <!-- <xacro:include
+        filename="$(find arm_description)/urdf/macros/materials.xacro" /> -->
+    <!-- <xacro:include
+        filename="$(find arm_description)/urdf/macros/utils.xacro" />  -->
+        <!-- Select robot variant(base, gazebo, or real) -->
+    <xacro:arg name="use_sim"
+        default="false" />
     <xacro:if value="$(arg use_sim)">
         <xacro:include filename="$(find arm_description)/urdf/arm_gazebo.xacro" />
     </xacro:if>
-    <xacro:unless value="$(arg use_sim)">
+    <xacro:unless
+        value="$(arg use_sim)">
         <xacro:include filename="$(find arm_description)/urdf/arm_real.xacro" />
     </xacro:unless>

File: src/robot_description/arm_description/urdf/arm_base.xacro (robot description, xacro)
@@ -2,5 +2,5 @@
 <robot xmlns:xacro="http://ros.org/wiki/xacro">
     <!-- Include macros -->
-    <!-- <xacro:include filename="$(find arm_description)/urdf/macros/materials.xacro" /> -->
+    <xacro:include filename="$(find arm_description)/urdf/macros/materials.xacro" />
     <!-- Base link -->
     <!-- <xacro:include filename="$(find arm_description)/urdf/links/base_link.xacro" /> -->

File: src/robot_description/arm_description/urdf/links/arm_links.xacro (robot description, xacro)
@@ -25,8 +25,5 @@
       </geometry>
       <material
-        name="">
-        <color
-          rgba="0.82353 0.82353 1 1" />
-      </material>
+        name="transparent"/>
     </visual>
     <collision>
@@ -103,8 +100,5 @@
       </geometry>
       <material
-        name="">
-        <color
-          rgba="0.792156862745098 0.819607843137255 0.933333333333333 1" />
-      </material>
+         name="transparent"/>
     </visual>
     <collision>

Commit message: Add Inspire left hand Fixes #117

File: src/robot_description/arm_description/urdf/arm.urdf.xacro (robot description, xacro)
@@ -9,4 +9,6 @@
     <xacro:arg name="use_sim"
         default="false" />
+    <xacro:arg name="hand_type"
+        default="inspire_hand" />
     <xacro:if value="$(arg use_sim)">
         <xacro:include filename="$(find arm_description)/urdf/arm_gazebo.xacro" />

File: src/robot_description/arm_description/urdf/arm_base.xacro (robot description, xacro)
@@ -9,3 +9,15 @@
     <!-- Arm Joints -->
     <xacro:include filename="$(find arm_description)/urdf/joints/arm_joints.xacro" />
+    <!-- Hand/Gripper macros -->
+    <xacro:include filename="$(find arm_description)/urdf/hands/simple_gripper.xacro" />
+    <xacro:include filename="$(find arm_description)/urdf/hands/inspire_hand_left.xacro" />
+    <!-- Resolve hand_type arg into a property for conditional evaluation -->
+    <xacro:property name="hand_type" value="$(arg hand_type)"/>
+    <!-- Conditionally instantiate hand based on hand_type arg -->
+    <xacro:if value="${hand_type == 'simple_gripper'}">
+        <xacro:simple_gripper parent="end_effector_link"/>
+    </xacro:if>
+    <xacro:if value="${hand_type == 'inspire_hand'}">
+        <xacro:inspire_hand_left parent="end_effector_link"/>
+    </xacro:if>
 </robot>

File: src/robot_description/arm_description/urdf/arm_gazebo.xacro (robot description, xacro)
@@ -10,5 +10,5 @@
     <!-- Load ros2_control macro -->
     <xacro:include filename="$(find arm_description)/urdf/macros/ros2_control.xacro"/>
-    <xacro:arm_ros2_control/>
+    <xacro:arm_ros2_control hand_type="$(arg hand_type)"/>
     <!-- Depth Camera -->
     <xacro:include filename="$(find arm_description)/urdf/macros/depth_camera.xacro"/>

File: src/robot_description/arm_description/urdf/arm_real.xacro (robot description, xacro)
@@ -3,4 +3,4 @@
     <xacro:include filename="$(find arm_description)/urdf/arm_base.xacro" />
     <xacro:include filename="$(find arm_description)/urdf/macros/ros2_control.xacro" />
-    <xacro:arm_ros2_control/>
+    <xacro:arm_ros2_control hand_type="$(arg hand_type)"/>
 </robot>

File: src/robot_description/arm_description/urdf/joints/arm_joints.xacro (robot description, xacro)
@@ -61,30 +61,3 @@
     <dynamics damping="0.5" friction="0.1"/>
   </joint>
-  <!-- Gripper: Fixed joint from wrist to palm -->
-  <joint name="palm_fixture" type="fixed">
-    <origin xyz="0 0.09 -0.02" rpy="0 0 0"/>
-    <parent link="end_effector_link"/>
-    <child link="left_palm"/>
-  </joint>
-  <!-- Gripper: Right finger (independent control) -->
-  <joint name="left_palm_right_finger" type="prismatic">
-    <origin xyz="0 0 0" rpy="0 0 0"/>
-    <parent link="left_palm"/>
-    <child link="left_palm_right_finger_link"/>
-    <axis xyz="-1 0 0"/>
-    <limit lower="-0.04" upper="0.0" effort="10" velocity="0.05"/>
-    <safety_controller soft_upper_limit="0.0" soft_lower_limit="-0.04" k_velocity="0"/>
-    <dynamics damping="0.1" friction="0.1"/>
-  </joint>
-  <!-- Gripper: Left finger (mimic of right finger) -->
-  <joint name="left_palm_left_finger" type="prismatic">
-    <origin xyz="0 0 0" rpy="0 0 0"/>
-    <parent link="left_palm"/>
-    <child link="left_palm_left_finger_link"/>
-    <axis xyz="-1 0 0"/>
-    <limit lower="0.0" upper="0.04" effort="10" velocity="0.05"/>
-    <safety_controller soft_upper_limit="0.04" soft_lower_limit="0.0" k_velocity="0"/>
-    <mimic joint="left_palm_right_finger" multiplier="-1.0" offset="0"/>
-    <dynamics damping="0.1" friction="1.0"/>
-  </joint>
 </robot>

File: src/robot_description/arm_description/urdf/links/arm_links.xacro (robot description, xacro)
@@ -453,68 +453,3 @@
     </collision>
   </link>
-  <!-- Gripper: Palm -->
-  <link name="left_palm">
-    <inertial>
-      <origin xyz="0 0.0065 0" rpy="0 0 0"/>
-      <mass value="0.048"/>
-      <inertia ixx="0.000148" ixy="0" ixz="0" iyy="0.000377" iyz="0" izz="0.000285"/>
-    </inertial>
-    <visual>
-      <origin xyz="0 0 0" rpy="0 0 0"/>
-      <geometry>
-        <mesh filename="package://arm_description/meshes/visual/left_palm.stl"/>
-      </geometry>
-      <material name="grey">
-        <color rgba="0.698 0.698 0.698 1"/>
-      </material>
-    </visual>
-    <collision>
-      <origin xyz="0 0 0" rpy="0 0 0"/>
-      <geometry>
-        <mesh filename="package://arm_description/meshes/visual/left_palm.stl"/>
-      </geometry>
-    </collision>
-  </link>
-  <!-- Gripper: Right finger (controlled) -->
-  <link name="left_palm_right_finger_link">
-    <inertial>
-      <origin xyz="0.022 0.050 0" rpy="0 0 0"/>
-      <mass value="0.029"/>
-      <inertia ixx="0.000106" ixy="1.28e-05" ixz="0" iyy="4.91e-05" iyz="0" izz="8.9e-05"/>
-    </inertial>
-    <visual>
-      <origin xyz="-0.005 0 0" rpy="0 0 0"/>
-      <geometry>
-        <mesh filename="package://arm_description/meshes/visual/left_palm_right_finger.stl"/>
-      </geometry>
-      <material name="grey"/>
-    </visual>
-    <collision>
-      <origin xyz="-0.005 0 0" rpy="0 0 0"/>
-      <geometry>
-        <mesh filename="package://arm_description/meshes/visual/left_palm_right_finger.stl"/>
-      </geometry>
-    </collision>
-  </link>
-  <!-- Gripper: Left finger (mimic) -->
-  <link name="left_palm_left_finger_link">
-    <inertial>
-      <origin xyz="-0.017 0.050 0" rpy="0 0 0"/>
-      <mass value="0.029"/>
-      <inertia ixx="0.000106" ixy="-1.28e-05" ixz="0" iyy="4.91e-05" iyz="0" izz="8.9e-05"/>
-    </inertial>
-    <visual>
-      <origin xyz="0 0 0" rpy="0 0 0"/>
-      <geometry>
-        <mesh filename="package://arm_description/meshes/visual/left_palm_left_finger.stl"/>
-      </geometry>
-      <material name="grey"/>
-    </visual>
-    <collision>
-      <origin xyz="0 0 0" rpy="0 0 0"/>
-      <geometry>
-        <mesh filename="package://arm_description/meshes/visual/left_palm_left_finger.stl"/>
-      </geometry>
-    </collision>
-  </link>
 </robot>

File: src/robot_description/arm_description/urdf/macros/ros2_control.xacro (robot description, xacro)
@@ -1,5 +1,5 @@
 <?xml version="1.0"?>
 <robot xmlns:xacro="http://ros.org/wiki/xacro">
-    <xacro:macro name="arm_ros2_control">
+    <xacro:macro name="arm_ros2_control" params="hand_type:=simple_gripper">
         <ros2_control name="ArmSystem" type="system">
             <hardware>
@@ -43,18 +43,102 @@
                 <state_interface name="effort"/>
             </joint>
-            <!-- Gripper: right finger (controlled) -->
-            <joint name="left_palm_right_finger">
-                <command_interface name="position"/>
-                <state_interface name="position"/>
-                <state_interface name="velocity"/>
-                <state_interface name="effort"/>
-            </joint>
-            <!-- Gripper: left finger (mimic - state only) -->
-            <joint name="left_palm_left_finger">
-                <state_interface name="position"/>
-                <state_interface name="velocity"/>
-                <state_interface name="effort"/>
-            </joint>
         </ros2_control>
+        <!-- Simple gripper ros2_control joints -->
+        <xacro:if value="${hand_type == 'simple_gripper'}">
+            <ros2_control name="GripperSystem" type="system">
+                <hardware>
+                    <plugin>gz_ros2_control/GazeboSimSystem</plugin>
+                </hardware>
+                <!-- Gripper: right finger (controlled) -->
+                <joint name="left_palm_right_finger">
+                    <command_interface name="position"/>
+                    <state_interface name="position"/>
+                    <state_interface name="velocity"/>
+                    <state_interface name="effort"/>
+                </joint>
+                <!-- Gripper: left finger (mimic - state only) -->
+                <joint name="left_palm_left_finger">
+                    <state_interface name="position"/>
+                    <state_interface name="velocity"/>
+                    <state_interface name="effort"/>
+                </joint>
+            </ros2_control>
+        </xacro:if>
+        <!-- Inspire hand ros2_control joints -->
+        <xacro:if value="${hand_type == 'inspire_hand'}">
+            <ros2_control name="HandSystem" type="system">
+                <hardware>
+                    <plugin>gz_ros2_control/GazeboSimSystem</plugin>
+                </hardware>
+                <!-- 6 actuated joints (command + state) -->
+                <joint name="thumb_proximal_yaw_joint">
+                    <command_interface name="position"/>
+                    <state_interface name="position"/>
+                    <state_interface name="velocity"/>
+                    <state_interface name="effort"/>
+                </joint>
+                <joint name="thumb_proximal_pitch_joint">
+                    <command_interface name="position"/>
+                    <state_interface name="position"/>
+                    <state_interface name="velocity"/>
+                    <state_interface name="effort"/>
+                </joint>
+                <joint name="index_proximal_joint">
+                    <command_interface name="position"/>
+                    <state_interface name="position"/>
+                    <state_interface name="velocity"/>
+                    <state_interface name="effort"/>
+                </joint>
+                <joint name="middle_proximal_joint">
+                    <command_interface name="position"/>
+                    <state_interface name="position"/>
+                    <state_interface name="velocity"/>
+                    <state_interface name="effort"/>
+                </joint>
+                <joint name="ring_proximal_joint">
+                    <command_interface name="position"/>
+                    <state_interface name="position"/>
+                    <state_interface name="velocity"/>
+                    <state_interface name="effort"/>
+                </joint>
+                <joint name="pinky_proximal_joint">
+                    <command_interface name="position"/>
+                    <state_interface name="position"/>
+                    <state_interface name="velocity"/>
+                    <state_interface name="effort"/>
+                </joint>
+                <!-- 6 mimic joints (state only) -->
+                <joint name="thumb_intermediate_joint">
+                    <state_interface name="position"/>
+                    <state_interface name="velocity"/>
+                    <state_interface name="effort"/>
+                </joint>
+                <joint name="thumb_distal_joint">
+                    <state_interface name="position"/>
+                    <state_interface name="velocity"/>
+                    <state_interface name="effort"/>
+                </joint>
+                <joint name="index_intermediate_joint">
+                    <state_interface name="position"/>
+                    <state_interface name="velocity"/>
+                    <state_interface name="effort"/>
+                </joint>
+                <joint name="middle_intermediate_joint">
+                    <state_interface name="position"/>
+                    <state_interface name="velocity"/>
+                    <state_interface name="effort"/>
+                </joint>
+                <joint name="ring_intermediate_joint">
+                    <state_interface name="position"/>
+                    <state_interface name="velocity"/>
+                    <state_interface name="effort"/>
+                </joint>
+                <joint name="pinky_intermediate_joint">
+                    <state_interface name="position"/>
+                    <state_interface name="velocity"/>
+                    <state_interface name="effort"/>
+                </joint>
+            </ros2_control>
+        </xacro:if>
     </xacro:macro>
 </robot>
