Commit message: Fix: moveit reconfigure, elow_shaft: 16kg fix

File: src/robot_description/arm_description/urdf/links/arm_links.xacro (robot description, xacro)
@@ -466,5 +466,5 @@
     <inertial>
       <origin xyz="-0.514023065887935 0.0789116739531359 -0.294612657237542" rpy="0 0 0" />
-      <mass value="16.3859228521728" />
+      <mass value="0.00163859228521728" />
       <inertia ixx="4.16738712851798" ixy="0.924028167542474" ixz="-3.13052395465567" iyy="7.10700860084082" iyz="1.12422208671553" izz="3.92149057920971" />
     </inertial>
