Commit message: controller upadte

File: src/robot_description/humanoid_leg_description/urdf/macros/ros2_control_gazebo.xacro (robot description, xacro)
@@ -7,5 +7,5 @@
             </hardware>
             <!-- LEFT LEG JOINTS -->
-            <joint name="${prefix}left_hip_pitch">
+            <joint name="${prefix}dof_left_hip_pitch_04">
                 <command_interface name="position"/>
                 <command_interface name="velocity"/>
@@ -16,5 +16,5 @@
                 <state_interface name="effort"/>
             </joint>
-            <joint name="${prefix}left_hip_roll">
+            <joint name="${prefix}dof_left_hip_roll_03">
                 <command_interface name="position"/>
                 <command_interface name="velocity"/>
@@ -25,5 +25,5 @@
                 <state_interface name="effort"/>
             </joint>
-            <joint name="${prefix}left_hip_yaw">
+            <joint name="${prefix}dof_left_hip_yaw_03">
                 <command_interface name="position"/>
                 <command_interface name="velocity"/>
@@ -34,5 +34,5 @@
                 <state_interface name="effort"/>
             </joint>
-            <joint name="${prefix}left_knee">
+            <joint name="${prefix}dof_left_knee_04">
                 <command_interface name="position"/>
                 <command_interface name="velocity"/>
@@ -43,14 +43,5 @@
                 <state_interface name="effort"/>
             </joint>
-            <joint name="${prefix}left_ankle">
-                <command_interface name="position"/>
-                <command_interface name="velocity"/>
-                <state_interface name="position">
-                    <param name="initial_value">0.0</param>
-                </state_interface>
-                <state_interface name="velocity"/>
-                <state_interface name="effort"/>
-            </joint>
-            <joint name="${prefix}left_foot">
+            <joint name="${prefix}dof_left_ankle_02">
                 <command_interface name="position"/>
                 <command_interface name="velocity"/>
@@ -62,5 +53,5 @@
             </joint>
             <!-- RIGHT LEG JOINTS -->
-            <joint name="${prefix}right_hip_pitch">
+            <joint name="${prefix}dof_right_hip_pitch_04">
                 <command_interface name="position"/>
                 <command_interface name="velocity"/>
@@ -71,5 +62,5 @@
                 <state_interface name="effort"/>
             </joint>
-            <joint name="${prefix}right_hip_roll">
+            <joint name="${prefix}dof_right_hip_roll_03">
                 <command_interface name="position"/>
                 <command_interface name="velocity"/>
@@ -80,5 +71,5 @@
                 <state_interface name="effort"/>
             </joint>
-            <joint name="${prefix}right_hip_yaw">
+            <joint name="${prefix}dof_right_hip_yaw_03">
                 <command_interface name="position"/>
                 <command_interface name="velocity"/>
@@ -89,5 +80,5 @@
                 <state_interface name="effort"/>
             </joint>
-            <joint name="${prefix}right_knee">
+            <joint name="${prefix}dof_right_knee_04">
                 <command_interface name="position"/>
                 <command_interface name="velocity"/>
@@ -98,14 +89,5 @@
                 <state_interface name="effort"/>
             </joint>
-            <joint name="${prefix}right_ankle">
-                <command_interface name="position"/>
-                <command_interface name="velocity"/>
-                <state_interface name="position">
-                    <param name="initial_value">0.0</param>
-                </state_interface>
-                <state_interface name="velocity"/>
-                <state_interface name="effort"/>
-            </joint>
-            <joint name="${prefix}right_foot">
+            <joint name="${prefix}dof_right_ankle_02">
                 <command_interface name="position"/>
                 <command_interface name="velocity"/>

Commit message: update kbot 2

File: src/robot_description/humanoid_leg_description/urdf/macros/ros2_control_gazebo.xacro (robot description, xacro)
@@ -98,4 +98,96 @@
                 <state_interface name="effort"/>
             </joint>
+            <!-- LEFT ARM JOINTS -->
+            <joint name="${prefix}dof_left_shoulder_pitch_03">
+                <command_interface name="position"/>
+                <command_interface name="velocity"/>
+                <state_interface name="position">
+                    <param name="initial_value">0.0</param>
+                </state_interface>
+                <state_interface name="velocity"/>
+                <state_interface name="effort"/>
+            </joint>
+            <joint name="${prefix}dof_left_shoulder_roll_03">
+                <command_interface name="position"/>
+                <command_interface name="velocity"/>
+                <state_interface name="position">
+                    <param name="initial_value">0.0</param>
+                </state_interface>
+                <state_interface name="velocity"/>
+                <state_interface name="effort"/>
+            </joint>
+            <joint name="${prefix}dof_left_shoulder_yaw_02">
+                <command_interface name="position"/>
+                <command_interface name="velocity"/>
+                <state_interface name="position">
+                    <param name="initial_value">0.0</param>
+                </state_interface>
+                <state_interface name="velocity"/>
+                <state_interface name="effort"/>
+            </joint>
+            <joint name="${prefix}dof_left_elbow_02">
+                <command_interface name="position"/>
+                <command_interface name="velocity"/>
+                <state_interface name="position">
+                    <param name="initial_value">0.0</param>
+                </state_interface>
+                <state_interface name="velocity"/>
+                <state_interface name="effort"/>
+            </joint>
+            <joint name="${prefix}dof_left_wrist_00">
+                <command_interface name="position"/>
+                <command_interface name="velocity"/>
+                <state_interface name="position">
+                    <param name="initial_value">0.0</param>
+                </state_interface>
+                <state_interface name="velocity"/>
+                <state_interface name="effort"/>
+            </joint>
+            <!-- RIGHT ARM JOINTS -->
+            <joint name="${prefix}dof_right_shoulder_pitch_03">
+                <command_interface name="position"/>
+                <command_interface name="velocity"/>
+                <state_interface name="position">
+                    <param name="initial_value">0.0</param>
+                </state_interface>
+                <state_interface name="velocity"/>
+                <state_interface name="effort"/>
+            </joint>
+            <joint name="${prefix}dof_right_shoulder_roll_03">
+                <command_interface name="position"/>
+                <command_interface name="velocity"/>
+                <state_interface name="position">
+                    <param name="initial_value">0.0</param>
+                </state_interface>
+                <state_interface name="velocity"/>
+                <state_interface name="effort"/>
+            </joint>
+            <joint name="${prefix}dof_right_shoulder_yaw_02">
+                <command_interface name="position"/>
+                <command_interface name="velocity"/>
+                <state_interface name="position">
+                    <param name="initial_value">0.0</param>
+                </state_interface>
+                <state_interface name="velocity"/>
+                <state_interface name="effort"/>
+            </joint>
+            <joint name="${prefix}dof_right_elbow_02">
+                <command_interface name="position"/>
+                <command_interface name="velocity"/>
+                <state_interface name="position">
+                    <param name="initial_value">0.0</param>
+                </state_interface>
+                <state_interface name="velocity"/>
+                <state_interface name="effort"/>
+            </joint>
+            <joint name="${prefix}dof_right_wrist_00">
+                <command_interface name="position"/>
+                <command_interface name="velocity"/>
+                <state_interface name="position">
+                    <param name="initial_value">0.0</param>
+                </state_interface>
+                <state_interface name="velocity"/>
+                <state_interface name="effort"/>
+            </joint>
         </ros2_control>
     </xacro:macro>
