Commit message: Tweak Inspire hand joint limits for MoveIt start stat

File: src/robot_description/arm_description/urdf/hands/inspire_hand_left.xacro (robot description, xacro)
@@ -100,5 +100,5 @@
       <child link="thumb_proximal_base"/>
       <axis xyz="0 0 1"/>
-      <limit lower="0" upper="1.308" effort="1" velocity="0.5"/>
+      <limit lower="0" upper="1.31" effort="1" velocity="0.5"/>
     </joint>
     <link name="thumb_proximal">
