Commit message: Create Gripper controller Fixes #86

File: src/robot_description/arm_description/urdf/joints/arm_joints.xacro (robot description, xacro)
@@ -133,4 +133,5 @@
         <axis xyz="0 0 0" />
     </joint>
+    <!-- Gripper finger joints: Main controller joint (right finger) -->
     <joint name="left_palm_right_finger" type="prismatic">
         <origin xyz="0 0 0" rpy="0 0 0" />
@@ -138,7 +139,9 @@
         <child link="left_palm_right_finger_link" />
         <axis xyz="-1 0 0" />
-        <limit lower="-0.033" upper="0.00026" effort="0" velocity="0" />
+        <limit lower="-0.033" upper="0.00026" effort="10" velocity="0.05" />
         <safety_controller soft_upper_limit="0.00026" soft_lower_limit="-0.033" k_velocity="0" />
+        <dynamics damping="0.1" friction="0.1" />
     </joint>
+    <!-- Left finger mimics right finger (symmetric movement) -->
     <joint name="left_palm_left_finger" type="prismatic">
         <origin xyz="0 0 0" rpy="0 0 0" />
@@ -146,6 +149,8 @@
         <child link="left_palm_left_finger_link" />
         <axis xyz="-1 0 0" />
-        <limit lower="-0.0041" upper="0.033" effort="0" velocity="0" />
+        <limit lower="-0.0041" upper="0.033" effort="10" velocity="0.05" />
         <safety_controller soft_upper_limit="0.033" soft_lower_limit="-0.0041" k_velocity="0" />
+        <mimic joint="left_palm_right_finger" multiplier="-1.0" offset="0" />
+        <dynamics damping="0.1" friction="0.1" />
     </joint>
 </robot>

File: src/robot_description/arm_description/urdf/macros/ros2_control.xacro (robot description, xacro)
@@ -36,4 +36,5 @@
                 <state_interface name="velocity" />
             </joint>
+            <!-- Gripper: Only control the main joint, left finger mimics automatically -->
             <joint name="left_palm_right_finger">
                 <command_interface name="position" />
@@ -41,9 +42,5 @@
                 <state_interface name="velocity" />
             </joint>
-            <joint name="left_palm_left_finger">
-                <command_interface name="position" />
-                <state_interface name="position" />
-                <state_interface name="velocity" />
-            </joint>
+            <!-- left_palm_left_finger is a mimic joint, controlled automatically by Gazebo -->
         </ros2_control>
     </xacro:macro>

Commit message: review Fixes #87

File: src/robot_description/arm_description/urdf/joints/arm_joints.xacro (robot description, xacro)
@@ -133,5 +133,5 @@
         <axis xyz="0 0 0" />
     </joint>
-    <!-- Gripper finger joints: Main controller joint (right finger) -->
+    <!-- Gripper finger joints: Right finger (independent control) -->
     <joint name="left_palm_right_finger" type="prismatic">
         <origin xyz="0 0 0" rpy="0 0 0" />
@@ -143,5 +143,5 @@
         <dynamics damping="0.1" friction="0.1" />
     </joint>
-    <!-- Left finger mimics right finger (symmetric movement) -->
+    <!-- Left finger (independent control) -->
     <joint name="left_palm_left_finger" type="prismatic">
         <origin xyz="0 0 0" rpy="0 0 0" />
@@ -151,5 +151,4 @@
         <limit lower="-0.0041" upper="0.033" effort="10" velocity="0.05" />
         <safety_controller soft_upper_limit="0.033" soft_lower_limit="-0.0041" k_velocity="0" />
-        <mimic joint="left_palm_right_finger" multiplier="-1.0" offset="0" />
         <dynamics damping="0.1" friction="0.1" />
     </joint>

File: src/robot_description/arm_description/urdf/macros/ros2_control.xacro (robot description, xacro)
@@ -36,5 +36,5 @@
                 <state_interface name="velocity" />
             </joint>
-            <!-- Gripper: Only control the main joint, left finger mimics automatically -->
+            <!-- Gripper: Independent control for both fingers -->
             <joint name="left_palm_right_finger">
                 <command_interface name="position" />
@@ -42,5 +42,9 @@
                 <state_interface name="velocity" />
             </joint>
-            <!-- left_palm_left_finger is a mimic joint, controlled automatically by Gazebo -->
+            <joint name="left_palm_left_finger">
+                <command_interface name="position" />
+                <state_interface name="position" />
+                <state_interface name="velocity" />
+            </joint>
         </ros2_control>
     </xacro:macro>

Commit message: use GripperActionController

File: src/robot_description/arm_description/urdf/joints/arm_joints.xacro (robot description, xacro)
@@ -143,5 +143,5 @@
         <dynamics damping="0.1" friction="0.1" />
     </joint>
-    <!-- Left finger (independent control) -->
+    <!-- Left finger mimics right finger (symmetric movement) -->
     <joint name="left_palm_left_finger" type="prismatic">
         <origin xyz="0 0 0" rpy="0 0 0" />
@@ -151,4 +151,5 @@
         <limit lower="-0.0041" upper="0.033" effort="10" velocity="0.05" />
         <safety_controller soft_upper_limit="0.033" soft_lower_limit="-0.0041" k_velocity="0" />
+        <mimic joint="left_palm_right_finger" multiplier="-1.0" offset="0" />
         <dynamics damping="0.1" friction="0.1" />
     </joint>

File: src/robot_description/arm_description/urdf/macros/ros2_control.xacro (robot description, xacro)
@@ -36,5 +36,5 @@
                 <state_interface name="velocity" />
             </joint>
-            <!-- Gripper: Independent control for both fingers -->
+            <!-- Gripper: Only control main joint, left finger mimics automatically -->
             <joint name="left_palm_right_finger">
                 <command_interface name="position" />
@@ -42,6 +42,6 @@
                 <state_interface name="velocity" />
             </joint>
+            <!-- left_palm_left_finger is a mimic joint - only state interfaces -->
             <joint name="left_palm_left_finger">
-                <command_interface name="position" />
                 <state_interface name="position" />
                 <state_interface name="velocity" />

Commit message: power calculator and joint limits effor correction

File: src/robot_description/arm_description/urdf/joints/arm_joints.xacro (robot description, xacro)
@@ -12,5 +12,5 @@
         <child link="left_shoulder_pitch_rs04_flange" />
         <axis xyz="1 0 0" />
-        <limit lower="-3.14" upper="3.14" effort="120" velocity="3" />
+        <limit lower="-3.14" upper="3.14" effort="40.0" velocity="17.49" />
         <safety_controller soft_upper_limit="3.14" soft_lower_limit="-3.14" k_velocity="0" />
     </joint>
@@ -32,5 +32,5 @@
         <child link="left_shoulder_roll_rs04_actuator" />
         <axis xyz="0 -1 0" />
-        <limit lower="-3.5" upper="0.6" effort="120" velocity="3" />
+        <limit lower="-3.5" upper="0.6" effort="40.0" velocity="17.49" />
         <safety_controller soft_upper_limit="3.14" soft_lower_limit="-3.14" k_velocity="0" />
     </joint>
@@ -52,5 +52,5 @@
         <child link="left_shoulder_yaw_rs03_flange" />
         <axis xyz="0 0 1" />
-        <limit lower="-3.14" upper="3.14" effort="60" velocity="1.6" />
+        <limit lower="-3.14" upper="3.14" effort="20.0" velocity="18.85" />
         <safety_controller soft_upper_limit="3.14" soft_lower_limit="-3.14" k_velocity="0" />
     </joint>
@@ -78,5 +78,5 @@
         <child link="left_elbow_rs03_flange" />
         <axis xyz="-1 0 0" />
-        <limit lower="-1.3" upper="1.9" effort="60" velocity="1.6" />
+        <limit lower="-1.3" upper="1.9" effort="20.0" velocity="18.85" />
         <safety_controller soft_upper_limit="3.14" soft_lower_limit="-3.14" k_velocity="0" />
     </joint>
@@ -98,5 +98,5 @@
         <child link="left_wrist_rs02_flange" />
         <axis xyz="0 1 0" />
-        <limit lower="-3.14" upper="3.14" effort="17" velocity="0.8" />
+        <limit lower="-3.14" upper="3.14" effort="6.0" velocity="37.70" />
         <safety_controller soft_upper_limit="3.14" soft_lower_limit="-3.14" k_velocity="0" />
     </joint>
@@ -118,5 +118,5 @@
         <child link="left_hand_rs02_flange" />
         <axis xyz="1 0 0" />
-        <limit lower="-1.5" upper="1.7" effort="17" velocity="0.8" />
+        <limit lower="-1.5" upper="1.7" effort="6.0" velocity="37.70" />
         <safety_controller soft_upper_limit="1.7" soft_lower_limit="-1.5" k_velocity="0" />
     </joint>

Commit message: Refactor MTCPickPlaceCylinder for improved object configuration and planning scene setup
- Introduced ObjectConfig struct to encapsulate object parameters (id, radius, height, pick and place positions).
- Added loadObjectConfig method to load parameters from the node.
- Updated setupPlanningScene to use loaded object configuration and conditionally spawn objects.
- Enhanced doTask method to return a boolean indicating success or failure.
- Adjusted task creation to utilize object configuration for grasping and placing.
- Modified arm joint definitions in URDF to correct orientation and limits.
- Adjusted visual and collision origins in arm links URDF for better alignment.
- Added YOLOv8 model file for object detection capabilities.

File: src/robot_description/arm_description/urdf/joints/arm_joints.xacro (robot description, xacro)
@@ -2,5 +2,5 @@
 <robot xmlns:xacro="http://www.ros.org/wiki/xacro">
     <joint name="left_shoulder_pitch_rs04_actuator_fixture_link" type="fixed">
-        <origin xyz="-0.1079 0 1.425" rpy="-0.67594 0 3.1416" />
+        <origin xyz="-0.1079 0 1.425" rpy="0 0 3.1416" />
         <parent link="base_link" />
         <child link="left_shoulder_pitch_rs04_actuator" />
@@ -22,5 +22,5 @@
     </joint>
     <joint name="left_shoulder_roll_rs04_flange_fixture" type="fixed">
-        <origin xyz="0.11678 0.0487 -2.7056E-05" rpy="0 0 3.1416" />
+        <origin xyz="0.11678 0.0487 -2.7056E-05" rpy="0 -0.1 3.1416" />
         <parent link="left_shoulder_pitch" />
         <child link="left_shoulder_roll_rs04_flange" />
@@ -108,5 +108,5 @@
     </joint>
     <joint name="left_hand_rs02_fixture_link" type="fixed">
-        <origin xyz="0 0.0945 0" rpy="0.64485 0.44406 0" />
+        <origin xyz="0 0.0945 0" rpy="0 0.44406 0" />
         <parent link="left_wrist" />
         <child link="left_hand_rs02_actuator" />
@@ -122,5 +122,5 @@
     </joint>
     <joint name="left_hand_fixture" type="fixed">
-        <origin xyz="0 0 0" rpy="0 0 0" />
+        <origin xyz="0 0 0" rpy="0.785 0 0" />
         <parent link="left_hand_rs02_flange" />
         <child link="left_hand" />
@@ -139,6 +139,6 @@
         <child link="left_palm_right_finger_link" />
         <axis xyz="-1 0 0" />
-        <limit lower="-0.033" upper="0.00026" effort="10" velocity="0.05" />
-        <safety_controller soft_upper_limit="0.00026" soft_lower_limit="-0.033" k_velocity="0" />
+        <limit lower="-0.033" upper="0.0" effort="10" velocity="0.05" />
+        <safety_controller soft_upper_limit="0.0" soft_lower_limit="-0.033" k_velocity="0" />
         <dynamics damping="0.1" friction="0.1" />
     </joint>
@@ -149,6 +149,6 @@
         <child link="left_palm_left_finger_link" />
         <axis xyz="-1 0 0" />
-        <limit lower="-0.0041" upper="0.033" effort="10" velocity="0.05" />
-        <safety_controller soft_upper_limit="0.033" soft_lower_limit="-0.0041" k_velocity="0" />
+        <limit lower="0.0" upper="0.033" effort="10" velocity="0.05" />
+        <safety_controller soft_upper_limit="0.033" soft_lower_limit="0.0" k_velocity="0" />
         <mimic joint="left_palm_right_finger" multiplier="-1.0" offset="0" />
         <dynamics damping="0.1" friction="0.1" />

File: src/robot_description/arm_description/urdf/links/arm_links.xacro (robot description, xacro)
@@ -470,5 +470,5 @@
     </inertial>
     <visual>
-      <origin xyz="0 0 0" rpy="0 0 0" />
+      <origin xyz="-0.005 0 0" rpy="0 0 0" />
       <geometry>
         <mesh filename="package://arm_description/meshes/visual/left_palm_right_finger.STL" />
@@ -479,5 +479,5 @@
     </visual>
     <collision>
-      <origin xyz="0 0 0" rpy="0 0 0" />
+      <origin xyz="-0.005 0 0" rpy="0 0 0" />
       <geometry>
         <mesh filename="package://arm_description/meshes/visual/left_palm_right_finger.STL" />

Commit message: review 2

File: src/robot_description/arm_description/urdf/joints/arm_joints.xacro (robot description, xacro)
@@ -139,7 +139,7 @@
         <child link="left_palm_right_finger_link" />
         <axis xyz="-1 0 0" />
-        <limit lower="-0.033" upper="0.00026" effort="10" velocity="0.05" />
-        <safety_controller soft_upper_limit="0.00026" soft_lower_limit="-0.033" k_velocity="0" />
-        <dynamics damping="0.1" friction="0.1" />
+        <limit lower="-0.040" upper="0.0" effort="100" velocity="0.05" />
+        <safety_controller soft_upper_limit="0.0" soft_lower_limit="-0.040" k_velocity="0" />
+        <dynamics damping="0.1" friction="1.0" />
     </joint>
     <!-- Left finger mimics right finger (symmetric movement) -->
@@ -149,8 +149,8 @@
         <child link="left_palm_left_finger_link" />
         <axis xyz="-1 0 0" />
-        <limit lower="-0.0041" upper="0.033" effort="10" velocity="0.05" />
-        <safety_controller soft_upper_limit="0.033" soft_lower_limit="-0.0041" k_velocity="0" />
+        <limit lower="0.0" upper="0.040" effort="100" velocity="0.05" />
+        <safety_controller soft_upper_limit="0.040" soft_lower_limit="0.0" k_velocity="0" />
         <mimic joint="left_palm_right_finger" multiplier="-1.0" offset="0" />
-        <dynamics damping="0.1" friction="0.1" />
+        <dynamics damping="0.1" friction="1.0" />
     </joint>
 </robot>

Commit message: review arm position

File: src/robot_description/arm_description/urdf/joints/arm_joints.xacro (robot description, xacro)
@@ -139,6 +139,6 @@
         <child link="left_palm_right_finger_link" />
         <axis xyz="-1 0 0" />
-        <limit lower="-0.033" upper="0.0" effort="10" velocity="0.05" />
-        <safety_controller soft_upper_limit="0.0" soft_lower_limit="-0.033" k_velocity="0" />
+        <limit lower="-0.04" upper="0.0" effort="10" velocity="0.05" />
+        <safety_controller soft_upper_limit="0.0" soft_lower_limit="-0.04" k_velocity="0" />
         <dynamics damping="0.1" friction="0.1" />
     </joint>
@@ -149,6 +149,6 @@
         <child link="left_palm_left_finger_link" />
         <axis xyz="-1 0 0" />
-        <limit lower="0.0" upper="0.033" effort="10" velocity="0.05" />
-        <safety_controller soft_upper_limit="0.033" soft_lower_limit="0.0" k_velocity="0" />
+        <limit lower="0.0" upper="0.04" effort="10" velocity="0.05" />
+        <safety_controller soft_upper_limit="0.04" soft_lower_limit="0.0" k_velocity="0" />
         <mimic joint="left_palm_right_finger" multiplier="-1.0" offset="0" />
         <dynamics damping="0.1" friction="1.0" />

File: src/robot_description/arm_description/urdf/macros/ros2_control.xacro (robot description, xacro)
@@ -8,7 +8,5 @@
             <joint name="left_shoulder_pitch_rs04">
                 <command_interface name="position" />
-                <state_interface name="position">
-                    <param name="initial_value">0.6766</param>
-                </state_interface>
+                <state_interface name="position"/>
                 <state_interface name="velocity" />
                 <state_interface name="effort" />
@@ -16,7 +14,5 @@
             <joint name="left_shoulder_roll_rs04">
                 <command_interface name="position" />
-                <state_interface name="position">
-                    <param name="initial_value">0.0421</param>
-                </state_interface>
+                <state_interface name="position"/>
                 <state_interface name="velocity" />
                 <state_interface name="effort" />
@@ -24,7 +20,5 @@
             <joint name="left_shoulder_yaw_rs03">
                 <command_interface name="position" />
-                <state_interface name="position">
-                    <param name="initial_value">-0.4337</param>
-                </state_interface>
+                <state_interface name="position"/>
                 <state_interface name="velocity" />
                 <state_interface name="effort" />
@@ -32,7 +26,5 @@
             <joint name="left_elbow_rs03">
                 <command_interface name="position" />
-                <state_interface name="position">
-                    <param name="initial_value">0.2912</param>
-                </state_interface>
+                <state_interface name="position"/>
                 <state_interface name="velocity" />
                 <state_interface name="effort" />
@@ -40,7 +32,5 @@
             <joint name="left_wrist_rs02">
                 <command_interface name="position" />
-                <state_interface name="position">
-                    <param name="initial_value">-0.5378</param>
-                </state_interface>
+                <state_interface name="position"/>
                 <state_interface name="velocity" />
                 <state_interface name="effort" />
@@ -48,7 +38,5 @@
             <joint name="left_hand_rs02">
                 <command_interface name="position" />
-                <state_interface name="position">
-                    <param name="initial_value">0.1088</param>
-                </state_interface>
+                <state_interface name="position"/>
                 <state_interface name="velocity" />
                 <state_interface name="effort" />

Commit message: create joint controller Fixes #108

File: src/robot_description/arm_description/urdf/joints/arm_joints.xacro (robot description, xacro)
@@ -14,4 +14,5 @@
         <limit lower="-3.14" upper="3.14" effort="40.0" velocity="17.49" />
         <safety_controller soft_upper_limit="3.14" soft_lower_limit="-3.14" k_velocity="0" />
+        <dynamics damping="0.5" friction="2.0" />
     </joint>
     <joint name="left_shoulder_pitch_fixture" type="fixed">
@@ -34,4 +35,5 @@
         <limit lower="-3.5" upper="0.6" effort="40.0" velocity="17.49" />
         <safety_controller soft_upper_limit="3.14" soft_lower_limit="-3.14" k_velocity="0" />
+        <dynamics damping="0.5" friction="2.0" />
     </joint>
     <joint name="left_shoulde_roll_fixture" type="fixed">
@@ -54,4 +56,5 @@
         <limit lower="-3.14" upper="3.14" effort="20.0" velocity="18.85" />
         <safety_controller soft_upper_limit="3.14" soft_lower_limit="-3.14" k_velocity="0" />
+        <dynamics damping="0.4" friction="1.5" />
     </joint>
     <joint name="left_shoulder_yaw_flange_fixture" type="fixed">
@@ -80,4 +83,5 @@
         <limit lower="-1.3" upper="1.9" effort="20.0" velocity="18.85" />
         <safety_controller soft_upper_limit="3.14" soft_lower_limit="-3.14" k_velocity="0" />
+        <dynamics damping="0.4" friction="1.5" />
     </joint>
     <joint name="left_elbow_fixture" type="fixed">
@@ -100,4 +104,5 @@
         <limit lower="-3.14" upper="3.14" effort="6.0" velocity="37.70" />
         <safety_controller soft_upper_limit="3.14" soft_lower_limit="-3.14" k_velocity="0" />
+        <dynamics damping="0.25" friction="0.8" />
     </joint>
     <joint name="left_wrist_fixture" type="fixed">
@@ -120,4 +125,5 @@
         <limit lower="-1.5" upper="1.7" effort="6.0" velocity="37.70" />
         <safety_controller soft_upper_limit="1.7" soft_lower_limit="-1.5" k_velocity="0" />
+        <dynamics damping="0.25" friction="0.8" />
     </joint>
     <joint name="left_hand_fixture" type="fixed">

File: src/robot_description/arm_description/urdf/macros/ros2_control.xacro (robot description, xacro)
@@ -8,4 +8,5 @@
             <joint name="left_shoulder_pitch_rs04">
                 <command_interface name="position" />
+                <command_interface name="effort" />
                 <state_interface name="position"/>
                 <state_interface name="velocity" />
@@ -14,4 +15,5 @@
             <joint name="left_shoulder_roll_rs04">
                 <command_interface name="position" />
+                <command_interface name="effort" />
                 <state_interface name="position"/>
                 <state_interface name="velocity" />
@@ -20,4 +22,5 @@
             <joint name="left_shoulder_yaw_rs03">
                 <command_interface name="position" />
+                <command_interface name="effort" />
                 <state_interface name="position"/>
                 <state_interface name="velocity" />
@@ -26,4 +29,5 @@
             <joint name="left_elbow_rs03">
                 <command_interface name="position" />
+                <command_interface name="effort" />
                 <state_interface name="position"/>
                 <state_interface name="velocity" />
@@ -32,4 +36,5 @@
             <joint name="left_wrist_rs02">
                 <command_interface name="position" />
+                <command_interface name="effort" />
                 <state_interface name="position"/>
                 <state_interface name="velocity" />
@@ -38,4 +43,5 @@
             <joint name="left_hand_rs02">
                 <command_interface name="position" />
+                <command_interface name="effort" />
                 <state_interface name="position"/>
                 <state_interface name="velocity" />
