Commit message: upadate with new urdf

File: src/robot_description/arm_description/urdf/joints/arm_joints.xacro (robot description, xacro)
@@ -7,47 +7,47 @@
     <child link="base_link"/>
   </joint>
-  <!-- Joint 1: Shoulder pitch (on table surface) -->
+  <!-- Joint 1: Shoulder pitch (from table to shoulder) -->
   <joint name="shoulder_pitch_joint" type="revolute">
-    <origin xyz="0.0498579 0.00126819 6.80296e-06" rpy="1.5708 1.59595e-15 1.5708"/>
+    <origin xyz="-0.100142 0.00126819 0.000179533" rpy="1.5708 0 1.5708"/>
     <parent link="base_link"/>
     <child link="shoulder_link"/>
     <axis xyz="0 0 1"/>
-    <limit lower="-1.5708" upper="3.14159" velocity="16.0" effort="20.0"/>
+    <limit lower="-1.5708" upper="3.14159" velocity="10.0" effort="10.0"/>
     <dynamics damping="0.5" friction="0.1"/>
   </joint>
   <!-- Joint 2: Shoulder roll -->
   <joint name="shoulder_roll_joint" type="revolute">
-    <origin xyz="0.029 1.02101e-17 -0.078" rpy="-1.5708 -9.59268e-17 1.5708"/>
+    <origin xyz="0.041 0 -0.078" rpy="-3.14159 -1.5708 0"/>
     <parent link="shoulder_link"/>
     <child link="upper_arm_link"/>
     <axis xyz="0 0 1"/>
-    <limit lower="-3.14159" upper="0.112" velocity="16.0" effort="20.0"/>
+    <limit lower="0" upper="3.14159" velocity="10.0" effort="10.0"/>
     <dynamics damping="0.5" friction="0.1"/>
   </joint>
   <!-- Joint 3: Shoulder yaw -->
   <joint name="shoulder_yaw_joint" type="revolute">
-    <origin xyz="-0.157 -1.83881e-16 0.029" rpy="-1.5708 0.000395729 -1.5708"/>
+    <origin xyz="0 0.175 -0.041" rpy="1.5708 -0.000395729 0"/>
     <parent link="upper_arm_link"/>
     <child link="elbow_link"/>
     <axis xyz="0 0 1"/>
-    <limit lower="-1.57119" upper="1.5704" velocity="16.0" effort="20.0"/>
+    <limit lower="-1.57119" upper="1.5704" velocity="10.0" effort="10.0"/>
     <dynamics damping="0.5" friction="0.1"/>
   </joint>
   <!-- Joint 4: Elbow pitch -->
   <joint name="elbow_pitch_joint" type="revolute">
-    <origin xyz="-0.023 4.35849e-17 -0.083" rpy="1.5708 -7.42674e-05 1.5708"/>
+    <origin xyz="-0.035 0 -0.065" rpy="-1.5708 0 1.5708"/>
     <parent link="elbow_link"/>
     <child link="upper_forearm_link"/>
     <axis xyz="0 0 1"/>
-    <limit lower="-1.57087" upper="1.57072" velocity="16.0" effort="10.0"/>
+    <limit lower="-1.5708" upper="1.5708" velocity="10.0" effort="10.0"/>
     <dynamics damping="0.5" friction="0.1"/>
   </joint>
   <!-- Joint 5: Elbow yaw -->
   <joint name="elbow_yaw_joint" type="revolute">
-    <origin xyz="7.37257e-17 -0.151 0.023" rpy="-1.5708 -1.5708 0"/>
+    <origin xyz="0 0.168 -0.035" rpy="1.5708 1.5708 0"/>
     <parent link="upper_forearm_link"/>
     <child link="end_effector_link"/>
     <axis xyz="0 0 1"/>
-    <limit lower="-1.5708" upper="1.5708" velocity="16.0" effort="10.0"/>
+    <limit lower="-1.5708" upper="1.5708" velocity="10.0" effort="10.0"/>
     <dynamics damping="0.5" friction="0.1"/>
   </joint>

File: src/robot_description/arm_description/urdf/links/arm_links.xacro (robot description, xacro)
@@ -1,104 +1,103 @@
 <?xml version="1.0"?>
 <robot xmlns:xacro="http://www.ros.org/wiki/xacro">
-  <!-- Base link (table/stand with menghina and stator) -->
+  <!-- Base link (table with torso_limiter, menghina, spacer, rotor, stator) -->
   <link name="base_link">
     <inertial>
-      <origin xyz="0.15231 0.00126822 -0.0733771" rpy="0 0 0"/>
-      <mass value="12.7824"/>
-      <inertia ixx="0.319682" ixy="2.7236e-08" ixz="0.0107613" iyy="0.0695316" iyz="1.98209e-07" izz="0.343485"/>
-    </inertial>
-    <!-- Table -->
-    <visual>
-      <origin xyz="0.171858 0.00126819 -0.0923205" rpy="-3.14159 2.84025e-16 -1.25251e-16"/>
+      <origin xyz="0.12034 0.00123257 -0.131533" rpy="0 0 0"/>
+      <mass value="12.8024"/>
+      <inertia ixx="0.726842" ixy="-8.82389e-05" ixz="0.080114" iyy="0.717447" iyz="8.76443e-05" izz="0.70335"/>
+    </inertial>
+    <!-- Part torso_limiter -->
+    <visual>
+      <origin xyz="-0.0767119 -0.0215341 0.0674325" rpy="0 0 0"/>
+      <geometry>
+        <mesh filename="package://arm_description/meshes/visual/torso_limiter.stl"/>
+      </geometry>
+      <material name="yellow">
+        <color rgba="1 0.756863 0.054902 1"/>
+      </material>
+    </visual>
+    <collision>
+      <origin xyz="-0.0767119 -0.0215341 0.0674325" rpy="0 0 0"/>
+      <geometry>
+        <mesh filename="package://arm_description/meshes/visual/torso_limiter.stl"/>
+      </geometry>
+    </collision>
+    <!-- Part menghina_x6 -->
+    <visual>
+      <origin xyz="-0.0631421 0.00126819 0.000179533" rpy="0 0 1.5708"/>
+      <geometry>
+        <mesh filename="package://arm_description/meshes/visual/menghina_x6.stl"/>
+      </geometry>
+      <material name="blue">
+        <color rgba="0.32549 0.529412 0.752941 1"/>
+      </material>
+    </visual>
+    <collision>
+      <origin xyz="-0.0631421 0.00126819 0.000179533" rpy="0 0 1.5708"/>
+      <geometry>
+        <mesh filename="package://arm_description/meshes/visual/menghina_x6.stl"/>
+      </geometry>
+    </collision>
+    <!-- Part spacer_x6_menghina_m4x60 -->
+    <visual>
+      <origin xyz="-0.0331421 0.00126819 0.000179533" rpy="3.14159 0 1.5708"/>
+      <geometry>
+        <mesh filename="package://arm_description/meshes/visual/spacer_x6_menghina_m4x60.stl"/>
+      </geometry>
+      <material name="purple">
+        <color rgba="0.596078 0.121569 0.67451 1"/>
+      </material>
+    </visual>
+    <collision>
+      <origin xyz="-0.0331421 0.00126819 0.000179533" rpy="3.14159 0 1.5708"/>
+      <geometry>
+        <mesh filename="package://arm_description/meshes/visual/spacer_x6_menghina_m4x60.stl"/>
+      </geometry>
+    </collision>
+    <!-- Part table -->
+    <visual>
+      <origin xyz="0.171858 0.00126819 -0.0923205" rpy="-3.14159 0 0"/>
       <geometry>
         <mesh filename="package://arm_description/meshes/visual/table.stl"/>
       </geometry>
-      <material name="blue"/>
-    </visual>
-    <collision>
-      <origin xyz="0.171858 0.00126819 -0.0923205" rpy="-3.14159 2.84025e-16 -1.25251e-16"/>
+      <material name="light_blue">
+        <color rgba="0.615686 0.811765 0.929412 1"/>
+      </material>
+    </visual>
+    <collision>
+      <origin xyz="0.171858 0.00126819 -0.0923205" rpy="-3.14159 0 0"/>
       <geometry>
         <mesh filename="package://arm_description/meshes/visual/table.stl"/>
       </geometry>
     </collision>
-    <!-- Table legs (2 legs) -->
-    <visual>
-      <origin xyz="0.08 0.17 -0.49" rpy="0 0 0"/>
-      <geometry>
-        <cylinder radius="0.025" length="0.75"/>
-      </geometry>
-      <material name="dark_blue"/>
-    </visual>
-    <collision>
-      <origin xyz="0.08 0.17 -0.49" rpy="0 0 0"/>
-      <geometry>
-        <cylinder radius="0.025" length="0.75"/>
-      </geometry>
-    </collision>
-    <visual>
-      <origin xyz="0.08 -0.17 -0.49" rpy="0 0 0"/>
-      <geometry>
-        <cylinder radius="0.025" length="0.75"/>
-      </geometry>
-      <material name="dark_blue"/>
-    </visual>
-    <collision>
-      <origin xyz="0.08 -0.17 -0.49" rpy="0 0 0"/>
-      <geometry>
-        <cylinder radius="0.025" length="0.75"/>
-      </geometry>
-    </collision>
-    <!-- Menghina mount (on table surface) -->
-    <visual>
-      <origin xyz="0.0868579 0.00126819 6.80296e-06" rpy="0 0 1.5708"/>
-      <geometry>
-        <mesh filename="package://arm_description/meshes/visual/menghina_x6.stl"/>
-      </geometry>
-      <material name="dark_blue"/>
-    </visual>
-    <collision>
-      <origin xyz="0.0868579 0.00126819 6.80296e-06" rpy="0 0 1.5708"/>
-      <geometry>
-        <mesh filename="package://arm_description/meshes/visual/menghina_x6.stl"/>
-      </geometry>
-    </collision>
-    <!-- Spacer between menghina and stator -->
-    <visual>
-      <origin xyz="0.00685786 0.00126819 6.80296e-06" rpy="1.5708 -1.5708 0"/>
-      <geometry>
-        <mesh filename="package://arm_description/meshes/visual/spacer_x6_menghina_m4x60.stl"/>
-      </geometry>
-      <material name="purple"/>
-    </visual>
-    <collision>
-      <origin xyz="0.00685786 0.00126819 6.80296e-06" rpy="1.5708 -1.5708 0"/>
-      <geometry>
-        <mesh filename="package://arm_description/meshes/visual/spacer_x6_menghina_m4x60.stl"/>
-      </geometry>
-    </collision>
-    <!-- Rotor X6 (base) -->
-    <visual>
-      <origin xyz="0.141358 0.00126819 6.80296e-06" rpy="0 -1.5708 0"/>
-      <geometry>
-        <mesh filename="package://arm_description/meshes/visual/rotor_x6_p20_60.stl"/>
-      </geometry>
-      <material name="orange"/>
-    </visual>
-    <collision>
-      <origin xyz="0.141358 0.00126819 6.80296e-06" rpy="0 -1.5708 0"/>
-      <geometry>
-        <mesh filename="package://arm_description/meshes/visual/rotor_x6_p20_60.stl"/>
-      </geometry>
-    </collision>
-    <!-- Stator X6 (on table surface) -->
-    <visual>
-      <origin xyz="0.141358 0.00126819 6.80296e-06" rpy="0 -1.5708 0"/>
-      <geometry>
-        <mesh filename="package://arm_description/meshes/visual/stator_x6_p20_60.stl"/>
-      </geometry>
-      <material name="gold"/>
-    </visual>
-    <collision>
-      <origin xyz="0.141358 0.00126819 6.80296e-06" rpy="0 -1.5708 0"/>
+    <!-- Part rotor_x6_p20_60 -->
+    <visual>
+      <origin xyz="-0.00864214 0.00126819 0.000179533" rpy="0 -1.5708 0"/>
+      <geometry>
+        <mesh filename="package://arm_description/meshes/visual/rotor_x6_p20_60.stl"/>
+      </geometry>
+      <material name="gold">
+        <color rgba="0.65098 0.486275 0.0196078 1"/>
+      </material>
+    </visual>
+    <collision>
+      <origin xyz="-0.00864214 0.00126819 0.000179533" rpy="0 -1.5708 0"/>
+      <geometry>
+        <mesh filename="package://arm_description/meshes/visual/rotor_x6_p20_60.stl"/>
+      </geometry>
+    </collision>
+    <!-- Part stator_x6_p20_60 -->
+    <visual>
+      <origin xyz="-0.00864214 0.00126819 0.000179533" rpy="0 -1.5708 0"/>
+      <geometry>
+        <mesh filename="package://arm_description/meshes/visual/stator_x6_p20_60.stl"/>
+      </geometry>
+      <material name="cream">
+        <color rgba="0.960784 0.835294 0.470588 1"/>
+      </material>
+    </visual>
+    <collision>
+      <origin xyz="-0.00864214 0.00126819 0.000179533" rpy="0 -1.5708 0"/>
       <geometry>
         <mesh filename="package://arm_description/meshes/visual/stator_x6_p20_60.stl"/>
@@ -109,9 +108,37 @@
   <link name="shoulder_link">
     <inertial>
-      <origin xyz="-0.00509657 -9.94177e-07 -0.0751786" rpy="0 0 0"/>
-      <mass value="2.97837"/>
-      <inertia ixx="0.00348255" ixy="-3.74291e-08" ixz="2.44885e-05" iyy="0.00306396" iyz="-6.6893e-08" izz="0.00281696"/>
-    </inertial>
-    <!-- Rotor X6 -->
+      <origin xyz="-0.00526655 -5.01444e-05 -0.0747997" rpy="0 0 0"/>
+      <mass value="2.99837"/>
+      <inertia ixx="0.00360636" ixy="-4.79289e-06" ixz="5.35805e-05" iyy="0.00316519" iyz="1.005e-05" izz="0.0029116"/>
+    </inertial>
+    <!-- Part shoulder_limiter -->
+    <visual>
+      <origin xyz="-0.0305797 -0.00737046 -0.0183842" rpy="-1.5708 -1.5708 0"/>
+      <geometry>
+        <mesh filename="package://arm_description/meshes/visual/shoulder_limiter.stl"/>
+      </geometry>
+      <material name="yellow"/>
+    </visual>
+    <collision>
+      <origin xyz="-0.0305797 -0.00737046 -0.0183842" rpy="-1.5708 -1.5708 0"/>
+      <geometry>
+        <mesh filename="package://arm_description/meshes/visual/shoulder_limiter.stl"/>
+      </geometry>
+    </collision>
+    <!-- Part l_shoulder -->
+    <visual>
+      <origin xyz="-0.00130076 -6.96521e-06 -0.0582746" rpy="-1.5708 -1.5708 0"/>
+      <geometry>
+        <mesh filename="package://arm_description/meshes/visual/l_shoulder.stl"/>
+      </geometry>
+      <material name="light_blue"/>
+    </visual>
+    <collision>
+      <origin xyz="-0.00130076 -6.96521e-06 -0.0582746" rpy="-1.5708 -1.5708 0"/>
+      <geometry>
+        <mesh filename="package://arm_description/meshes/visual/l_shoulder.stl"/>
+      </geometry>
+    </collision>
+    <!-- Part rotor_x6_p20_60_2 -->
     <visual>
       <origin xyz="-0.0385 0 -0.078" rpy="-3.14159 -1.5708 0"/>
@@ -119,5 +146,5 @@
         <mesh filename="package://arm_description/meshes/visual/rotor_x6_p20_60.stl"/>
       </geometry>
-      <material name="orange"/>
+      <material name="gold"/>
     </visual>
     <collision>
@@ -127,19 +154,5 @@
       </geometry>
     </collision>
-    <!-- L Shoulder -->
-    <visual>
-      <origin xyz="-0.00130076 -6.96521e-06 -0.0582746" rpy="-1.5708 -1.5708 0"/>
-      <geometry>
-        <mesh filename="package://arm_description/meshes/visual/l_shoulder.stl"/>
-      </geometry>
-      <material name="blue"/>
-    </visual>
-    <collision>
-      <origin xyz="-0.00130076 -6.96521e-06 -0.0582746" rpy="-1.5708 -1.5708 0"/>
-      <geometry>
-        <mesh filename="package://arm_description/meshes/visual/l_shoulder.stl"/>
-      </geometry>
-    </collision>
-    <!-- Stator X6 for next joint -->
+    <!-- Part stator_x6_p20_60_2 -->
     <visual>
       <origin xyz="-0.0385 0 -0.078" rpy="-3.14159 -1.5708 0"/>
@@ -147,5 +160,5 @@
         <mesh filename="package://arm_description/meshes/visual/stator_x6_p20_60.stl"/>
       </geometry>
-      <material name="gold"/>
+      <material name="cream"/>
     </visual>
     <collision>
@@ -159,46 +172,64 @@
   <link name="upper_arm_link">
     <inertial>
-      <origin xyz="-0.112126 -2.19492e-08 0.0230405" rpy="0 0 0"/>
-      <mass value="1.54329"/>
-      <inertia ixx="0.00133766" ixy="6.04381e-10" ixz="0.000537695" iyy="0.00254134" iyz="7.1395e-08" izz="0.00234132"/>
-    </inertial>
-    <!-- Rotor X6 -->
-    <visual>
-      <origin xyz="0.0445 0 -0.083" rpy="-3.14159 1.5708 0"/>
-      <geometry>
-        <mesh filename="package://arm_description/meshes/visual/rotor_x6_p20_60.stl"/>
-      </geometry>
-      <material name="orange"/>
-    </visual>
-    <collision>
-      <origin xyz="0.0445 0 -0.083" rpy="-3.14159 1.5708 0"/>
-      <geometry>
-        <mesh filename="package://arm_description/meshes/visual/rotor_x6_p20_60.stl"/>
-      </geometry>
-    </collision>
-    <!-- L Upper Arm -->
-    <visual>
-      <origin xyz="-0.0912885 -6.25469e-08 0.00867029" rpy="-1.5708 0 -1.5708"/>
+      <origin xyz="0.000527863 0.112716 -0.0353918" rpy="0 0 0"/>
+      <mass value="1.56329"/>
+      <inertia ixx="0.00261957" ixy="-3.7804e-05" ixz="1.27536e-05" iyy="0.00141519" iyz="0.000562166" izz="0.00242582"/>
+    </inertial>
+    <!-- Part arm_limiter -->
+    <visual>
+      <origin xyz="0.0412588 0.158216 -0.0625065" rpy="1.5708 0 0"/>
+      <geometry>
+        <mesh filename="package://arm_description/meshes/visual/arm_limiter.stl"/>
+      </geometry>
+      <material name="yellow"/>
+    </visual>
+    <collision>
+      <origin xyz="0.0412588 0.158216 -0.0625065" rpy="1.5708 0 0"/>
+      <geometry>
+        <mesh filename="package://arm_description/meshes/visual/arm_limiter.stl"/>
+      </geometry>
+    </collision>
+    <!-- Part l_upper_arm -->
+    <visual>
+      <origin xyz="0 0.0912885 -0.0206703" rpy="1.5708 0 0"/>
       <geometry>
         <mesh filename="package://arm_description/meshes/visual/l_upper_arm.stl"/>
       </geometry>
-      <material name="blue"/>
-    </visual>
-    <collision>
-      <origin xyz="-0.0912885 -6.25469e-08 0.00867029" rpy="-1.5708 0 -1.5708"/>
+      <material name="light_blue"/>
+    </visual>
+    <collision>
+      <origin xyz="0 0.0912885 -0.0206703" rpy="1.5708 0 0"/>
       <geometry>
         <mesh filename="package://arm_description/meshes/visual/l_upper_arm.stl"/>
       </geometry>
     </collision>
-    <!-- Stator X4 for next joint -->
-    <visual>
-      <origin xyz="-0.091 0 0.029" rpy="1.5708 0 -1.5708"/>
+    <!-- Part rotor_x4_p36_36 -->
+    <visual>
+      <origin xyz="0 0.091 -0.041" rpy="-1.5708 0 0"/>
+      <geometry>
+        <mesh filename="package://arm_description/meshes/visual/rotor_x4_p36_36.stl"/>
+      </geometry>
+      <material name="dark_purple">
+        <color rgba="0.380392 0.0470588 0.435294 1"/>
+      </material>
+    </visual>
+    <collision>
+      <origin xyz="0 0.091 -0.041" rpy="-1.5708 0 0"/>
+      <geometry>
+        <mesh filename="package://arm_description/meshes/visual/rotor_x4_p36_36.stl"/>
+      </geometry>
+    </collision>
+    <!-- Part stator_x4_p36_36 -->
+    <visual>
+      <origin xyz="0 0.091 -0.041" rpy="-1.5708 0 0"/>
       <geometry>
         <mesh filename="package://arm_description/meshes/visual/stator_x4_p36_36.stl"/>
       </geometry>
-      <material name="purple"/>
-    </visual>
-    <collision>
-      <origin xyz="-0.091 0 0.029" rpy="1.5708 0 -1.5708"/>
+      <material name="light_purple">
+        <color rgba="0.764706 0.545098 0.803922 1"/>
+      </material>
+    </visual>
+    <collision>
+      <origin xyz="0 0.091 -0.041" rpy="-1.5708 0 0"/>
       <geometry>
         <mesh filename="package://arm_description/meshes/visual/stator_x4_p36_36.stl"/>
@@ -209,46 +240,60 @@
   <link name="elbow_link">
     <inertial>
-      <origin xyz="0.0103789 1.30908e-06 -0.0814648" rpy="0 0 0"/>
-      <mass value="2.87437"/>
-      <inertia ixx="0.00300002" ixy="3.78723e-08" ixz="7.45868e-05" iyy="0.00280783" iyz="1.59723e-08" izz="0.00247115"/>
-    </inertial>
-    <!-- Rotor X4 -->
-    <visual>
-      <origin xyz="-0.091 0 0.029" rpy="1.5708 0 -1.5708"/>
-      <geometry>
-        <mesh filename="package://arm_description/meshes/visual/rotor_x4_p36_36.stl"/>
-      </geometry>
-      <material name="dark_purple"/>
-    </visual>
-    <collision>
-      <origin xyz="-0.091 0 0.029" rpy="1.5708 0 -1.5708"/>
-      <geometry>
-        <mesh filename="package://arm_description/meshes/visual/rotor_x4_p36_36.stl"/>
-      </geometry>
-    </collision>
-    <!-- L Elbow -->
-    <visual>
-      <origin xyz="-0.000331628 1.15447e-05 -0.0692953" rpy="0 0 0"/>
+      <origin xyz="0.0100547 -0.000241015 -0.0630889" rpy="0 0 0"/>
+      <mass value="2.89437"/>
+      <inertia ixx="0.00309417" ixy="-2.35227e-05" ixz="0.000125711" iyy="0.00292161" iyz="3.72513e-05" izz="0.00256028"/>
+    </inertial>
+    <!-- Part elbow_limiter -->
+    <visual>
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
Commit message: effort review

File: src/robot_description/arm_description/urdf/joints/arm_joints.xacro (robot description, xacro)
@@ -13,5 +13,5 @@
     <child link="shoulder_link"/>
     <axis xyz="0 0 1"/>
-    <limit lower="-1.5708" upper="3.14159" velocity="10.0" effort="10.0"/>
+    <limit lower="-1.5708" upper="3.14159" velocity="10.0" effort="40.0"/>
     <dynamics damping="0.5" friction="0.1"/>
   </joint>
@@ -22,5 +22,5 @@
     <child link="upper_arm_link"/>
     <axis xyz="0 0 1"/>
-    <limit lower="0" upper="3.14159" velocity="10.0" effort="10.0"/>
+    <limit lower="0" upper="3.14159" velocity="10.0" effort="40.0"/>
     <dynamics damping="0.5" friction="0.1"/>
   </joint>
@@ -31,5 +31,5 @@
     <child link="elbow_link"/>
     <axis xyz="0 0 1"/>
-    <limit lower="-1.57119" upper="1.5704" velocity="10.0" effort="10.0"/>
+    <limit lower="-1.57119" upper="1.5704" velocity="10.0" effort="40.0"/>
     <dynamics damping="0.5" friction="0.1"/>
   </joint>
@@ -40,5 +40,5 @@
     <child link="upper_forearm_link"/>
     <axis xyz="0 0 1"/>
-    <limit lower="-1.5708" upper="1.5708" velocity="10.0" effort="10.0"/>
+    <limit lower="-1.5708" upper="1.5708" velocity="10.0" effort="40.0"/>
     <dynamics damping="0.5" friction="0.1"/>
   </joint>
@@ -49,5 +49,5 @@
     <child link="end_effector_link"/>
     <axis xyz="0 0 1"/>
-    <limit lower="-1.5708" upper="1.5708" velocity="10.0" effort="10.0"/>
+    <limit lower="-1.5708" upper="1.5708" velocity="10.0" effort="40.0"/>
     <dynamics damping="0.5" friction="0.1"/>
   </joint>
