Commit message: update urdf

File: src/robot_description/arm_description/urdf/joints/arm_joints.xacro (robot description, xacro)
@@ -45,6 +45,15 @@
   <!-- Joint 5: Elbow yaw -->
   <joint name="elbow_yaw_joint" type="revolute">
-    <origin xyz="0 0.168 -0.035" rpy="1.5708 1.5708 0"/>
+    <origin xyz="0 0.163 -0.035" rpy="1.5708 1.5708 0"/>
     <parent link="upper_forearm_link"/>
+    <child link="lower_forearm_link"/>
+    <axis xyz="0 0 1"/>
+    <limit lower="-2.35619" upper="2.35619" velocity="10.0" effort="40.0"/>
+    <dynamics damping="0.5" friction="0.1"/>
+  </joint>
+  <!-- Joint 6: Wrist roll (NEW) -->
+  <joint name="wrist_roll_joint" type="revolute">
+    <origin xyz="0 0.03 -0.0615" rpy="-1.5708 0 0"/>
+    <parent link="lower_forearm_link"/>
     <child link="end_effector_link"/>
     <axis xyz="0 0 1"/>

File: src/robot_description/arm_description/urdf/links/arm_links.xacro (robot description, xacro)
@@ -105,5 +105,5 @@
     </collision>
   </link>
-  <!-- Link 1: Shoulder (pitch rotation) -->
+  <!-- Link 1: Shoulder -->
   <link name="shoulder_link">
     <inertial>
@@ -169,5 +169,5 @@
     </collision>
   </link>
-  <!-- Link 2: Upper arm (roll rotation) -->
+  <!-- Link 2: Upper arm -->
   <link name="upper_arm_link">
     <inertial>
@@ -237,5 +237,5 @@
     </collision>
   </link>
-  <!-- Link 3: Elbow (yaw rotation) -->
+  <!-- Link 3: Elbow -->
   <link name="elbow_link">
     <inertial>
@@ -301,5 +301,5 @@
     </collision>
   </link>
-  <!-- Link 4: Upper forearm (pitch rotation) -->
+  <!-- Link 4: Upper forearm -->
   <link name="upper_forearm_link">
     <inertial>
@@ -365,42 +365,94 @@
     </collision>
   </link>
-  <!-- Link 5: End effector (lower forearm with hand and fingers) -->
+  <!-- Link 5: Lower forearm -->
+  <link name="lower_forearm_link">
+    <inertial>
+      <origin xyz="-0.000489596 -0.0073574 -0.0580014" rpy="0 0 0"/>
+      <mass value="1.29529"/>
+      <inertia ixx="0.000900028" ixy="-5.08249e-06" ixz="2.89909e-05" iyy="0.000825354" iyz="-2.4554e-05" izz="0.000743839"/>
+    </inertial>
+    <!-- Part hand_limiter -->
+    <visual>
+      <origin xyz="-0.0317086 -0.0248862 -0.0127911" rpy="-7.42674e-05 0 0"/>
+      <geometry>
+        <mesh filename="package://arm_description/meshes/visual/hand_limiter.stl"/>
+      </geometry>
+      <material name="yellow"/>
+    </visual>
+    <collision>
+      <origin xyz="-0.0317086 -0.0248862 -0.0127911" rpy="-7.42674e-05 0 0"/>
+      <geometry>
+        <mesh filename="package://arm_description/meshes/visual/hand_limiter.stl"/>
+      </geometry>
+    </collision>
+    <!-- Part l_lower_forearm -->
+    <visual>
+      <origin xyz="0 0.00195591 -0.0398386" rpy="0 0 0"/>
+      <geometry>
+        <mesh filename="package://arm_description/meshes/visual/l_lower_forearm.stl"/>
+      </geometry>
+      <material name="teal">
+        <color rgba="0.537255 0.854902 0.827451 1"/>
+      </material>
+    </visual>
+    <collision>
+      <origin xyz="0 0.00195591 -0.0398386" rpy="0 0 0"/>
+      <geometry>
+        <mesh filename="package://arm_description/meshes/visual/l_lower_forearm.stl"/>
+      </geometry>
+    </collision>
+    <!-- Part rotor_x4_p36_36_3 -->
+    <visual>
+      <origin xyz="0 -0.038 -0.0615" rpy="1.5708 0 3.14159"/>
+      <geometry>
+        <mesh filename="package://arm_description/meshes/visual/rotor_x4_p36_36.stl"/>
+      </geometry>
+      <material name="dark_purple"/>
+    </visual>
+    <collision>
+      <origin xyz="0 -0.038 -0.0615" rpy="1.5708 0 3.14159"/>
+      <geometry>
+        <mesh filename="package://arm_description/meshes/visual/rotor_x4_p36_36.stl"/>
+      </geometry>
+    </collision>
+    <!-- Part stator_x4_p36_36_3 -->
+    <visual>
+      <origin xyz="0 -0.038 -0.0615" rpy="1.5708 0 3.14159"/>
+      <geometry>
+        <mesh filename="package://arm_description/meshes/visual/stator_x4_p36_36.stl"/>
+      </geometry>
+      <material name="light_purple"/>
+    </visual>
+    <collision>
+      <origin xyz="0 -0.038 -0.0615" rpy="1.5708 0 3.14159"/>
+      <geometry>
+        <mesh filename="package://arm_description/meshes/visual/stator_x4_p36_36.stl"/>
+      </geometry>
+    </collision>
+  </link>
+  <!-- Link 6: End effector (wrist with hand and fingers) -->
   <link name="end_effector_link">
     <inertial>
-      <origin xyz="-0.00112403 0.00121856 -0.125798" rpy="0 0 0"/>
-      <mass value="0.578"/>
-      <inertia ixx="0.00413859" ixy="-1.05389e-05" ixz="7.52215e-05" iyy="0.00406943" iyz="4.22994e-05" izz="0.000463612"/>
-    </inertial>
-    <!-- Part hand_limiter -->
-    <visual>
-      <origin xyz="-0.0317086 -0.0248862 -0.00779106" rpy="-7.42674e-05 0 0"/>
-      <geometry>
-        <mesh filename="package://arm_description/meshes/visual/hand_limiter.stl"/>
-      </geometry>
-      <material name="yellow"/>
-    </visual>
-    <collision>
-      <origin xyz="-0.0317086 -0.0248862 -0.00779106" rpy="-7.42674e-05 0 0"/>
-      <geometry>
-        <mesh filename="package://arm_description/meshes/visual/hand_limiter.stl"/>
-      </geometry>
-    </collision>
-    <!-- Part l_lower_forearm -->
-    <visual>
-      <origin xyz="-6.05561e-05 0.00294052 -0.058703" rpy="0 0 0"/>
-      <geometry>
-        <mesh filename="package://arm_description/meshes/visual/l_lower_forearm.stl"/>
+      <origin xyz="-5.18072e-05 0.112389 -0.0262499" rpy="0 0 0"/>
+      <mass value="0.398"/>
+      <inertia ixx="0.00159798" ixy="-1.08516e-06" ixz="-7.58273e-08" iyy="0.000261878" iyz="7.53453e-05" izz="0.00147321"/>
+    </inertial>
+    <!-- Part l_wrist -->
+    <visual>
+      <origin xyz="-0.000210278 0.0435776 -0.0192949" rpy="1.5708 0 0"/>
+      <geometry>
+        <mesh filename="package://arm_description/meshes/visual/l_wrist.stl"/>
       </geometry>
       <material name="light_blue"/>
     </visual>
     <collision>
-      <origin xyz="-6.05561e-05 0.00294052 -0.058703" rpy="0 0 0"/>
-      <geometry>
-        <mesh filename="package://arm_description/meshes/visual/l_lower_forearm.stl"/>
+      <origin xyz="-0.000210278 0.0435776 -0.0192949" rpy="1.5708 0 0"/>
+      <geometry>
+        <mesh filename="package://arm_description/meshes/visual/l_wrist.stl"/>
       </geometry>
     </collision>
     <!-- Part hand -->
     <visual>
-      <origin xyz="0 0 -0.235" rpy="0 0 1.5708"/>
+      <origin xyz="0 0.1785 -0.03" rpy="1.5708 -1.5708 0"/>
       <geometry>
         <mesh filename="package://arm_description/meshes/visual/hand.stl"/>
@@ -411,5 +463,5 @@
     </visual>
     <collision>
-      <origin xyz="0 0 -0.235" rpy="0 0 1.5708"/>
+      <origin xyz="0 0.1785 -0.03" rpy="1.5708 -1.5708 0"/>
       <geometry>
         <mesh filename="package://arm_description/meshes/visual/hand.stl"/>
@@ -418,5 +470,5 @@
     <!-- Fingers f1-f5 -->
     <visual>
-      <origin xyz="0 0 -0.235" rpy="0 0 1.5708"/>
+      <origin xyz="0 0.1785 -0.03" rpy="1.5708 -1.5708 0"/>
       <geometry>
         <mesh filename="package://arm_description/meshes/visual/f1.stl"/>
@@ -425,5 +477,5 @@
     </visual>
     <collision>
-      <origin xyz="0 0 -0.235" rpy="0 0 1.5708"/>
+      <origin xyz="0 0.1785 -0.03" rpy="1.5708 -1.5708 0"/>
       <geometry>
         <mesh filename="package://arm_description/meshes/visual/f1.stl"/>
@@ -431,5 +483,5 @@
     </collision>
     <visual>
-      <origin xyz="0 0 -0.235" rpy="0 0 1.5708"/>
+      <origin xyz="0 0.1785 -0.03" rpy="1.5708 -1.5708 0"/>
       <geometry>
         <mesh filename="package://arm_description/meshes/visual/f2.stl"/>
@@ -438,5 +490,5 @@
     </visual>
     <collision>
-      <origin xyz="0 0 -0.235" rpy="0 0 1.5708"/>
+      <origin xyz="0 0.1785 -0.03" rpy="1.5708 -1.5708 0"/>
       <geometry>
         <mesh filename="package://arm_description/meshes/visual/f2.stl"/>
@@ -444,5 +496,5 @@
     </collision>
     <visual>
-      <origin xyz="0 0 -0.235" rpy="0 0 1.5708"/>
+      <origin xyz="0 0.1785 -0.03" rpy="1.5708 -1.5708 0"/>
       <geometry>
         <mesh filename="package://arm_description/meshes/visual/f3.stl"/>
@@ -451,5 +503,5 @@
     </visual>
     <collision>
-      <origin xyz="0 0 -0.235" rpy="0 0 1.5708"/>
+      <origin xyz="0 0.1785 -0.03" rpy="1.5708 -1.5708 0"/>
       <geometry>
         <mesh filename="package://arm_description/meshes/visual/f3.stl"/>
@@ -457,5 +509,5 @@
     </collision>
     <visual>
-      <origin xyz="0 0 -0.235" rpy="0 0 1.5708"/>
+      <origin xyz="0 0.1785 -0.03" rpy="1.5708 -1.5708 0"/>
       <geometry>
         <mesh filename="package://arm_description/meshes/visual/f4.stl"/>
@@ -464,5 +516,5 @@
     </visual>
     <collision>
-      <origin xyz="0 0 -0.235" rpy="0 0 1.5708"/>
+      <origin xyz="0 0.1785 -0.03" rpy="1.5708 -1.5708 0"/>
       <geometry>
         <mesh filename="package://arm_description/meshes/visual/f4.stl"/>
@@ -470,5 +522,5 @@
     </collision>
     <visual>
-      <origin xyz="0 0 -0.235" rpy="0 0 1.5708"/>
+      <origin xyz="0 0.1785 -0.03" rpy="1.5708 -1.5708 0"/>
       <geometry>
         <mesh filename="package://arm_description/meshes/visual/f5.stl"/>
@@ -477,5 +529,5 @@
     </visual>
     <collision>
-      <origin xyz="0 0 -0.235" rpy="0 0 1.5708"/>
+      <origin xyz="0 0.1785 -0.03" rpy="1.5708 -1.5708 0"/>
       <geometry>
         <mesh filename="package://arm_description/meshes/visual/f5.stl"/>

File: src/robot_description/arm_description/urdf/macros/ros2_control.xacro (robot description, xacro)
@@ -6,5 +6,5 @@
                 <plugin>gz_ros2_control/GazeboSimSystem</plugin>
             </hardware>
-            <!-- Arm joints (5 DOF) -->
+            <!-- Arm joints (6 DOF) -->
             <joint name="shoulder_pitch_joint">
                 <command_interface name="position"/>
@@ -37,4 +37,10 @@
                 <state_interface name="effort"/>
             </joint>
+            <joint name="wrist_roll_joint">
+                <command_interface name="position"/>
+                <state_interface name="position"/>
+                <state_interface name="velocity"/>
+                <state_interface name="effort"/>
+            </joint>
         </ros2_control>
     </xacro:macro>

Commit message: add back old gripper

File: src/robot_description/arm_description/urdf/joints/arm_joints.xacro (robot description, xacro)
@@ -52,5 +52,5 @@
     <dynamics damping="0.5" friction="0.1"/>
   </joint>
-  <!-- Joint 6: Wrist roll (NEW) -->
+  <!-- Joint 6: Wrist roll -->
   <joint name="wrist_roll_joint" type="revolute">
     <origin xyz="0 0.03 -0.0615" rpy="-1.5708 0 0"/>
@@ -61,3 +61,30 @@
     <dynamics damping="0.5" friction="0.1"/>
   </joint>
+  <!-- Gripper: Fixed joint from wrist to palm -->
+  <joint name="palm_fixture" type="fixed">
+    <origin xyz="0 0.09 -0.02" rpy="0 0 0"/>
+    <parent link="end_effector_link"/>
+    <child link="left_palm"/>
+  </joint>
+  <!-- Gripper: Right finger (independent control) -->
+  <joint name="left_palm_right_finger" type="prismatic">
+    <origin xyz="0 0 0" rpy="0 0 0"/>
+    <parent link="left_palm"/>
+    <child link="left_palm_right_finger_link"/>
+    <axis xyz="-1 0 0"/>
+    <limit lower="-0.04" upper="0.0" effort="10" velocity="0.05"/>
+    <safety_controller soft_upper_limit="0.0" soft_lower_limit="-0.04" k_velocity="0"/>
+    <dynamics damping="0.1" friction="0.1"/>
+  </joint>
+  <!-- Gripper: Left finger (mimic of right finger) -->
+  <joint name="left_palm_left_finger" type="prismatic">
+    <origin xyz="0 0 0" rpy="0 0 0"/>
+    <parent link="left_palm"/>
+    <child link="left_palm_left_finger_link"/>
+    <axis xyz="-1 0 0"/>
+    <limit lower="0.0" upper="0.04" effort="10" velocity="0.05"/>
+    <safety_controller soft_upper_limit="0.04" soft_lower_limit="0.0" k_velocity="0"/>
+    <mimic joint="left_palm_right_finger" multiplier="-1.0" offset="0"/>
+    <dynamics damping="0.1" friction="1.0"/>
+  </joint>
 </robot>

File: src/robot_description/arm_description/urdf/links/arm_links.xacro (robot description, xacro)
@@ -431,10 +431,10 @@
     </collision>
   </link>
-  <!-- Link 6: End effector (wrist with hand and fingers) -->
+  <!-- Link 6: End effector (wrist only) -->
   <link name="end_effector_link">
     <inertial>
-      <origin xyz="-5.18072e-05 0.112389 -0.0262499" rpy="0 0 0"/>
-      <mass value="0.398"/>
-      <inertia ixx="0.00159798" ixy="-1.08516e-06" ixz="-7.58273e-08" iyy="0.000261878" iyz="7.53453e-05" izz="0.00147321"/>
+      <origin xyz="-0.0002 0.044 -0.019" rpy="0 0 0"/>
+      <mass value="0.15"/>
+      <inertia ixx="0.0002" ixy="0" ixz="0" iyy="0.0001" iyz="0" izz="0.0002"/>
     </inertial>
     <!-- Part l_wrist -->
@@ -452,84 +452,67 @@
       </geometry>
     </collision>
-    <!-- Part hand -->
-    <visual>
-      <origin xyz="0 0.1785 -0.03" rpy="1.5708 -1.5708 0"/>
-      <geometry>
-        <mesh filename="package://arm_description/meshes/visual/hand.stl"/>
-      </geometry>
-      <material name="white">
-        <color rgba="1 1 1 1"/>
-      </material>
-    </visual>
-    <collision>
-      <origin xyz="0 0.1785 -0.03" rpy="1.5708 -1.5708 0"/>
-      <geometry>
-        <mesh filename="package://arm_description/meshes/visual/hand.stl"/>
-      </geometry>
-    </collision>
-    <!-- Fingers f1-f5 -->
-    <visual>
-      <origin xyz="0 0.1785 -0.03" rpy="1.5708 -1.5708 0"/>
-      <geometry>
-        <mesh filename="package://arm_description/meshes/visual/f1.stl"/>
-      </geometry>
-      <material name="white"/>
-    </visual>
-    <collision>
-      <origin xyz="0 0.1785 -0.03" rpy="1.5708 -1.5708 0"/>
-      <geometry>
-        <mesh filename="package://arm_description/meshes/visual/f1.stl"/>
-      </geometry>
-    </collision>
-    <visual>
-      <origin xyz="0 0.1785 -0.03" rpy="1.5708 -1.5708 0"/>
-      <geometry>
-        <mesh filename="package://arm_description/meshes/visual/f2.stl"/>
-      </geometry>
-      <material name="white"/>
-    </visual>
-    <collision>
-      <origin xyz="0 0.1785 -0.03" rpy="1.5708 -1.5708 0"/>
-      <geometry>
-        <mesh filename="package://arm_description/meshes/visual/f2.stl"/>
-      </geometry>
-    </collision>
-    <visual>
-      <origin xyz="0 0.1785 -0.03" rpy="1.5708 -1.5708 0"/>
-      <geometry>
-        <mesh filename="package://arm_description/meshes/visual/f3.stl"/>
-      </geometry>
-      <material name="white"/>
-    </visual>
-    <collision>
-      <origin xyz="0 0.1785 -0.03" rpy="1.5708 -1.5708 0"/>
-      <geometry>
-        <mesh filename="package://arm_description/meshes/visual/f3.stl"/>
-      </geometry>
-    </collision>
-    <visual>
-      <origin xyz="0 0.1785 -0.03" rpy="1.5708 -1.5708 0"/>
-      <geometry>
-        <mesh filename="package://arm_description/meshes/visual/f4.stl"/>
-      </geometry>
-      <material name="white"/>
-    </visual>
-    <collision>
-      <origin xyz="0 0.1785 -0.03" rpy="1.5708 -1.5708 0"/>
-      <geometry>
-        <mesh filename="package://arm_description/meshes/visual/f4.stl"/>
-      </geometry>
-    </collision>
-    <visual>
-      <origin xyz="0 0.1785 -0.03" rpy="1.5708 -1.5708 0"/>
-      <geometry>
-        <mesh filename="package://arm_description/meshes/visual/f5.stl"/>
-      </geometry>
-      <material name="white"/>
-    </visual>
-    <collision>
-      <origin xyz="0 0.1785 -0.03" rpy="1.5708 -1.5708 0"/>
-      <geometry>
-        <mesh filename="package://arm_description/meshes/visual/f5.stl"/>
+  </link>
+  <!-- Gripper: Palm -->
+  <link name="left_palm">
+    <inertial>
+      <origin xyz="0 0.0065 0" rpy="0 0 0"/>
+      <mass value="0.048"/>
+      <inertia ixx="0.000148" ixy="0" ixz="0" iyy="0.000377" iyz="0" izz="0.000285"/>
+    </inertial>
+    <visual>
+      <origin xyz="0 0 0" rpy="0 0 0"/>
+      <geometry>
+        <mesh filename="package://arm_description/meshes/visual/left_palm.stl"/>
+      </geometry>
+      <material name="grey">
+        <color rgba="0.698 0.698 0.698 1"/>
+      </material>
+    </visual>
+    <collision>
+      <origin xyz="0 0 0" rpy="0 0 0"/>
+      <geometry>
+        <mesh filename="package://arm_description/meshes/visual/left_palm.stl"/>
+      </geometry>
+    </collision>
+  </link>
+  <!-- Gripper: Right finger (controlled) -->
+  <link name="left_palm_right_finger_link">
+    <inertial>
+      <origin xyz="0.022 0.050 0" rpy="0 0 0"/>
+      <mass value="0.029"/>
+      <inertia ixx="0.000106" ixy="1.28e-05" ixz="0" iyy="4.91e-05" iyz="0" izz="8.9e-05"/>
+    </inertial>
+    <visual>
+      <origin xyz="-0.005 0 0" rpy="0 0 0"/>
+      <geometry>
+        <mesh filename="package://arm_description/meshes/visual/left_palm_right_finger.stl"/>
+      </geometry>
+      <material name="grey"/>
+    </visual>
+    <collision>
+      <origin xyz="-0.005 0 0" rpy="0 0 0"/>
+      <geometry>
+        <mesh filename="package://arm_description/meshes/visual/left_palm_right_finger.stl"/>
+      </geometry>
+    </collision>
+  </link>
+  <!-- Gripper: Left finger (mimic) -->
+  <link name="left_palm_left_finger_link">
+    <inertial>
+      <origin xyz="-0.017 0.050 0" rpy="0 0 0"/>
+      <mass value="0.029"/>
+      <inertia ixx="0.000106" ixy="-1.28e-05" ixz="0" iyy="4.91e-05" iyz="0" izz="8.9e-05"/>
+    </inertial>
+    <visual>
+      <origin xyz="0 0 0" rpy="0 0 0"/>
+      <geometry>
+        <mesh filename="package://arm_description/meshes/visual/left_palm_left_finger.stl"/>
+      </geometry>
+      <material name="grey"/>
+    </visual>
+    <collision>
+      <origin xyz="0 0 0" rpy="0 0 0"/>
+      <geometry>
+        <mesh filename="package://arm_description/meshes/visual/left_palm_left_finger.stl"/>
       </geometry>
     </collision>

File: src/robot_description/arm_description/urdf/macros/ros2_control.xacro (robot description, xacro)
@@ -43,4 +43,17 @@
                 <state_interface name="effort"/>
             </joint>
+            <!-- Gripper: right finger (controlled) -->
+            <joint name="left_palm_right_finger">
+                <command_interface name="position"/>
+                <state_interface name="position"/>
+                <state_interface name="velocity"/>
+                <state_interface name="effort"/>
+            </joint>
+            <!-- Gripper: left finger (mimic - state only) -->
+            <joint name="left_palm_left_finger">
+                <state_interface name="position"/>
+                <state_interface name="velocity"/>
+                <state_interface name="effort"/>
+            </joint>
         </ros2_control>
     </xacro:macro>

Commit message: Align world frame across URDF and RViz configs

File: src/robot_description/arm_description/urdf/joints/arm_joints.xacro (robot description, xacro)
@@ -3,5 +3,5 @@
   <link name="world"/>
   <joint name="base_fixed_joint" type="fixed">
-    <origin xyz="0 0 0" rpy="0 0 0"/>
+    <origin xyz="0 0 0.807" rpy="0 0 0"/>
     <parent link="world"/>
     <child link="base_link"/>
