Commit message: Fix: find and rename for every changed joint found. added the new wrist joint

File: src/planning/arm_moveit_config/config/arm_description.ros2_control.xacro (robot description, xacro)
@@ -8,36 +8,43 @@
                 <plugin>mock_components/GenericSystem</plugin>
             </hardware>
-            <joint name="base_rotation_joint">
+            <joint name="left_shoulder_pitch_rs04_joint">
                 <command_interface name="position"/>
                 <state_interface name="position">
-                  <param name="initial_value">${initial_positions['base_rotation_joint']}</param>
+                  <param name="initial_value">${initial_positions['left_shoulder_pitch_rs04_joint']}</param>
                 </state_interface>
                 <state_interface name="velocity"/>
             </joint>
-            <joint name="shoulder_pitch_joint">
+            <joint name="left_shoulder_roll_rs04_joint">
                 <command_interface name="position"/>
                 <state_interface name="position">
-                  <param name="initial_value">${initial_positions['shoulder_pitch_joint']}</param>
+                  <param name="initial_value">${initial_positions['left_shoulder_roll_rs04_joint']}</param>
                 </state_interface>
                 <state_interface name="velocity"/>
             </joint>
-            <joint name="elbow_pitch_joint">
+            <joint name="left_shoulder_yaw_rs03_joint">
                 <command_interface name="position"/>
                 <state_interface name="position">
-                  <param name="initial_value">${initial_positions['elbow_pitch_joint']}</param>
+                  <param name="initial_value">${initial_positions['left_shoulder_yaw_rs03_joint']}</param>
                 </state_interface>
                 <state_interface name="velocity"/>
             </joint>
-            <joint name="wrist_pitch_joint">
+            <joint name="left_elbow_rs03_joint">
                 <command_interface name="position"/>
                 <state_interface name="position">
-                  <param name="initial_value">${initial_positions['wrist_pitch_joint']}</param>
+                  <param name="initial_value">${initial_positions['left_elbow_rs03_joint']}</param>
                 </state_interface>
                 <state_interface name="velocity"/>
             </joint>
-            <joint name="wrist_roll_joint">
+            <joint name="left_wrist_rs02_joint">
                 <command_interface name="position"/>
                 <state_interface name="position">
-                  <param name="initial_value">${initial_positions['wrist_roll_joint']}</param>
+                  <param name="initial_value">${initial_positions['left_wrist_rs02_joint']}</param>
+                </state_interface>
+                <state_interface name="velocity"/>
+            </joint>
+            <joint name="left_hand_rs02_joint">
+                <command_interface name="position"/>
+                <state_interface name="position">
+                  <param name="initial_value">${initial_positions['left_hand_rs02_joint']}</param>
                 </state_interface>
                 <state_interface name="velocity"/>

File: src/robot_description/arm_description/urdf/macros/gazebo_extensions.xacro (robot description, xacro)
@@ -3,13 +3,25 @@
     <xacro:property name="damping" value="0.05" />
     <xacro:property name="friction" value="0.01" />
-    <gazebo reference="base_rotation_joint">
+    <gazebo reference="left_shoulder_pitch_rs04_joint">
         <damping>${damping}</damping>
         <friction>${friction}</friction>
     </gazebo>
-    <gazebo reference="shoulder_pitch_joint">
+    <gazebo reference="left_shoulder_roll_rs04_joint">
         <damping>${damping}</damping>
         <friction>${friction}</friction>
     </gazebo>
-    <gazebo reference="elbow_pitch_joint">
+    <gazebo reference="left_shoulder_yaw_rs03_joint">
+        <damping>${damping}</damping>
+        <friction>${friction}</friction>
+    </gazebo>
+    <gazebo reference="left_elbow_rs03_joint">
+        <damping>${damping}</damping>
+        <friction>${friction}</friction>
+    </gazebo>
+    <gazebo reference="left_wrist_rs02_joint">
+        <damping>${damping}</damping>
+        <friction>${friction}</friction>
+    </gazebo>
+    <gazebo reference="left_hand_rs02_joint">
         <damping>${damping}</damping>
         <friction>${friction}</friction>

File: src/robot_description/arm_description/urdf/macros/ros2_control.xacro (robot description, xacro)
@@ -6,25 +6,30 @@
                 <plugin>gz_ros2_control/GazeboSimSystem</plugin>
             </hardware>
-            <joint name="base_rotation_joint">
+            <joint name="left_shoulder_pitch_rs04_joint">
                 <command_interface name="position" />
                 <state_interface name="position" />
                 <state_interface name="velocity" />
             </joint>
-            <joint name="shoulder_pitch_joint">
+            <joint name="left_shoulder_roll_rs04_joint">
                 <command_interface name="position" />
                 <state_interface name="position" />
                 <state_interface name="velocity" />
             </joint>
-            <joint name="elbow_pitch_joint">
+            <joint name="left_shoulder_yaw_rs03_joint">
                 <command_interface name="position" />
                 <state_interface name="position" />
                 <state_interface name="velocity" />
             </joint>
-            <joint name="wrist_pitch_joint">
+            <joint name="left_elbow_rs03_joint">
                 <command_interface name="position" />
                 <state_interface name="position" />
                 <state_interface name="velocity" />
             </joint>
-            <joint name="wrist_roll_joint">
+            <joint name="left_wrist_rs02_joint">
+                <command_interface name="position" />
+                <state_interface name="position" />
+                <state_interface name="velocity" />
+            </joint>
+            <joint name="left_hand_rs02_joint">
                 <command_interface name="position" />
                 <state_interface name="position" />

Commit message: joints renaming, gazebo rotation fro robot and camera

File: src/planning/arm_moveit_config/config/arm_description.ros2_control.xacro (robot description, xacro)
@@ -8,43 +8,57 @@
                 <plugin>mock_components/GenericSystem</plugin>
             </hardware>
-            <joint name="left_shoulder_pitch_rs04_joint">
+            <joint name="left_shoulder_pitch_rs04">
                 <command_interface name="position"/>
                 <state_interface name="position">
-                  <param name="initial_value">${initial_positions['left_shoulder_pitch_rs04_joint']}</param>
+                  <param name="initial_value">${initial_positions['left_shoulder_pitch_rs04']}</param>
                 </state_interface>
                 <state_interface name="velocity"/>
             </joint>
-            <joint name="left_shoulder_roll_rs04_joint">
+            <joint name="left_shoulder_roll_rs04">
                 <command_interface name="position"/>
                 <state_interface name="position">
-                  <param name="initial_value">${initial_positions['left_shoulder_roll_rs04_joint']}</param>
+                  <param name="initial_value">${initial_positions['left_shoulder_roll_rs04']}</param>
                 </state_interface>
                 <state_interface name="velocity"/>
             </joint>
-            <joint name="left_shoulder_yaw_rs03_joint">
+            <joint name="left_shoulder_yaw_rs03">
                 <command_interface name="position"/>
                 <state_interface name="position">
-                  <param name="initial_value">${initial_positions['left_shoulder_yaw_rs03_joint']}</param>
+                  <param name="initial_value">${initial_positions['left_shoulder_yaw_rs03']}</param>
                 </state_interface>
                 <state_interface name="velocity"/>
             </joint>
-            <joint name="left_elbow_rs03_joint">
+            <joint name="left_elbow_rs03">
                 <command_interface name="position"/>
                 <state_interface name="position">
-                  <param name="initial_value">${initial_positions['left_elbow_rs03_joint']}</param>
+                  <param name="initial_value">${initial_positions['left_elbow_rs03']}</param>
                 </state_interface>
                 <state_interface name="velocity"/>
             </joint>
-            <joint name="left_wrist_rs02_joint">
+            <joint name="left_wrist_rs02">
                 <command_interface name="position"/>
                 <state_interface name="position">
-                  <param name="initial_value">${initial_positions['left_wrist_rs02_joint']}</param>
+                  <param name="initial_value">${initial_positions['left_wrist_rs02']}</param>
                 </state_interface>
                 <state_interface name="velocity"/>
             </joint>
-            <joint name="left_hand_rs02_joint">
+            <joint name="left_hand_rs02">
                 <command_interface name="position"/>
                 <state_interface name="position">
-                  <param name="initial_value">${initial_positions['left_hand_rs02_joint']}</param>
+                  <param name="initial_value">${initial_positions['left_hand_rs02']}</param>
+                </state_interface>
+                <state_interface name="velocity"/>
+            </joint>
+            <joint name="left_palm_right_finger">
+                <command_interface name="position"/>
+                <state_interface name="position">
+                  <param name="initial_value">${initial_positions['left_palm_right_finger']}</param>
+                </state_interface>
+                <state_interface name="velocity"/>
+            </joint>
+            <joint name="left_palm_left_finger">
+                <command_interface name="position"/>
+                <state_interface name="position">
+                  <param name="initial_value">${initial_positions['left_palm_left_finger']}</param>
                 </state_interface>
                 <state_interface name="velocity"/>

File: src/robot_description/arm_description/urdf/arm_gazebo.xacro (robot description, xacro)
@@ -15,5 +15,5 @@
     <xacro:include filename="$(find arm_description)/urdf/macros/depth_camera.xacro"/>
     <!-- Mount camera on base_link, 2m above the robot, rotated 90° left and tilted 15° down -->
-    <xacro:depth_camera parent_link="base_link" xyz="0.0 0.0 1.75" rpy="0 ${pi/12} 0" name="camera"/>
+    <xacro:depth_camera parent_link="base_link" xyz="0.0 0.0 1.75" rpy="0 ${pi/12} ${pi/2}" name="camera"/>
     <!-- Gazebo plugins -->
     <gazebo>

File: src/robot_description/arm_description/urdf/joints/arm_joints.xacro (robot description, xacro)
@@ -21,5 +21,5 @@
         <axis xyz="0 0 0" />
     </joint>
-    <joint name="left_shoulder_roll_rs04_flange" type="fixed">
+    <joint name="left_shoulder_roll_rs04_flange_fixture" type="fixed">
         <origin xyz="0.11678 0.0487 -2.7056E-05" rpy="0 0 3.1416" />
         <parent link="left_shoulder_pitch" />
@@ -110,10 +110,10 @@
         <origin xyz="0 0.0945 0" rpy="0.64485 0.44406 0" />
         <parent link="left_wrist" />
-        <child link="left_hand_rs02" />
+        <child link="left_hand_rs02_actuator" />
         <axis xyz="0 0 0" />
     </joint>
     <joint name="left_hand_rs02" type="revolute">
         <origin xyz="0 0 0" rpy="0 0 0" />
-        <parent link="left_hand_rs02" />
+        <parent link="left_hand_rs02_actuator" />
         <child link="left_hand_rs02_flange" />
         <axis xyz="1 0 0" />
@@ -136,5 +136,5 @@
         <origin xyz="0 0 0" rpy="0 0 0" />
         <parent link="left_palm" />
-        <child link="left_palm_right_finger" />
+        <child link="left_palm_right_finger_link" />
         <axis xyz="-1 0 0" />
         <limit lower="-0.033" upper="0.00026" effort="0" velocity="0" />
@@ -144,5 +144,5 @@
         <origin xyz="0 0 0" rpy="0 0 0" />
         <parent link="left_palm" />
-        <child link="left_palm_left_finger" />
+        <child link="left_palm_left_finger_link" />
         <axis xyz="-1 0 0" />
         <limit lower="-0.0041" upper="0.033" effort="0" velocity="0" />

File: src/robot_description/arm_description/urdf/links/arm_links.xacro (robot description, xacro)
@@ -375,5 +375,5 @@
     </collision>
   </link>
-  <link name="left_hand_rs02">
+  <link name="left_hand_rs02_actuator">
     <inertial>
       <origin xyz="-0.023014 2.2389E-07 3.2595E-07" rpy="0 0 0" />
@@ -463,5 +463,5 @@
     </collision>
   </link>
-  <link name="left_palm_right_finger">
+  <link name="left_palm_right_finger_link">
     <inertial>
       <origin xyz="0.021797 0.050369 1.1072E-11" rpy="0 0 0" />
@@ -485,5 +485,5 @@
     </collision>
   </link>
-  <link name="left_palm_left_finger">
+  <link name="left_palm_left_finger_link">
     <inertial>
       <origin xyz="-0.017013 0.050369 1.1072E-11" rpy="0 0 0" />

File: src/robot_description/arm_description/urdf/macros/gazebo_extensions.xacro (robot description, xacro)
@@ -3,25 +3,33 @@
     <xacro:property name="damping" value="0.05" />
     <xacro:property name="friction" value="0.01" />
-    <gazebo reference="left_shoulder_pitch_rs04_joint">
+    <gazebo reference="left_shoulder_pitch_rs04">
         <damping>${damping}</damping>
         <friction>${friction}</friction>
     </gazebo>
-    <gazebo reference="left_shoulder_roll_rs04_joint">
+    <gazebo reference="left_shoulder_roll_rs04">
         <damping>${damping}</damping>
         <friction>${friction}</friction>
     </gazebo>
-    <gazebo reference="left_shoulder_yaw_rs03_joint">
+    <gazebo reference="left_shoulder_yaw_rs03">
         <damping>${damping}</damping>
         <friction>${friction}</friction>
     </gazebo>
-    <gazebo reference="left_elbow_rs03_joint">
+    <gazebo reference="left_elbow_rs03">
         <damping>${damping}</damping>
         <friction>${friction}</friction>
     </gazebo>
-    <gazebo reference="left_wrist_rs02_joint">
+    <gazebo reference="left_wrist_rs02">
         <damping>${damping}</damping>
         <friction>${friction}</friction>
     </gazebo>
-    <gazebo reference="left_hand_rs02_joint">
+    <gazebo reference="left_hand_rs02">
+        <damping>${damping}</damping>
+        <friction>${friction}</friction>
+    </gazebo>
+    <gazebo reference="left_palm_right_finger_joint">
+        <damping>${damping}</damping>
+        <friction>${friction}</friction>
+    </gazebo>
+    <gazebo reference="left_palm_left_finger_joint">
         <damping>${damping}</damping>
         <friction>${friction}</friction>

File: src/robot_description/arm_description/urdf/macros/ros2_control.xacro (robot description, xacro)
@@ -6,30 +6,40 @@
                 <plugin>gz_ros2_control/GazeboSimSystem</plugin>
             </hardware>
-            <joint name="left_shoulder_pitch_rs04_joint">
+            <joint name="left_shoulder_pitch_rs04">
                 <command_interface name="position" />
                 <state_interface name="position" />
                 <state_interface name="velocity" />
             </joint>
-            <joint name="left_shoulder_roll_rs04_joint">
+            <joint name="left_shoulder_roll_rs04">
                 <command_interface name="position" />
                 <state_interface name="position" />
                 <state_interface name="velocity" />
             </joint>
-            <joint name="left_shoulder_yaw_rs03_joint">
+            <joint name="left_shoulder_yaw_rs03">
                 <command_interface name="position" />
                 <state_interface name="position" />
                 <state_interface name="velocity" />
             </joint>
-            <joint name="left_elbow_rs03_joint">
+            <joint name="left_elbow_rs03">
                 <command_interface name="position" />
                 <state_interface name="position" />
                 <state_interface name="velocity" />
             </joint>
-            <joint name="left_wrist_rs02_joint">
+            <joint name="left_wrist_rs02">
                 <command_interface name="position" />
                 <state_interface name="position" />
                 <state_interface name="velocity" />
             </joint>
-            <joint name="left_hand_rs02_joint">
+            <joint name="left_hand_rs02">
+                <command_interface name="position" />
+                <state_interface name="position" />
+                <state_interface name="velocity" />
+            </joint>
+            <joint name="left_palm_right_finger">
+                <command_interface name="position" />
+                <state_interface name="position" />
+                <state_interface name="velocity" />
+            </joint>
+            <joint name="left_palm_left_finger">
                 <command_interface name="position" />
                 <state_interface name="position" />

Commit message: moveit config for arm and hand. arm_controller

File: src/planning/arm_moveit_config/config/arm_description.ros2_control.xacro (robot description, xacro)
@@ -50,4 +50,11 @@
                 <state_interface name="velocity"/>
             </joint>
+            <joint name="left_palm_left_finger">
+                <command_interface name="position"/>
+                <state_interface name="position">
+                  <param name="initial_value">${initial_positions['left_palm_left_finger']}</param>
+                </state_interface>
+                <state_interface name="velocity"/>
+            </joint>
             <joint name="left_palm_right_finger">
                 <command_interface name="position"/>
@@ -57,11 +64,4 @@
                 <state_interface name="velocity"/>
             </joint>
-            <joint name="left_palm_left_finger">
-                <command_interface name="position"/>
-                <state_interface name="position">
-                  <param name="initial_value">${initial_positions['left_palm_left_finger']}</param>
-                </state_interface>
-                <state_interface name="velocity"/>
-            </joint>
         </ros2_control>
     </xacro:macro>
