Commit message: modify for new urdf

File: src/planning/arm_moveit_config/config/arm_description.ros2_control.xacro (robot description, xacro)
@@ -8,57 +8,36 @@
                 <plugin>mock_components/GenericSystem</plugin>
             </hardware>
-            <joint name="left_shoulder_pitch_rs04">
+            <joint name="joint1">
                 <command_interface name="position"/>
                 <state_interface name="position">
-                  <param name="initial_value">${initial_positions['left_shoulder_pitch_rs04']}</param>
+                  <param name="initial_value">${initial_positions['joint1']}</param>
                 </state_interface>
                 <state_interface name="velocity"/>
             </joint>
-            <joint name="left_shoulder_roll_rs04">
+            <joint name="joint2">
                 <command_interface name="position"/>
                 <state_interface name="position">
-                  <param name="initial_value">${initial_positions['left_shoulder_roll_rs04']}</param>
+                  <param name="initial_value">${initial_positions['joint2']}</param>
                 </state_interface>
                 <state_interface name="velocity"/>
             </joint>
-            <joint name="left_shoulder_yaw_rs03">
+            <joint name="joint3">
                 <command_interface name="position"/>
                 <state_interface name="position">
-                  <param name="initial_value">${initial_positions['left_shoulder_yaw_rs03']}</param>
+                  <param name="initial_value">${initial_positions['joint3']}</param>
                 </state_interface>
                 <state_interface name="velocity"/>
             </joint>
-            <joint name="left_elbow_rs03">
+            <joint name="joint4">
                 <command_interface name="position"/>
                 <state_interface name="position">
-                  <param name="initial_value">${initial_positions['left_elbow_rs03']}</param>
+                  <param name="initial_value">${initial_positions['joint4']}</param>
                 </state_interface>
                 <state_interface name="velocity"/>
             </joint>
-            <joint name="left_wrist_rs02">
+            <joint name="joint5">
                 <command_interface name="position"/>
                 <state_interface name="position">
-                  <param name="initial_value">${initial_positions['left_wrist_rs02']}</param>
-                </state_interface>
-                <state_interface name="velocity"/>
-            </joint>
-            <joint name="left_hand_rs02">
-                <command_interface name="position"/>
-                <state_interface name="position">
-                  <param name="initial_value">${initial_positions['left_hand_rs02']}</param>
-                </state_interface>
-                <state_interface name="velocity"/>
-            </joint>
-            <joint name="left_palm_left_finger">
-                <command_interface name="position"/>
-                <state_interface name="position">
-                  <param name="initial_value">${initial_positions['left_palm_left_finger']}</param>
-                </state_interface>
-                <state_interface name="velocity"/>
-            </joint>
-            <joint name="left_palm_right_finger">
-                <command_interface name="position"/>
-                <state_interface name="position">
-                  <param name="initial_value">${initial_positions['left_palm_right_finger']}</param>
+                  <param name="initial_value">${initial_positions['joint5']}</param>
                 </state_interface>
                 <state_interface name="velocity"/>

File: src/planning/arm_moveit_config/config/arm_description.urdf.xacro (robot description, xacro)
@@ -1,8 +1,9 @@
 <?xml version="1.0"?>
 <robot xmlns:xacro="http://www.ros.org/wiki/xacro" name="arm_description">
+    <xacro:arg name="pkg_share" default=""/>
     <xacro:arg name="initial_positions_file" default="initial_positions.yaml" />
-    <!-- Import arm_description urdf file -->
+    <!-- Include robot description (links and joints only, no ros2_control) -->
     <xacro:include filename="$(find arm_description)/urdf/arm.urdf.xacro" />
-    <!-- Import control_xacro -->
+    <!-- ros2_control configuration -->
     <xacro:include filename="arm_description.ros2_control.xacro" />
     <xacro:arm_description_ros2_control name="FakeSystem" initial_positions_file="$(arg initial_positions_file)"/>

File: src/robot_description/arm_description/urdf/arm_gazebo.xacro (robot description, xacro)
@@ -1,5 +1,5 @@
 <?xml version="1.0"?>
 <robot xmlns:xacro="http://ros.org/wiki/xacro">
-    <!-- Publix args so launches can change them -->
+    <!-- Public args so launches can change them -->
     <xacro:arg name="robot_name" default="arm_description"/>
     <xacro:arg name="mesh_dir" default="$(find arm_description)/meshes"/>
@@ -11,9 +11,10 @@
     <xacro:include filename="$(find arm_description)/urdf/macros/ros2_control.xacro"/>
     <xacro:arm_ros2_control/>
-    <!-- <xacro:include filename="$(find arm_description)/urdf/macros/camera.xacro"/> -->
     <!-- Depth Camera -->
     <xacro:include filename="$(find arm_description)/urdf/macros/depth_camera.xacro"/>
-    <!-- Mount camera on base_link, 2m above the robot, rotated 90° left and tilted 15° down -->
-    <xacro:depth_camera parent_link="base_link" xyz="0.0 0.0 1.75" rpy="0 ${pi/12} ${pi/2}" name="camera"/>
+    <!-- Mount camera on base_link, positioned to view the workspace -->
+    <!-- The new robot has the table at z=0, arm starts at table level -->
+    <!-- Position camera 0.5m behind and 0.8m above the robot base, looking down slightly -->
+    <xacro:depth_camera parent_link="base_link" xyz="-0.3 0.0 0.8" rpy="0 ${pi/6} 0" name="camera"/>
     <!-- Gazebo plugins -->
     <gazebo>

File: src/robot_description/arm_description/urdf/joints/arm_joints.xacro (robot description, xacro)
@@ -1,156 +1,54 @@
 <?xml version="1.0"?>
 <robot xmlns:xacro="http://www.ros.org/wiki/xacro">
-    <joint name="left_shoulder_pitch_rs04_actuator_fixture_link" type="fixed">
-        <origin xyz="-0.1079 0 1.425" rpy="0 0 3.1416" />
-        <parent link="base_link" />
-        <child link="left_shoulder_pitch_rs04_actuator" />
-        <axis xyz="0 0 0" />
-    </joint>
-    <joint name="left_shoulder_pitch_rs04" type="revolute">
-        <origin xyz="0 0 0" rpy="0 0 0" />
-        <parent link="left_shoulder_pitch_rs04_actuator" />
-        <child link="left_shoulder_pitch_rs04_flange" />
-        <axis xyz="1 0 0" />
-        <limit lower="-3.14" upper="3.14" effort="40.0" velocity="17.49" />
-        <safety_controller soft_upper_limit="3.14" soft_lower_limit="-3.14" k_velocity="0" />
-    </joint>
-    <joint name="left_shoulder_pitch_fixture" type="fixed">
-        <origin xyz="0 0 0" rpy="0 0 0" />
-        <parent link="left_shoulder_pitch_rs04_flange" />
-        <child link="left_shoulder_pitch" />
-        <axis xyz="0 0 0" />
-    </joint>
-    <joint name="left_shoulder_roll_rs04_flange_fixture" type="fixed">
-        <origin xyz="0.11678 0.0487 -2.7056E-05" rpy="0 -0.1 3.1416" />
-        <parent link="left_shoulder_pitch" />
-        <child link="left_shoulder_roll_rs04_flange" />
-        <axis xyz="0 0 0" />
-    </joint>
-    <joint name="left_shoulder_roll_rs04" type="revolute">
-        <origin xyz="0 0 0" rpy="0 0 0" />
-        <parent link="left_shoulder_roll_rs04_flange" />
-        <child link="left_shoulder_roll_rs04_actuator" />
-        <axis xyz="0 -1 0" />
-        <limit lower="-3.5" upper="0.6" effort="40.0" velocity="17.49" />
-        <safety_controller soft_upper_limit="3.14" soft_lower_limit="-3.14" k_velocity="0" />
-    </joint>
-    <joint name="left_shoulde_roll_fixture" type="fixed">
-        <origin xyz="0 0 0" rpy="0 0 0" />
-        <parent link="left_shoulder_roll_rs04_actuator" />
-        <child link="left_shoulder_roll" />
-        <axis xyz="0 0 0" />
-    </joint>
-    <joint name="left_shoulder_yaw_rs03_actuator_fixture_link" type="fixed">
-        <origin xyz="-0.021972 0.0377 -0.17358" rpy="0.057123 0.11257 0.47088" />
-        <parent link="left_shoulder_roll" />
-        <child link="left_shoulder_yaw_rs03_actuator" />
-        <axis xyz="0 0 0" />
-    </joint>
-    <joint name="left_shoulder_yaw_rs03" type="revolute">
-        <origin xyz="0 0 0" rpy="0 0 0" />
-        <parent link="left_shoulder_yaw_rs03_actuator" />
-        <child link="left_shoulder_yaw_rs03_flange" />
-        <axis xyz="0 0 1" />
-        <limit lower="-3.14" upper="3.14" effort="20.0" velocity="18.85" />
-        <safety_controller soft_upper_limit="3.14" soft_lower_limit="-3.14" k_velocity="0" />
-    </joint>
-    <joint name="left_shoulder_yaw_flange_fixture" type="fixed">
-        <origin xyz="0 0 0" rpy="0 0 0" />
-        <parent link="left_shoulder_yaw_rs03_flange" />
-        <child link="left_shoulder_yaw_flange" />
-        <axis xyz="0 0 0" />
-    </joint>
-    <joint name="left_shoulder_yaw_fixture" type="fixed">
-        <origin xyz="0 0 0" rpy="0 0 0" />
-        <parent link="left_shoulder_yaw_flange" />
-        <child link="left_shoulder_yaw" />
-        <axis xyz="0 0 0" />
-    </joint>
-    <joint name="left_elbow_rs03_actuator_ficture_link" type="fixed">
-        <origin xyz="0 0 -0.0987" rpy="0 0 0" />
-        <parent link="left_shoulder_yaw" />
-        <child link="left_elbow_rs03_actuator" />
-        <axis xyz="0 0 0" />
-    </joint>
-    <joint name="left_elbow_rs03" type="revolute">
-        <origin xyz="0 0 0" rpy="0 0 0" />
-        <parent link="left_elbow_rs03_actuator" />
-        <child link="left_elbow_rs03_flange" />
-        <axis xyz="-1 0 0" />
-        <limit lower="-1.3" upper="1.9" effort="20.0" velocity="18.85" />
-        <safety_controller soft_upper_limit="3.14" soft_lower_limit="-3.14" k_velocity="0" />
-    </joint>
-    <joint name="left_elbow_fixture" type="fixed">
-        <origin xyz="0 0 0" rpy="0 0 0" />
-        <parent link="left_elbow_rs03_flange" />
-        <child link="left_elbow" />
-        <axis xyz="0 0 0" />
-    </joint>
-    <joint name="left_wrist_rs02_actuator_fixture_link" type="fixed">
-        <origin xyz="0.0055 0.044061 -0.15849" rpy="-1.2996 0 0" />
-        <parent link="left_elbow" />
-        <child link="left_wrist_actuator" />
-        <axis xyz="0 0 0" />
-    </joint>
-    <joint name="left_wrist_rs02" type="revolute">
-        <origin xyz="0 0 0" rpy="0 0 0" />
-        <parent link="left_wrist_actuator" />
-        <child link="left_wrist_rs02_flange" />
-        <axis xyz="0 1 0" />
-        <limit lower="-3.14" upper="3.14" effort="6.0" velocity="37.70" />
-        <safety_controller soft_upper_limit="3.14" soft_lower_limit="-3.14" k_velocity="0" />
-    </joint>
-    <joint name="left_wrist_fixture" type="fixed">
-        <origin xyz="0 0 0" rpy="0 0 0" />
-        <parent link="left_wrist_rs02_flange" />
-        <child link="left_wrist" />
-        <axis xyz="0 0 0" />
-    </joint>
-    <joint name="left_hand_rs02_fixture_link" type="fixed">
-        <origin xyz="0 0.0945 0" rpy="0 0.44406 0" />
-        <parent link="left_wrist" />
-        <child link="left_hand_rs02_actuator" />
-        <axis xyz="0 0 0" />
-    </joint>
-    <joint name="left_hand_rs02" type="revolute">
-        <origin xyz="0 0 0" rpy="0 0 0" />
-        <parent link="left_hand_rs02_actuator" />
-        <child link="left_hand_rs02_flange" />
-        <axis xyz="1 0 0" />
-        <limit lower="-1.5" upper="1.7" effort="6.0" velocity="37.70" />
-        <safety_controller soft_upper_limit="1.7" soft_lower_limit="-1.5" k_velocity="0" />
-    </joint>
-    <joint name="left_hand_fixture" type="fixed">
-        <origin xyz="0 0 0" rpy="0.785 0 0" />
-        <parent link="left_hand_rs02_flange" />
-        <child link="left_hand" />
-        <axis xyz="0 0 0" />
-    </joint>
-    <joint name="left_palm_fixture" type="fixed">
-        <origin xyz="0 0.046829 -0.045845" rpy="-0.77494 -0.017568 0.017203" />
-        <parent link="left_hand" />
-        <child link="left_palm" />
-        <axis xyz="0 0 0" />
-    </joint>
-    <!-- Gripper finger joints: Right finger (independent control) -->
-    <joint name="left_palm_right_finger" type="prismatic">
-        <origin xyz="0 0 0" rpy="0 0 0" />
-        <parent link="left_palm" />
-        <child link="left_palm_right_finger_link" />
-        <axis xyz="-1 0 0" />
-        <limit lower="-0.04" upper="0.0" effort="10" velocity="0.05" />
-        <safety_controller soft_upper_limit="0.0" soft_lower_limit="-0.04" k_velocity="0" />
-        <dynamics damping="0.1" friction="0.1" />
-    </joint>
-    <!-- Left finger mimics right finger (symmetric movement) -->
-    <joint name="left_palm_left_finger" type="prismatic">
-        <origin xyz="0 0 0" rpy="0 0 0" />
-        <parent link="left_palm" />
-        <child link="left_palm_left_finger_link" />
-        <axis xyz="-1 0 0" />
-        <limit lower="0.0" upper="0.04" effort="10" velocity="0.05" />
-        <safety_controller soft_upper_limit="0.04" soft_lower_limit="0.0" k_velocity="0" />
-        <mimic joint="left_palm_right_finger" multiplier="-1.0" offset="0" />
-        <dynamics damping="0.1" friction="1.0" />
-    </joint>
+  <link name="world"/>
+  <joint name="base_fixed_joint" type="fixed">
+    <origin xyz="0 0 0" rpy="0 0 0"/>
+    <parent link="world"/>
+    <child link="base_link"/>
+  </joint>
+  <!-- Joint 1: Shoulder pitch (on table surface) -->
+  <joint name="joint1" type="revolute">
+    <origin xyz="0.0498579 0.00126819 6.80296e-06" rpy="1.5708 1.59595e-15 1.5708"/>
+    <parent link="base_link"/>
+    <child link="shoulder_link"/>
+    <axis xyz="0 0 1"/>
+    <limit lower="-1.5708" upper="3.14159" velocity="16.0" effort="20.0"/>
+    <dynamics damping="0.5" friction="0.1"/>
+  </joint>
+  <!-- Joint 2: Shoulder roll -->
+  <joint name="joint2" type="revolute">
+    <origin xyz="0.029 1.02101e-17 -0.078" rpy="-1.5708 -9.59268e-17 1.5708"/>
+    <parent link="shoulder_link"/>
+    <child link="upper_arm_link"/>
+    <axis xyz="0 0 1"/>
+    <limit lower="-3.14159" upper="0.112" velocity="16.0" effort="20.0"/>
+    <dynamics damping="0.5" friction="0.1"/>
+  </joint>
+  <!-- Joint 3: Shoulder yaw -->
+  <joint name="joint3" type="revolute">
+    <origin xyz="-0.157 -1.83881e-16 0.029" rpy="-1.5708 0.000395729 -1.5708"/>
+    <parent link="upper_arm_link"/>
+    <child link="elbow_link"/>
+    <axis xyz="0 0 1"/>
+    <limit lower="-1.57119" upper="1.5704" velocity="16.0" effort="20.0"/>
+    <dynamics damping="0.5" friction="0.1"/>
+  </joint>
+  <!-- Joint 4: Elbow pitch -->
+  <joint name="joint4" type="revolute">
+    <origin xyz="-0.023 4.35849e-17 -0.083" rpy="1.5708 -7.42674e-05 1.5708"/>
+    <parent link="elbow_link"/>
+    <child link="upper_forearm_link"/>
+    <axis xyz="0 0 1"/>
+    <limit lower="-1.57087" upper="1.57072" velocity="16.0" effort="10.0"/>
+    <dynamics damping="0.5" friction="0.1"/>
+  </joint>
+  <!-- Joint 5: Elbow yaw -->
+  <joint name="joint5" type="revolute">
+    <origin xyz="7.37257e-17 -0.151 0.023" rpy="-1.5708 -1.5708 0"/>
+    <parent link="upper_forearm_link"/>
+    <child link="end_effector_link"/>
+    <axis xyz="0 0 1"/>
+    <limit lower="-1.5708" upper="1.5708" velocity="16.0" effort="10.0"/>
+    <dynamics damping="0.5" friction="0.1"/>
+  </joint>
 </robot>
