Commit message: modify for new urdf

File: src/robot_description/arm_description/urdf/links/arm_links.xacro (robot description, xacro)
@@ -1,509 +1,344 @@
 <?xml version="1.0"?>
 <robot xmlns:xacro="http://www.ros.org/wiki/xacro">
+  <!-- Base link (table/stand with menghina and stator) -->
   <link name="base_link">
     <inertial>
-      <origin xyz="-1.4142E-08 1.4615E-08 0.35593" rpy="0 0 0" />
-      <mass value="77.718" />
-      <inertia ixx="21.025" ixy="-8.8504E-08" ixz="6.1541E-07" iyy="21.028" iyz="-1.1273E-06" izz="1.008" />
-    </inertial>
-    <visual>
-      <origin xyz="0 0 0" rpy="0 0 0" />
-      <geometry>
-        <mesh filename="package://arm_description/meshes/visual/base_link.STL" />
-      </geometry>
-      <material name="">
-        <color rgba="1 0.94902 0.9098 1" />
-      </material>
-    </visual>
-    <collision>
-      <origin xyz="0 0 0" rpy="0 0 0" />
-      <geometry>
-        <mesh filename="package://arm_description/meshes/visual/base_link.STL" />
-      </geometry>
-    </collision>
-  </link>
-  <link name="left_shoulder_pitch_rs04_actuator">
-    <inertial>
-      <origin xyz="-0.024532 6.1284E-13 3.0664E-13" rpy="0 0 0" />
-      <mass value="1.345" />
-      <inertia ixx="0.00087641" ixy="-1.2177E-17" ixz="-1.4781E-16" iyy="0.0005424" iyz="-3.5471E-06" izz="0.00054116" />
-    </inertial>
-    <visual>
-      <origin xyz="0 0 0" rpy="0 0 0" />
-      <geometry>
-        <mesh filename="package://arm_description/meshes/visual/left_shoulder_pitch_rs04_actuator.STL" />
-      </geometry>
-      <material name="">
-        <color rgba="0.82353 0.82353 1 1" />
-      </material>
-    </visual>
-    <collision>
-      <origin xyz="0 0 0" rpy="0 0 0" />
-      <geometry>
-        <mesh filename="package://arm_description/meshes/visual/left_shoulder_pitch_rs04_actuator.STL" />
-      </geometry>
-    </collision>
-  </link>
-  <link name="left_shoulder_pitch_rs04_flange">
-    <inertial>
-      <origin xyz="-0.0018894 -9.5572E-05 2.5808E-05" rpy="0 0 0" />
-      <mass value="0.0075" />
-      <inertia ixx="2.3623E-06" ixy="6.4388E-21" ixz="-7.1204E-21" iyy="1.1941E-06" iyz="3.6528E-21" izz="1.1941E-06" />
-    </inertial>
-    <visual>
-      <origin xyz="0 0 0" rpy="0 0 0" />
-      <geometry>
-        <mesh filename="package://arm_description/meshes/visual/left_shoulder_pitch_rs04_flange.STL" />
-      </geometry>
-      <material name="">
-        <color rgba="0.82353 0.82353 1 1" />
-      </material>
-    </visual>
-    <collision>
-      <origin xyz="0 0 0" rpy="0 0 0" />
-      <geometry>
-        <mesh filename="package://arm_description/meshes/visual/left_shoulder_pitch_rs04_flange.STL" />
-      </geometry>
-    </collision>
-  </link>
-  <link name="left_shoulder_pitch">
-    <inertial>
-      <origin xyz="0.068247 0.039551 -5.234E-06" rpy="0 0 0" />
-      <mass value="0.29944" />
-      <inertia ixx="0.0043457" ixy="-0.0020544" ixz="-3.8776E-07" iyy="0.0075578" iyz="-1.6186E-07" izz="0.0076907" />
-    </inertial>
-    <visual>
-      <origin xyz="0 0 0" rpy="0 0 0" />
-      <geometry>
-        <mesh filename="package://arm_description/meshes/visual/left_shoulder_pitch.STL" />
-      </geometry>
-      <material name="">
-        <color rgba="0.69804 0.69804 0.69804 1" />
-      </material>
-    </visual>
-    <collision>
-      <origin xyz="0 0 0" rpy="0 0 0" />
-      <geometry>
-        <mesh filename="package://arm_description/meshes/visual/left_shoulder_pitch.STL" />
-      </geometry>
-    </collision>
-  </link>
-  <link name="left_shoulder_roll_rs04_flange">
-    <inertial>
-      <origin xyz="-5.7019E-12 -0.0021106 2.1706E-10" rpy="0 0 0" />
-      <mass value="0.0075" />
-      <inertia ixx="1.1941E-06" ixy="3.5072E-22" ixz="1.0191E-21" iyy="2.3623E-06" iyz="-4.903E-15" izz="1.1941E-06" />
-    </inertial>
-    <visual>
-      <origin xyz="0 0 0" rpy="0 0 0" />
-      <geometry>
-        <mesh filename="package://arm_description/meshes/visual/left_shoulder_roll_rs04_flange.STL" />
-      </geometry>
-      <material name="">
-        <color rgba="0.82353 0.82353 1 1" />
-      </material>
-    </visual>
-    <collision>
-      <origin xyz="0 0 0" rpy="0 0 0" />
-      <geometry>
-        <mesh filename="package://arm_description/meshes/visual/left_shoulder_roll_rs04_flange.STL" />
-      </geometry>
-    </collision>
-  </link>
-  <link name="left_shoulder_roll_rs04_actuator">
-    <inertial>
-      <origin xyz="7.5431E-05 0.020532 2.7056E-05" rpy="0 0 0" />
-      <mass value="1.345" />
-      <inertia ixx="0.00054201" ixy="-1.5116E-14" ixz="-3.5941E-06" iyy="0.00087641" iyz="-1.4055E-12" izz="0.00054156" />
-    </inertial>
-    <visual>
-      <origin xyz="0 0 0" rpy="0 0 0" />
-      <geometry>
-        <mesh filename="package://arm_description/meshes/visual/left_shoulder_roll_rs04_actuator.STL" />
-      </geometry>
-      <material name="">
-        <color rgba="0.82353 0.82353 1 1" />
-      </material>
-    </visual>
-    <collision>
-      <origin xyz="0 0 0" rpy="0 0 0" />
-      <geometry>
-        <mesh filename="package://arm_description/meshes/visual/left_shoulder_roll_rs04_actuator.STL" />
-      </geometry>
-    </collision>
-  </link>
-  <link name="left_shoulder_roll">
-    <inertial>
-      <origin xyz="-0.0075223 0.049755 -0.055681" rpy="0 0 0" />
-      <mass value="0.2494" />
-      <inertia ixx="0.0066808" ixy="-0.00010577" ixz="-0.00053776" iyy="0.0073988" iyz="-0.0008009" izz="0.0022285" />
-    </inertial>
-    <visual>
-      <origin xyz="0 0 0" rpy="0 0 0" />
-      <geometry>
-        <mesh filename="package://arm_description/meshes/visual/left_shoulder_roll.STL" />
-      </geometry>
-      <material name="">
-        <color rgba="0.69804 0.69804 0.69804 1" />
-      </material>
-    </visual>
-    <collision>
-      <origin xyz="0 0 0" rpy="0 0 0" />
-      <geometry>
-        <mesh filename="package://arm_description/meshes/visual/left_shoulder_roll.STL" />
-      </geometry>
-    </collision>
-  </link>
-  <link name="left_shoulder_yaw_rs03_actuator">
-    <inertial>
-      <origin xyz="-0.00013735 -0.00027 0.025084" rpy="0 0 0" />
-      <mass value="0.83" />
-      <inertia ixx="0.00027432" ixy="-2.0735E-06" ixz="-2.5625E-07" iyy="0.00027129" iyz="-5.1493E-07" izz="0.00038166" />
-    </inertial>
-    <visual>
-      <origin xyz="0 0 0" rpy="0 0 0" />
-      <geometry>
-        <mesh filename="package://arm_description/meshes/visual/left_shoulder_yaw_rs03_actuator.STL" />
-      </geometry>
-      <material name="">
-        <color rgba="0.82353 0.82353 1 1" />
-      </material>
-    </visual>
-    <collision>
-      <origin xyz="0 0 0" rpy="0 0 0" />
-      <geometry>
-        <mesh filename="package://arm_description/meshes/visual/left_shoulder_yaw_rs03_actuator.STL" />
-      </geometry>
-    </collision>
-  </link>
-  <link name="left_shoulder_yaw_rs03_flange">
-    <inertial>
-      <origin xyz="-2.6865E-10 -6.8053E-10 -0.0012563" rpy="0 0 0" />
-      <mass value="0.005" />
-      <inertia ixx="5.6768E-07" ixy="8.5365E-22" ixz="8.5365E-22" iyy="5.6768E-07" iyz="2.647E-23" izz="1.1311E-06" />
-    </inertial>
-    <visual>
-      <origin xyz="0 0 0" rpy="0 0 0" />
-      <geometry>
-        <mesh filename="package://arm_description/meshes/visual/left_shoulder_yaw_rs03_flange.STL" />
-      </geometry>
-      <material name="">
-        <color rgba="0.82353 0.82353 1 1" />
-      </material>
-    </visual>
-    <collision>
-      <origin xyz="0 0 0" rpy="0 0 0" />
-      <geometry>
-        <mesh filename="package://arm_description/meshes/visual/left_shoulder_yaw_rs03_flange.STL" />
-      </geometry>
-    </collision>
-  </link>
-  <link name="left_shoulder_yaw_flange">
-    <inertial>
-      <origin xyz="-2.2214E-10 -3.6885E-10 -0.0089804" rpy="0 0 0" />
-      <mass value="0.008838" />
-      <inertia ixx="1.2318E-05" ixy="-9.4259E-08" ixz="4.4901E-16" iyy="1.1992E-05" iyz="-6.0556E-16" izz="2.339E-05" />
-    </inertial>
-    <visual>
-      <origin xyz="0 0 0" rpy="0 0 0" />
-      <geometry>
-        <mesh filename="package://arm_description/meshes/visual/left_shoulder_yaw_flange.STL" />
-      </geometry>
-      <material name="">
-        <color rgba="0.69804 0.69804 0.69804 1" />
-      </material>
-    </visual>
-    <collision>
-      <origin xyz="0 0 0" rpy="0 0 0" />
-      <geometry>
-        <mesh filename="package://arm_description/meshes/visual/left_shoulder_yaw_flange.STL" />
-      </geometry>
-    </collision>
-  </link>
-  <link name="left_shoulder_yaw">
-    <inertial>
-      <origin xyz="-0.027609 1.0122E-06 -0.076632" rpy="0 0 0" />
-      <mass value="0.122018" />
-      <inertia ixx="0.0018364" ixy="2.5971E-07" ixz="-0.00033902" iyy="0.0016454" iyz="8.6387E-08" izz="0.0010145" />
-    </inertial>
-    <visual>
-      <origin xyz="0 0 0" rpy="0 0 0" />
-      <geometry>
-        <mesh filename="package://arm_description/meshes/visual/left_shoulder_yaw.STL" />
-      </geometry>
-      <material name="">
-        <color rgba="0.69804 0.69804 0.69804 1" />
-      </material>
-    </visual>
-    <collision>
-      <origin xyz="0 0 0" rpy="0 0 0" />
-      <geometry>
-        <mesh filename="package://arm_description/meshes/visual/left_shoulder_yaw.STL" />
-      </geometry>
-    </collision>
-  </link>
-  <link name="left_elbow_rs03_actuator">
-    <inertial>
-      <origin xyz="-0.025084 8.1191E-07 -0.00030291" rpy="0 0 0" />
-      <mass value="0.83" />
-      <inertia ixx="0.00038166" ixy="3.1874E-09" ixz="5.7519E-07" iyy="0.00027537" iyz="1.1044E-08" izz="0.00027024" />
-    </inertial>
-    <visual>
-      <origin xyz="0 0 0" rpy="0 0 0" />
-      <geometry>
-        <mesh filename="package://arm_description/meshes/visual/left_elbow_rs03_actuator.STL" />
-      </geometry>
-      <material name="">
-        <color rgba="0.82353 0.82353 1 1" />
-      </material>
-    </visual>
-    <collision>
-      <origin xyz="0 0 0" rpy="0 0 0" />
-      <geometry>
-        <mesh filename="package://arm_description/meshes/visual/left_elbow_rs03_actuator.STL" />
-      </geometry>
-    </collision>
-  </link>
-  <link name="left_elbow_rs03_flange">
-    <inertial>
-      <origin xyz="0.0012563 -1.3773E-09 -1.6467E-10" rpy="0 0 0" />
-      <mass value="0.005" />
-      <inertia ixx="1.1311E-06" ixy="1.3467E-21" ixz="4.7778E-21" iyy="5.6768E-07" iyz="-4.4999E-22" izz="5.6768E-07" />
-    </inertial>
-    <visual>
-      <origin xyz="0 0 0" rpy="0 0 0" />
-      <geometry>
-        <mesh filename="package://arm_description/meshes/visual/left_elbow_rs03_flange.STL" />
-      </geometry>
-      <material name="">
-        <color rgba="0.82353 0.82353 1 1" />
-      </material>
-    </visual>
-    <collision>
-      <origin xyz="0 0 0" rpy="0 0 0" />
-      <geometry>
-        <mesh filename="package://arm_description/meshes/visual/left_elbow_rs03_flange.STL" />
-      </geometry>
-    </collision>
-  </link>
-  <link name="left_elbow">
-    <inertial>
-      <origin xyz="0.020821 0.0089724 -0.03236" rpy="0 0 0" />
-      <mass value="0.1949" />
-      <inertia ixx="0.0036503" ixy="0.00012418" ixz="-0.00045842" iyy="0.0031234" iyz="0.00057257" izz="0.001216" />
-    </inertial>
-    <visual>
-      <origin xyz="0 0 0" rpy="0 0 0" />
-      <geometry>
-        <mesh filename="package://arm_description/meshes/visual/left_elbow.STL" />
-      </geometry>
-      <material name="">
-        <color rgba="0.69804 0.69804 0.69804 1" />
-      </material>
-    </visual>
-    <collision>
-      <origin xyz="0 0 0" rpy="0 0 0" />
-      <geometry>
-        <mesh filename="package://arm_description/meshes/visual/left_elbow.STL" />
-      </geometry>
-    </collision>
-  </link>
-  <link name="left_wrist_actuator">
-    <inertial>
-      <origin xyz="-6.2313E-10 -0.023014 2.7886E-07" rpy="0 0 0" />
-      <mass value="0.38" />
-      <inertia ixx="8.809E-05" ixy="-1.0059E-17" ixz="-7.708E-20" iyy="0.000127" iyz="3.6839E-17" izz="8.809E-05" />
-    </inertial>
-    <visual>
-      <origin xyz="0 0 0" rpy="0 0 0" />
-      <geometry>
-        <mesh filename="package://arm_description/meshes/visual/left_wrist_actuator.STL" />
-      </geometry>
-      <material name="">
-        <color rgba="0.82353 0.82353 1 1" />
-      </material>
-    </visual>
-    <collision>
-      <origin xyz="0 0 0" rpy="0 0 0" />
-      <geometry>
-        <mesh filename="package://arm_description/meshes/visual/left_wrist_actuator.STL" />
-      </geometry>
-    </collision>
-  </link>
-  <link name="left_wrist_rs02_flange">
-    <inertial>
-      <origin xyz="-3.2202E-10 -0.0019899 2.7874E-07" rpy="0 0 0" />
-      <mass value="0.0025" />
-      <inertia ixx="1.3495E-07" ixy="8.3809E-20" ixz="-2.7711E-22" iyy="2.634E-07" iyz="1.0102E-19" izz="1.3495E-07" />
-    </inertial>
-    <visual>
-      <origin xyz="0 0 0" rpy="0 0 0" />
-      <geometry>
-        <mesh filename="package://arm_description/meshes/visual/left_wrist_rs02_flange.STL" />
-      </geometry>
-      <material name="">
-        <color rgba="0.82353 0.82353 1 1" />
-      </material>
-    </visual>
-    <collision>
-      <origin xyz="0 0 0" rpy="0 0 0" />
-      <geometry>
-        <mesh filename="package://arm_description/meshes/visual/left_wrist_rs02_flange.STL" />
-      </geometry>
-    </collision>
-  </link>
-  <link name="left_wrist">
-    <inertial>
-      <origin xyz="-0.012628 0.041809 0.0059405" rpy="0 0 0" />
-      <mass value="0.09723" />
-      <inertia ixx="0.0010421" ixy="0.00023897" ixz="2.5575E-06" iyy="0.00064729" iyz="-0.00011195" izz="0.0010487" />
-    </inertial>
-    <visual>
-      <origin xyz="0 0 0" rpy="0 0 0" />
-      <geometry>
-        <mesh filename="package://arm_description/meshes/visual/left_wrist.STL" />
-      </geometry>
-      <material name="">
-        <color rgba="0.69804 0.69804 0.69804 1" />
-      </material>
-    </visual>
-    <collision>
-      <origin xyz="0 0 0" rpy="0 0 0" />
-      <geometry>
-        <mesh filename="package://arm_description/meshes/visual/left_wrist.STL" />
-      </geometry>
-    </collision>
-  </link>
-  <link name="left_hand_rs02_actuator">
-    <inertial>
-      <origin xyz="-0.023014 2.2389E-07 3.2595E-07" rpy="0 0 0" />
-      <mass value="0.38" />
-      <inertia ixx="0.000127" ixy="2.2647E-11" ixz="-1.704E-11" iyy="8.809E-05" iyz="-9.7485E-18" izz="8.809E-05" />
-    </inertial>
-    <visual>
-      <origin xyz="0 0 0" rpy="0 0 0" />
-      <geometry>
-        <mesh filename="package://arm_description/meshes/visual/left_hand_rs02.STL" />
-      </geometry>
-      <material name="">
-        <color rgba="0.82353 0.82353 1 1" />
-      </material>
-    </visual>
-    <collision>
-      <origin xyz="0 0 0" rpy="0 0 0" />
-      <geometry>
-        <mesh filename="package://arm_description/meshes/visual/left_hand_rs02.STL" />
-      </geometry>
-    </collision>
-  </link>
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
File: src/robot_description/arm_description/urdf/macros/gazebo_extensions.xacro (robot description, xacro)
@@ -3,33 +3,21 @@
     <xacro:property name="damping" value="0.05" />
     <xacro:property name="friction" value="0.01" />
-    <gazebo reference="left_shoulder_pitch_rs04">
+    <gazebo reference="joint1">
         <damping>${damping}</damping>
         <friction>${friction}</friction>
     </gazebo>
-    <gazebo reference="left_shoulder_roll_rs04">
+    <gazebo reference="joint2">
         <damping>${damping}</damping>
         <friction>${friction}</friction>
     </gazebo>
-    <gazebo reference="left_shoulder_yaw_rs03">
+    <gazebo reference="joint3">
         <damping>${damping}</damping>
         <friction>${friction}</friction>
     </gazebo>
-    <gazebo reference="left_elbow_rs03">
+    <gazebo reference="joint4">
         <damping>${damping}</damping>
         <friction>${friction}</friction>
     </gazebo>
-    <gazebo reference="left_wrist_rs02">
-        <damping>${damping}</damping>
-        <friction>${friction}</friction>
-    </gazebo>
-    <gazebo reference="left_hand_rs02">
-        <damping>${damping}</damping>
-        <friction>${friction}</friction>
-    </gazebo>
-    <gazebo reference="left_palm_right_finger_joint">
-        <damping>${damping}</damping>
-        <friction>${friction}</friction>
-    </gazebo>
-    <gazebo reference="left_palm_left_finger_joint">
+    <gazebo reference="joint5">
         <damping>${damping}</damping>
         <friction>${friction}</friction>

File: src/robot_description/arm_description/urdf/macros/materials.xacro (robot description, xacro)
@@ -1,10 +1,29 @@
 <?xml version="1.0"?>
 <robot xmlns:xacro="http://www.ros.org/wiki/xacro">
-  <!-- Basic colors -->
+  <!-- Source robot colors -->
+  <material name="blue">
+    <color rgba="0.615686 0.811765 0.929412 1"/>
+  </material>
+  <material name="dark_blue">
+    <color rgba="0.32549 0.529412 0.752941 1"/>
+  </material>
+  <material name="gold">
+    <color rgba="0.960784 0.835294 0.470588 1"/>
+  </material>
+  <material name="orange">
+    <color rgba="0.65098 0.486275 0.0196078 1"/>
+  </material>
+  <material name="purple">
+    <color rgba="0.764706 0.545098 0.803922 1"/>
+  </material>
+  <material name="dark_purple">
+    <color rgba="0.380392 0.0470588 0.435294 1"/>
+  </material>
+  <material name="white">
+    <color rgba="1 1 1 1"/>
+  </material>
+  <!-- Additional basic colors -->
   <material name="black">
     <color rgba="0.0 0.0 0.0 1.0"/>
-  </material>
-  <material name="white">
-    <color rgba="1.0 1.0 1.0 1.0"/>
   </material>
   <material name="red">
@@ -14,15 +33,6 @@
     <color rgba="0.0 1.0 0.0 1.0"/>
   </material>
-  <material name="blue">
-    <color rgba="0.0 0.0 1.0 1.0"/>
-  </material>
   <material name="yellow">
     <color rgba="1.0 1.0 0.0 1.0"/>
-  </material>
-  <material name="orange">
-    <color rgba="1.0 0.647 0.0 1.0"/>
-  </material>
-  <material name="purple">
-    <color rgba="0.5 0.0 0.5 1.0"/>
   </material>
   <!-- Grayscale variations -->
@@ -39,7 +49,4 @@
   <material name="silver">
     <color rgba="0.75 0.75 0.75 1.0"/>
-  </material>
-  <material name="gold">
-    <color rgba="1.0 0.843 0.0 1.0"/>
   </material>
   <material name="bronze">

File: src/robot_description/arm_description/urdf/macros/ros2_control.xacro (robot description, xacro)
@@ -6,52 +6,34 @@
                 <plugin>gz_ros2_control/GazeboSimSystem</plugin>
             </hardware>
-            <joint name="left_shoulder_pitch_rs04">
-                <command_interface name="position" />
+            <!-- Arm joints (5 DOF) -->
+            <joint name="joint1">
+                <command_interface name="position"/>
                 <state_interface name="position"/>
-                <state_interface name="velocity" />
-                <state_interface name="effort" />
+                <state_interface name="velocity"/>
+                <state_interface name="effort"/>
             </joint>
-            <joint name="left_shoulder_roll_rs04">
-                <command_interface name="position" />
+            <joint name="joint2">
+                <command_interface name="position"/>
                 <state_interface name="position"/>
-                <state_interface name="velocity" />
-                <state_interface name="effort" />
+                <state_interface name="velocity"/>
+                <state_interface name="effort"/>
             </joint>
-            <joint name="left_shoulder_yaw_rs03">
-                <command_interface name="position" />
+            <joint name="joint3">
+                <command_interface name="position"/>
                 <state_interface name="position"/>
-                <state_interface name="velocity" />
-                <state_interface name="effort" />
+                <state_interface name="velocity"/>
+                <state_interface name="effort"/>
             </joint>
-            <joint name="left_elbow_rs03">
-                <command_interface name="position" />
+            <joint name="joint4">
+                <command_interface name="position"/>
                 <state_interface name="position"/>
-                <state_interface name="velocity" />
-                <state_interface name="effort" />
+                <state_interface name="velocity"/>
+                <state_interface name="effort"/>
             </joint>
-            <joint name="left_wrist_rs02">
-                <command_interface name="position" />
+            <joint name="joint5">
+                <command_interface name="position"/>
                 <state_interface name="position"/>
-                <state_interface name="velocity" />
-                <state_interface name="effort" />
-            </joint>
-            <joint name="left_hand_rs02">
-                <command_interface name="position" />
-                <state_interface name="position"/>
-                <state_interface name="velocity" />
-                <state_interface name="effort" />
-            </joint>
-            <!-- Gripper: Only control main joint, left finger mimics automatically -->
-            <joint name="left_palm_right_finger">
-                <command_interface name="position" />
-                <state_interface name="position" />
-                <state_interface name="velocity" />
-                <state_interface name="effort" />
-            </joint>
-            <!-- left_palm_left_finger is a mimic joint - only state interfaces -->
-            <joint name="left_palm_left_finger">
-                <state_interface name="position" />
-                <state_interface name="velocity" />
-                <state_interface name="effort" />
+                <state_interface name="velocity"/>
+                <state_interface name="effort"/>
             </joint>
         </ros2_control>
