Commit message: review all joints

File: src/planning/arm_moveit_config/config/arm_description.ros2_control.xacro (robot description, xacro)
@@ -8,36 +8,36 @@
                 <plugin>mock_components/GenericSystem</plugin>
             </hardware>
-            <joint name="joint1">
+            <joint name="shoulder_pitch_joint">
                 <command_interface name="position"/>
                 <state_interface name="position">
-                  <param name="initial_value">${initial_positions['joint1']}</param>
+                  <param name="initial_value">${initial_positions['shoulder_pitch_joint']}</param>
                 </state_interface>
                 <state_interface name="velocity"/>
             </joint>
-            <joint name="joint2">
+            <joint name="shoulder_roll_joint">
                 <command_interface name="position"/>
                 <state_interface name="position">
-                  <param name="initial_value">${initial_positions['joint2']}</param>
+                  <param name="initial_value">${initial_positions['shoulder_roll_joint']}</param>
                 </state_interface>
                 <state_interface name="velocity"/>
             </joint>
-            <joint name="joint3">
+            <joint name="shoulder_yaw_joint">
                 <command_interface name="position"/>
                 <state_interface name="position">
-                  <param name="initial_value">${initial_positions['joint3']}</param>
+                  <param name="initial_value">${initial_positions['shoulder_yaw_joint']}</param>
                 </state_interface>
                 <state_interface name="velocity"/>
             </joint>
-            <joint name="joint4">
+            <joint name="elbow_pitch_joint">
                 <command_interface name="position"/>
                 <state_interface name="position">
-                  <param name="initial_value">${initial_positions['joint4']}</param>
+                  <param name="initial_value">${initial_positions['elbow_pitch_joint']}</param>
                 </state_interface>
                 <state_interface name="velocity"/>
             </joint>
-            <joint name="joint5">
+            <joint name="elbow_yaw_joint">
                 <command_interface name="position"/>
                 <state_interface name="position">
-                  <param name="initial_value">${initial_positions['joint5']}</param>
+                  <param name="initial_value">${initial_positions['elbow_yaw_joint']}</param>
                 </state_interface>
                 <state_interface name="velocity"/>

File: src/robot_description/arm_description/urdf/joints/arm_joints.xacro (robot description, xacro)
@@ -8,5 +8,5 @@
   </joint>
   <!-- Joint 1: Shoulder pitch (on table surface) -->
-  <joint name="joint1" type="revolute">
+  <joint name="shoulder_pitch_joint" type="revolute">
     <origin xyz="0.0498579 0.00126819 6.80296e-06" rpy="1.5708 1.59595e-15 1.5708"/>
     <parent link="base_link"/>
@@ -17,5 +17,5 @@
   </joint>
   <!-- Joint 2: Shoulder roll -->
-  <joint name="joint2" type="revolute">
+  <joint name="shoulder_roll_joint" type="revolute">
     <origin xyz="0.029 1.02101e-17 -0.078" rpy="-1.5708 -9.59268e-17 1.5708"/>
     <parent link="shoulder_link"/>
@@ -26,5 +26,5 @@
   </joint>
   <!-- Joint 3: Shoulder yaw -->
-  <joint name="joint3" type="revolute">
+  <joint name="shoulder_yaw_joint" type="revolute">
     <origin xyz="-0.157 -1.83881e-16 0.029" rpy="-1.5708 0.000395729 -1.5708"/>
     <parent link="upper_arm_link"/>
@@ -35,5 +35,5 @@
   </joint>
   <!-- Joint 4: Elbow pitch -->
-  <joint name="joint4" type="revolute">
+  <joint name="elbow_pitch_joint" type="revolute">
     <origin xyz="-0.023 4.35849e-17 -0.083" rpy="1.5708 -7.42674e-05 1.5708"/>
     <parent link="elbow_link"/>
@@ -44,5 +44,5 @@
   </joint>
   <!-- Joint 5: Elbow yaw -->
-  <joint name="joint5" type="revolute">
+  <joint name="elbow_yaw_joint" type="revolute">
     <origin xyz="7.37257e-17 -0.151 0.023" rpy="-1.5708 -1.5708 0"/>
     <parent link="upper_forearm_link"/>

File: src/robot_description/arm_description/urdf/macros/gazebo_extensions.xacro (robot description, xacro)
@@ -3,21 +3,21 @@
     <xacro:property name="damping" value="0.05" />
     <xacro:property name="friction" value="0.01" />
-    <gazebo reference="joint1">
+    <gazebo reference="shoulder_pitch_joint">
         <damping>${damping}</damping>
         <friction>${friction}</friction>
     </gazebo>
-    <gazebo reference="joint2">
+    <gazebo reference="shoulder_roll_joint">
         <damping>${damping}</damping>
         <friction>${friction}</friction>
     </gazebo>
-    <gazebo reference="joint3">
+    <gazebo reference="shoulder_yaw_joint">
         <damping>${damping}</damping>
         <friction>${friction}</friction>
     </gazebo>
-    <gazebo reference="joint4">
+    <gazebo reference="elbow_pitch_joint">
         <damping>${damping}</damping>
         <friction>${friction}</friction>
     </gazebo>
-    <gazebo reference="joint5">
+    <gazebo reference="elbow_yaw_joint">
         <damping>${damping}</damping>
         <friction>${friction}</friction>

File: src/robot_description/arm_description/urdf/macros/ros2_control.xacro (robot description, xacro)
@@ -7,5 +7,5 @@
             </hardware>
             <!-- Arm joints (5 DOF) -->
-            <joint name="joint1">
+            <joint name="shoulder_pitch_joint">
                 <command_interface name="position"/>
                 <state_interface name="position"/>
@@ -13,5 +13,5 @@
                 <state_interface name="effort"/>
             </joint>
-            <joint name="joint2">
+            <joint name="shoulder_roll_joint">
                 <command_interface name="position"/>
                 <state_interface name="position"/>
@@ -19,5 +19,5 @@
                 <state_interface name="effort"/>
             </joint>
-            <joint name="joint3">
+            <joint name="shoulder_yaw_joint">
                 <command_interface name="position"/>
                 <state_interface name="position"/>
@@ -25,5 +25,5 @@
                 <state_interface name="effort"/>
             </joint>
-            <joint name="joint4">
+            <joint name="elbow_pitch_joint">
                 <command_interface name="position"/>
                 <state_interface name="position"/>
@@ -31,5 +31,5 @@
                 <state_interface name="effort"/>
             </joint>
-            <joint name="joint5">
+            <joint name="elbow_yaw_joint">
                 <command_interface name="position"/>
                 <state_interface name="position"/>

Commit message: Adapt MoveIt config for Inspire hand Fixes #117

File: src/planning/arm_moveit_config/config/arm_description.ros2_control.xacro (robot description, xacro)
@@ -43,4 +43,53 @@
                 <state_interface name="velocity"/>
             </joint>
+            <joint name="wrist_roll_joint">
+                <command_interface name="position"/>
+                <state_interface name="position">
+                  <param name="initial_value">${initial_positions['wrist_roll_joint']}</param>
+                </state_interface>
+                <state_interface name="velocity"/>
+            </joint>
+            <joint name="thumb_proximal_yaw_joint">
+                <command_interface name="position"/>
+                <state_interface name="position">
+                  <param name="initial_value">${initial_positions['thumb_proximal_yaw_joint']}</param>
+                </state_interface>
+                <state_interface name="velocity"/>
+            </joint>
+            <joint name="thumb_proximal_pitch_joint">
+                <command_interface name="position"/>
+                <state_interface name="position">
+                  <param name="initial_value">${initial_positions['thumb_proximal_pitch_joint']}</param>
+                </state_interface>
+                <state_interface name="velocity"/>
+            </joint>
+            <joint name="index_proximal_joint">
+                <command_interface name="position"/>
+                <state_interface name="position">
+                  <param name="initial_value">${initial_positions['index_proximal_joint']}</param>
+                </state_interface>
+                <state_interface name="velocity"/>
+            </joint>
+            <joint name="middle_proximal_joint">
+                <command_interface name="position"/>
+                <state_interface name="position">
+                  <param name="initial_value">${initial_positions['middle_proximal_joint']}</param>
+                </state_interface>
+                <state_interface name="velocity"/>
+            </joint>
+            <joint name="ring_proximal_joint">
+                <command_interface name="position"/>
+                <state_interface name="position">
+                  <param name="initial_value">${initial_positions['ring_proximal_joint']}</param>
+                </state_interface>
+                <state_interface name="velocity"/>
+            </joint>
+            <joint name="pinky_proximal_joint">
+                <command_interface name="position"/>
+                <state_interface name="position">
+                  <param name="initial_value">${initial_positions['pinky_proximal_joint']}</param>
+                </state_interface>
+                <state_interface name="velocity"/>
+            </joint>
         </ros2_control>
     </xacro:macro>

File: src/robot_description/arm_description/urdf/hands/inspire_hand_left.xacro (robot description, xacro)
@@ -127,5 +127,5 @@
       <child link="thumb_proximal"/>
       <axis xyz="0 0 -1"/>
-      <limit lower="0" upper="0.6" effort="1" velocity="0.5"/>
+      <limit lower="0" upper="0.61" effort="1" velocity="0.5"/>
     </joint>
     <link name="thumb_intermediate">
