Commit message: hand prefix optimization

File: src/planning/arm_moveit_config/config/arm_description.ros2_control.xacro (robot description, xacro)
@@ -50,43 +50,43 @@
                 <state_interface name="velocity"/>
             </joint>
-            <joint name="thumb_proximal_yaw_joint">
+            <joint name="left_thumb_proximal_yaw_joint">
                 <command_interface name="position"/>
                 <state_interface name="position">
-                  <param name="initial_value">${initial_positions['thumb_proximal_yaw_joint']}</param>
+                  <param name="initial_value">${initial_positions['left_thumb_proximal_yaw_joint']}</param>
                 </state_interface>
                 <state_interface name="velocity"/>
             </joint>
-            <joint name="thumb_proximal_pitch_joint">
+            <joint name="left_thumb_proximal_pitch_joint">
                 <command_interface name="position"/>
                 <state_interface name="position">
-                  <param name="initial_value">${initial_positions['thumb_proximal_pitch_joint']}</param>
+                  <param name="initial_value">${initial_positions['left_thumb_proximal_pitch_joint']}</param>
                 </state_interface>
                 <state_interface name="velocity"/>
             </joint>
-            <joint name="index_proximal_joint">
+            <joint name="left_index_proximal_joint">
                 <command_interface name="position"/>
                 <state_interface name="position">
-                  <param name="initial_value">${initial_positions['index_proximal_joint']}</param>
+                  <param name="initial_value">${initial_positions['left_index_proximal_joint']}</param>
                 </state_interface>
                 <state_interface name="velocity"/>
             </joint>
-            <joint name="middle_proximal_joint">
+            <joint name="left_middle_proximal_joint">
                 <command_interface name="position"/>
                 <state_interface name="position">
-                  <param name="initial_value">${initial_positions['middle_proximal_joint']}</param>
+                  <param name="initial_value">${initial_positions['left_middle_proximal_joint']}</param>
                 </state_interface>
                 <state_interface name="velocity"/>
             </joint>
-            <joint name="ring_proximal_joint">
+            <joint name="left_ring_proximal_joint">
                 <command_interface name="position"/>
                 <state_interface name="position">
-                  <param name="initial_value">${initial_positions['ring_proximal_joint']}</param>
+                  <param name="initial_value">${initial_positions['left_ring_proximal_joint']}</param>
                 </state_interface>
                 <state_interface name="velocity"/>
             </joint>
-            <joint name="pinky_proximal_joint">
+            <joint name="left_pinky_proximal_joint">
                 <command_interface name="position"/>
                 <state_interface name="position">
-                  <param name="initial_value">${initial_positions['pinky_proximal_joint']}</param>
+                  <param name="initial_value">${initial_positions['left_pinky_proximal_joint']}</param>
                 </state_interface>
                 <state_interface name="velocity"/>

File: src/robot_description/arm_description/urdf/macros/ros2_control.xacro (robot description, xacro)
@@ -72,5 +72,5 @@
                 </hardware>
                 <!-- 6 actuated joints (command + state) -->
-                <joint name="thumb_proximal_yaw_joint">
+                <joint name="left_thumb_proximal_yaw_joint">
                     <command_interface name="position"/>
                     <state_interface name="position"/>
@@ -78,5 +78,5 @@
                     <state_interface name="effort"/>
                 </joint>
-                <joint name="thumb_proximal_pitch_joint">
+                <joint name="left_thumb_proximal_pitch_joint">
                     <command_interface name="position"/>
                     <state_interface name="position"/>
@@ -84,5 +84,5 @@
                     <state_interface name="effort"/>
                 </joint>
-                <joint name="index_proximal_joint">
+                <joint name="left_index_proximal_joint">
                     <command_interface name="position"/>
                     <state_interface name="position"/>
@@ -90,5 +90,5 @@
                     <state_interface name="effort"/>
                 </joint>
-                <joint name="middle_proximal_joint">
+                <joint name="left_middle_proximal_joint">
                     <command_interface name="position"/>
                     <state_interface name="position"/>
@@ -96,5 +96,5 @@
                     <state_interface name="effort"/>
                 </joint>
-                <joint name="ring_proximal_joint">
+                <joint name="left_ring_proximal_joint">
                     <command_interface name="position"/>
                     <state_interface name="position"/>
@@ -102,5 +102,5 @@
                     <state_interface name="effort"/>
                 </joint>
-                <joint name="pinky_proximal_joint">
+                <joint name="left_pinky_proximal_joint">
                     <command_interface name="position"/>
                     <state_interface name="position"/>
@@ -109,30 +109,30 @@
                 </joint>
                 <!-- 6 mimic joints (state only) -->
-                <joint name="thumb_intermediate_joint">
+                <joint name="left_thumb_intermediate_joint">
                     <state_interface name="position"/>
                     <state_interface name="velocity"/>
                     <state_interface name="effort"/>
                 </joint>
-                <joint name="thumb_distal_joint">
+                <joint name="left_thumb_distal_joint">
                     <state_interface name="position"/>
                     <state_interface name="velocity"/>
                     <state_interface name="effort"/>
                 </joint>
-                <joint name="index_intermediate_joint">
+                <joint name="left_index_intermediate_joint">
                     <state_interface name="position"/>
                     <state_interface name="velocity"/>
                     <state_interface name="effort"/>
                 </joint>
-                <joint name="middle_intermediate_joint">
+                <joint name="left_middle_intermediate_joint">
                     <state_interface name="position"/>
                     <state_interface name="velocity"/>
                     <state_interface name="effort"/>
                 </joint>
-                <joint name="ring_intermediate_joint">
+                <joint name="left_ring_intermediate_joint">
                     <state_interface name="position"/>
                     <state_interface name="velocity"/>
                     <state_interface name="effort"/>
                 </joint>
-                <joint name="pinky_intermediate_joint">
+                <joint name="left_pinky_intermediate_joint">
                     <state_interface name="position"/>
                     <state_interface name="velocity"/>

File: src/robot_description/dual_arm_description/urdf/dual_arm_base.xacro (robot description, xacro)
@@ -7,4 +7,5 @@
   <xacro:inspire_hand_left
     parent="urdf_l_wrist_assembly"
+    prefix="left_"
     mount_x="-0.0"
     mount_y="-0.07"
@@ -15,4 +16,5 @@
   <xacro:inspire_hand_right
     parent="urdf_r_wrist_assembly"
+    prefix="right_"
     mount_x="-0.0"
     mount_y="-0.07"

File: src/robot_description/hand_description/urdf/hands/inspire_hand_left.xacro (robot description, xacro)
@@ -6,12 +6,12 @@
        6 actuated joints + 6 mimic joints + 5 tip fixed joints
        Collision geometry uses box primitives (OBJ meshes lack normals for DART) -->
-  <xacro:macro name="inspire_hand_left" params="parent mount_x:=0.0 mount_y:=0.07 mount_z:=-0.03 mount_roll:=0.0 mount_pitch:=0.0 mount_yaw:=3.14159">
+  <xacro:macro name="inspire_hand_left" params="parent prefix:=left_ mount_x:=0.0 mount_y:=0.07 mount_z:=-0.03 mount_roll:=0.0 mount_pitch:=0.0 mount_yaw:=3.14159">
     <!-- Attach hand_base_link directly to parent (replaces dummy base link) -->
-    <joint name="hand_base_joint" type="fixed">
+    <joint name="${prefix}hand_base_joint" type="fixed">
       <origin xyz="${mount_x} ${mount_y} ${mount_z}" rpy="${mount_roll} ${mount_pitch} ${mount_yaw}"/>
       <parent link="${parent}"/>
-      <child link="hand_base_link"/>
-    </joint>
-    <link name="hand_base_link">
+      <child link="${prefix}hand_base_link"/>
+    </joint>
+    <link name="${prefix}hand_base_link">
       <inertial>
         <origin xyz="-0.0025264 -0.066047 -0.0019598" rpy="0 0 0"/>
@@ -75,5 +75,5 @@
     </link>
     <!-- ========== THUMB ========== -->
-    <link name="thumb_proximal_base">
+    <link name="${prefix}thumb_proximal_base">
       <inertial>
         <origin xyz="0.0048817 0.0009382 -0.00722" rpy="0 0 0"/>
@@ -95,12 +95,12 @@
     </link>
     <!-- Actuated: thumb yaw -->
-    <joint name="thumb_proximal_yaw_joint" type="revolute">
+    <joint name="${prefix}thumb_proximal_yaw_joint" type="revolute">
       <origin xyz="-0.01696 -0.0691 0.02045" rpy="1.5708 -1.5708 0"/>
-      <parent link="hand_base_link"/>
-      <child link="thumb_proximal_base"/>
+      <parent link="${prefix}hand_base_link"/>
+      <child link="${prefix}thumb_proximal_base"/>
       <axis xyz="0 0 1"/>
       <limit lower="0" upper="1.31" effort="1" velocity="0.5"/>
     </joint>
-    <link name="thumb_proximal">
+    <link name="${prefix}thumb_proximal">
       <inertial>
         <origin xyz="0.021932 -0.012785 -0.0080386" rpy="0 0 0"/>
@@ -122,12 +122,12 @@
     </link>
     <!-- Actuated: thumb pitch -->
-    <joint name="thumb_proximal_pitch_joint" type="revolute">
+    <joint name="${prefix}thumb_proximal_pitch_joint" type="revolute">
       <origin xyz="0.0099867 0.0098242 -0.0089" rpy="-1.5708 0 0.16939"/>
-      <parent link="thumb_proximal_base"/>
-      <child link="thumb_proximal"/>
+      <parent link="${prefix}thumb_proximal_base"/>
+      <child link="${prefix}thumb_proximal"/>
       <axis xyz="0 0 -1"/>
       <limit lower="0" upper="0.61" effort="1" velocity="0.5"/>
     </joint>
-    <link name="thumb_intermediate">
+    <link name="${prefix}thumb_intermediate">
       <inertial>
         <origin xyz="0.0095544 0.0016282 -0.0071997" rpy="0 0 0"/>
@@ -149,13 +149,13 @@
     </link>
     <!-- Mimic: thumb intermediate (follows thumb_proximal_pitch) -->
-    <joint name="thumb_intermediate_joint" type="revolute">
+    <joint name="${prefix}thumb_intermediate_joint" type="revolute">
       <origin xyz="0.04407 -0.034553 -0.0008" rpy="0 0 0"/>
-      <parent link="thumb_proximal"/>
-      <child link="thumb_intermediate"/>
+      <parent link="${prefix}thumb_proximal"/>
+      <child link="${prefix}thumb_intermediate"/>
       <axis xyz="0 0 -1"/>
       <limit lower="0" upper="0.8" effort="1" velocity="0.5"/>
-      <mimic joint="thumb_proximal_pitch_joint" multiplier="1.334" offset="0"/>
-    </joint>
-    <link name="thumb_distal">
+      <mimic joint="${prefix}thumb_proximal_pitch_joint" multiplier="1.334" offset="0"/>
+    </joint>
+    <link name="${prefix}thumb_distal">
       <inertial>
         <origin xyz="0.0092888 -0.0049529 -0.0060033" rpy="0 0 0"/>
@@ -177,14 +177,14 @@
     </link>
     <!-- Mimic: thumb distal (follows thumb_proximal_pitch) -->
-    <joint name="thumb_distal_joint" type="revolute">
+    <joint name="${prefix}thumb_distal_joint" type="revolute">
       <origin xyz="0.020248 -0.010156 -0.0012" rpy="0 0 0"/>
-      <parent link="thumb_intermediate"/>
-      <child link="thumb_distal"/>
+      <parent link="${prefix}thumb_intermediate"/>
+      <child link="${prefix}thumb_distal"/>
       <axis xyz="0 0 -1"/>
       <limit lower="0" upper="0.4" effort="1" velocity="0.5"/>
-      <mimic joint="thumb_proximal_pitch_joint" multiplier="0.667" offset="0"/>
+      <mimic joint="${prefix}thumb_proximal_pitch_joint" multiplier="0.667" offset="0"/>
     </joint>
     <!-- ========== INDEX FINGER ========== -->
-    <link name="index_proximal">
+    <link name="${prefix}index_proximal">
       <inertial>
         <origin xyz="0.0012259 -0.011942 -0.0060001" rpy="0 0 0"/>
@@ -206,12 +206,12 @@
     </link>
     <!-- Actuated: index proximal -->
-    <joint name="index_proximal_joint" type="revolute">
+    <joint name="${prefix}index_proximal_joint" type="revolute">
       <origin xyz="0.00028533 -0.13653 0.032268" rpy="-0.034907 0 0"/>
-      <parent link="hand_base_link"/>
-      <child link="index_proximal"/>
+      <parent link="${prefix}hand_base_link"/>
+      <child link="${prefix}index_proximal"/>
       <axis xyz="0 0 -1"/>
       <limit lower="0" upper="1.47" effort="1" velocity="0.5"/>
     </joint>
-    <link name="index_intermediate">
+    <link name="${prefix}index_intermediate">
       <inertial>
         <origin xyz="0.0019697 -0.019589 -0.005" rpy="0 0 0"/>
@@ -233,14 +233,14 @@
     </link>
     <!-- Mimic: index intermediate (follows index_proximal) -->
-    <joint name="index_intermediate_joint" type="revolute">
+    <joint name="${prefix}index_intermediate_joint" type="revolute">
       <origin xyz="-0.0026138 -0.032026 -0.001" rpy="0 0 0"/>
-      <parent link="index_proximal"/>
-      <child link="index_intermediate"/>
+      <parent link="${prefix}index_proximal"/>
+      <child link="${prefix}index_intermediate"/>
       <axis xyz="0 0 -1"/>
       <limit lower="-0.04545" upper="1.56" effort="1" velocity="0.5"/>
-      <mimic joint="index_proximal_joint" multiplier="1.06399" offset="-0.04545"/>
+      <mimic joint="${prefix}index_proximal_joint" multiplier="1.06399" offset="-0.04545"/>
     </joint>
     <!-- ========== MIDDLE FINGER ========== -->
-    <link name="middle_proximal">
+    <link name="${prefix}middle_proximal">
       <inertial>
         <origin xyz="0.001297 -0.011934 -0.0060001" rpy="0 0 0"/>
@@ -262,12 +262,12 @@
     </link>
     <!-- Actuated: middle proximal -->
-    <joint name="middle_proximal_joint" type="revolute">
+    <joint name="${prefix}middle_proximal_joint" type="revolute">
       <origin xyz="0.00028533 -0.1371 0.01295" rpy="0 0 0"/>
-      <parent link="hand_base_link"/>
-      <child link="middle_proximal"/>
+      <parent link="${prefix}hand_base_link"/>
+      <child link="${prefix}middle_proximal"/>
       <axis xyz="0 0 -1"/>
       <limit lower="0" upper="1.47" effort="1" velocity="0.5"/>
     </joint>
-    <link name="middle_intermediate">
+    <link name="${prefix}middle_intermediate">
       <inertial>
         <origin xyz="0.001921 -0.020796 -0.005" rpy="0 0 0"/>
@@ -289,14 +289,14 @@
     </link>
     <!-- Mimic: middle intermediate (follows middle_proximal) -->
-    <joint name="middle_intermediate_joint" type="revolute">
+    <joint name="${prefix}middle_intermediate_joint" type="revolute">
       <origin xyz="-0.0024229 -0.032041 -0.001" rpy="0 0 0"/>
-      <parent link="middle_proximal"/>
-      <child link="middle_intermediate"/>
+      <parent link="${prefix}middle_proximal"/>
+      <child link="${prefix}middle_intermediate"/>
       <axis xyz="0 0 -1"/>
       <limit lower="-0.04545" upper="1.56" effort="1" velocity="0.5"/>
-      <mimic joint="middle_proximal_joint" multiplier="1.06399" offset="-0.04545"/>
+      <mimic joint="${prefix}middle_proximal_joint" multiplier="1.06399" offset="-0.04545"/>
     </joint>
     <!-- ========== RING FINGER ========== -->
-    <link name="ring_proximal">
+    <link name="${prefix}ring_proximal">
       <inertial>
         <origin xyz="0.001297 -0.011934 -0.0060002" rpy="0 0 0"/>
@@ -318,12 +318,12 @@
     </link>
     <!-- Actuated: ring proximal -->
-    <joint name="ring_proximal_joint" type="revolute">
+    <joint name="${prefix}ring_proximal_joint" type="revolute">
       <origin xyz="0.00028533 -0.13691 -0.0062872" rpy="0.05236 0 0"/>
-      <parent link="hand_base_link"/>
-      <child link="ring_proximal"/>
+      <parent link="${prefix}hand_base_link"/>
+      <child link="${prefix}ring_proximal"/>
       <axis xyz="0 0 -1"/>
       <limit lower="0" upper="1.47" effort="1" velocity="0.5"/>
     </joint>
-    <link name="ring_intermediate">
+    <link name="${prefix}ring_intermediate">
       <inertial>
         <origin xyz="0.0021753 -0.019567 -0.005" rpy="0 0 0"/>
@@ -345,14 +345,14 @@
     </link>
     <!-- Mimic: ring intermediate (follows ring_proximal) -->
-    <joint name="ring_intermediate_joint" type="revolute">
+    <joint name="${prefix}ring_intermediate_joint" type="revolute">
       <origin xyz="-0.0024229 -0.032041 -0.001" rpy="0 0 0"/>
-      <parent link="ring_proximal"/>
-      <child link="ring_intermediate"/>
+      <parent link="${prefix}ring_proximal"/>
+      <child link="${prefix}ring_intermediate"/>
       <axis xyz="0 0 -1"/>
       <limit lower="-0.04545" upper="1.56" effort="1" velocity="0.5"/>
-      <mimic joint="ring_proximal_joint" multiplier="1.06399" offset="-0.04545"/>
+      <mimic joint="${prefix}ring_proximal_joint" multiplier="1.06399" offset="-0.04545"/>
     </joint>
     <!-- ========== PINKY FINGER ========== -->
-    <link name="pinky_proximal">
+    <link name="${prefix}pinky_proximal">
       <inertial>
         <origin xyz="0.001297 -0.011934 -0.0060001" rpy="0 0 0"/>
@@ -374,12 +374,12 @@
     </link>
     <!-- Actuated: pinky proximal -->
-    <joint name="pinky_proximal_joint" type="revolute">
+    <joint name="${prefix}pinky_proximal_joint" type="revolute">
       <origin xyz="0.00028533 -0.13571 -0.025488" rpy="0.10472 0 0"/>
-      <parent link="hand_base_link"/>
-      <child link="pinky_proximal"/>
+      <parent link="${prefix}hand_base_link"/>
+      <child link="${prefix}pinky_proximal"/>
       <axis xyz="0 0 -1"/>
       <limit lower="0" upper="1.47" effort="1" velocity="0.5"/>
     </joint>
-    <link name="pinky_intermediate">
+    <link name="${prefix}pinky_intermediate">
       <inertial>
         <origin xyz="0.0024748 -0.016203 -0.0050031" rpy="0 0 0"/>
@@ -401,42 +401,42 @@
     </link>
     <!-- Mimic: pinky intermediate (follows pinky_proximal) -->
-    <joint name="pinky_intermediate_joint" type="revolute">
+    <joint name="${prefix}pinky_intermediate_joint" type="revolute">
       <origin xyz="-0.0024229 -0.032041 -0.001" rpy="0 0 0"/>
-      <parent link="pinky_proximal"/>
-      <child link="pinky_intermediate"/>
+      <parent link="${prefix}pinky_proximal"/>
+      <child link="${prefix}pinky_intermediate"/>
       <axis xyz="0 0 -1"/>
       <limit lower="-0.04545" upper="1.56" effort="1" velocity="0.5"/>
-      <mimic joint="pinky_proximal_joint" multiplier="1.06399" offset="-0.04545"/>
+      <mimic joint="${prefix}pinky_proximal_joint" multiplier="1.06399" offset="-0.04545"/>
     </joint>
     <!-- ========== FINGERTIP LINKS (fixed) ========== -->
-    <link name="thumb_tip"/>
-    <joint name="thumb_tip_joint" type="fixed">
+    <link name="${prefix}thumb_tip"/>
+    <joint name="${prefix}thumb_tip_joint" type="fixed">
       <origin xyz="0.0202 -0.0140 -0.006" rpy="0 0 0"/>
-      <parent link="thumb_distal"/>
-      <child link="thumb_tip"/>
-    </joint>
-    <link name="index_tip"/>
-    <joint name="index_tip_joint" type="fixed">
+      <parent link="${prefix}thumb_distal"/>
+      <child link="${prefix}thumb_tip"/>
+    </joint>
+    <link name="${prefix}index_tip"/>
+    <joint name="${prefix}index_tip_joint" type="fixed">
       <origin xyz="-0.0008 -0.045 -0.005" rpy="0 0 0"/>
-      <parent link="index_intermediate"/>
-      <child link="index_tip"/>
-    </joint>
-    <link name="middle_tip"/>
-    <joint name="middle_tip_joint" type="fixed">
+      <parent link="${prefix}index_intermediate"/>
+      <child link="${prefix}index_tip"/>
+    </joint>
+    <link name="${prefix}middle_tip"/>
+    <joint name="${prefix}middle_tip_joint" type="fixed">
       <origin xyz="-0.001 -0.048 -0.005" rpy="0 0 0"/>
-      <parent link="middle_intermediate"/>
-      <child link="middle_tip"/>
-    </joint>
-    <link name="ring_tip"/>
-    <joint name="ring_tip_joint" type="fixed">
+      <parent link="${prefix}middle_intermediate"/>
+      <child link="${prefix}middle_tip"/>
+    </joint>
+    <link name="${prefix}ring_tip"/>
+    <joint name="${prefix}ring_tip_joint" type="fixed">
       <origin xyz="-0.0008 -0.045 -0.005" rpy="0 0 0"/>
-      <parent link="ring_intermediate"/>
-      <child link="ring_tip"/>
-    </joint>
-    <link name="pinky_tip"/>
-    <joint name="pinky_tip_joint" type="fixed">
+      <parent link="${prefix}ring_intermediate"/>
+      <child link="${prefix}ring_tip"/>
+    </joint>
+    <link name="${prefix}pinky_tip"/>
+    <joint name="${prefix}pinky_tip_joint" type="fixed">
       <origin xyz="-0.0008 -0.037 -0.005" rpy="0 0 0"/>
-      <parent link="pinky_intermediate"/>
-      <child link="pinky_tip"/>
+      <parent link="${prefix}pinky_intermediate"/>
+      <child link="${prefix}pinky_tip"/>
     </joint>
   </xacro:macro>
